File: pcb/board/termistor.sch (KiCad schematic (older format))
At the start: 10 parts, among them U1 OPA356xxD, U2 OPA356xxD

Commit message: Tidy up thermistor schematic
Parts:
- removed R1: 2k7, symbol pspice:R
- removed R2, R5: 1k, symbol pspice:R
- removed R3: 3k3, symbol pspice:R
- removed R4: 1k8, symbol pspice:R
- removed R6: 180, symbol pspice:R
- removed TH1: KTY81, symbol Sensor_Temperature:KTY81
- removed TH2: Thermistor_NTC, symbol Device:Thermistor_NTC
- removed U1, U2: OPA356xxD, Package_SO:SOIC-8_3.9x4.9mm_P1.27mm, symbol Amplifier_Operational:OPA356xxD
- added R?: 3.3k, symbol Device:R
- added R? (x2): 1k, symbol Device:R
- added R?: 2.7k, symbol Device:R
- added R?: 180, symbol Device:R
- added R?: 1.8k, symbol Device:R
- added TH?: KTY81, symbol Sensor_Temperature:KTY81
- added TH?: Thermistor_NTC, symbol Device:Thermistor_NTC
- added U? (x2): OPA356xxD, Package_SO:SOIC-8_3.9x4.9mm_P1.27mm, symbol Amplifier_Operational:OPA356xxD
Connections:
- net labels added: +3V3
- wire segments 26 -> 30
Other:
- note added: "IGBTs"
- note added: "Motor"
