File: pcb/board/electric-FIAT.sch (KiCad schematic (older format))
At the start: 0 parts

Commit message: Thermistor
Parts:
- added R?: 3.3k, symbol Device:R
- added R? (x2): 1k, symbol Device:R
- added R?: 2.7k, symbol Device:R
- added R?: 180, symbol Device:R
- added R?: 1.8k, symbol Device:R
- added TH?: KTY81, symbol Sensor_Temperature:KTY81
- added TH?: Thermistor_NTC, symbol Device:Thermistor_NTC
- added U? (x2): OPA356xxD, Package_SO:SOIC-8_3.9x4.9mm_P1.27mm, symbol Amplifier_Operational:OPA356xxD
Connections:
- new net: R?.1, R?.2, U?.2 (-) (x2)
- new net: R?.1, TH?.2, U?.3 (+) (x2)
- new net +1V8: R?.2, R?.2
- new net +3V3: TH?.1, TH?.1, U?.7 (V+), U?.7 (V+)
- new net GND: R?.2, R?.2, U?.4 (V-), U?.4 (V-)
- new net Inverter_temp: R?.1, U?.6
- new net Motor_temp: R?.1, U?.6
Other:
- note added: "IGBTs"
- note added: "Motor"
- note added: "Temperature Sensors"

Commit message: Anotate Schematic
Parts:
- gave numbers to parts that had none: 10
Changed lines of the file:
@@
 EESchema Schematic File Version 4
-LIBS:electric-FIAT-cache
 EELAYER 30 0
 EELAYER END
@@
 $EndSheet
 $Comp
-L Amplifier_Operational:OPA356xxD U?
+L Amplifier_Operational:OPA356xxD U4
 U 1 1 5DBC9E5B
 P 8350 1700
-F 0 "U?" H 8400 2000 50  0000 L CNN
+F 0 "U4" H 8400 2000 50  0000 L CNN
 F 1 "OPA356xxD" H 8400 1900 50  0000 L CNN
 F 2 "Package_SO:SOIC-8_3.9x4.9mm_P1.27mm" H 8250 1500 50  0001 L CNN
@@
 $EndComp
 $Comp
-L Device:R R?
+L Device:R R4
 U 1 1 5DBCC022
 P 8250 2600
-F 0 "R?" V 8043 2600 50  0000 C CNN
+F 0 "R4" V 8043 2600 50  0000 C CNN
 F 1 "3.3k" V 8134 2600 50  0000 C CNN
 F 2 "" V 8180 2600 50  0001 C CNN
@@
 	8400 2600 8650 2600
 $Comp
-L power:+3.3V #PWR?
+L power:+3.3V #PWR018
 U 1 1 5DBD0637
 P 8250 1350
-F 0 "#PWR?" H 8250 1200 50  0001 C CNN
+F 0 "#PWR018" H 8250 1200 50  0001 C CNN
 F 1 "+3.3V" H 8265 1523 50  0000 C CNN
 F 2 "" H 8250 1350 50  0001 C CNN
@@
 	8250 1350 8250 1400
 $Comp
-L power:GND #PWR?
+L power:GND #PWR022
 U 1 1 5DBD246A
 P 8250 2050
-F 0 "#PWR?" H 8250 1800 50  0001 C CNN
+F 0 "#PWR022" H 8250 1800 50  0001 C CNN
 F 1 "GND" H 8255 1877 50  0000 C CNN
 F 2 "" H 8250 2050 50  0001 C CNN
@@
 	7950 1800 8050 1800
 $Comp
-L power:+1V8 #PWR?
+L power:+1V8 #PWR024
 U 1 1 5DBD45BD
 P 7400 2550
-F 0 "#PWR?" H 7400 2400 50  0001 C CNN
+F 0 "#PWR024" H 7400 2400 50  0001 C CNN
 F 1 "+1V8" H 7415 2723 50  0000 C CNN
 F 2 "" H 7400 2550 50  0001 C CNN
@@
 $EndComp
 $Comp
-L Device:R R?
+L Device:R R3
 U 1 1 5DBD5C6F
 P 7700 2600
-F 0 "R?" V 7493 2600 50  0000 C CNN
+F 0 "R3" V 7493 2600 50  0000 C CNN
 F 1 "1k" V 7584 2600 50  0000 C CNN
 F 2 "" V 7630 2600 50  0001 C CNN
@@
 Connection ~ 7950 2600
 $Comp
-L Sensor_Temperature:KTY81 TH?
+L Sensor_Temperature:KTY81 TH1
 U 1 1 5DBD769F
 P 7400 1400
-F 0 "TH?" H 7497 1446 50  0000 L CNN
+F 0 "TH1" H 7497 1446 50  0000 L CNN
 F 1 "KTY81" H 7497 1355 50  0000 L CNN
 F 2 "" V 7600 1400 50  0001 C CNN
@@
 $EndComp
 $Comp
-L Device:R R?
+L Device:R R1
 U 1 1 5DBD9F8E
 P 7400 1800
-F 0 "R?" H 7470 1846 50  0000 L CNN
+F 0 "R1" H 7470 1846 50  0000 L CNN
 F 1 "2.7k" H 7470 1755 50  0000 L CNN
 F 2 "" V 7330 1800 50  0001 C CNN
@@
 	7400 1600 7400 1650
 $Comp
-L power:GND #PWR?
+L power:GND #PWR020
 U 1 1 5DBDC474
 P 7400 2000
-F 0 "#PWR?" H 7400 1750 50  0001 C CNN
+F 0 "#PWR020" H 7400 1750 50  0001 C CNN
 F 1 "GND" H 7405 1827 50  0000 C CNN
 F 2 "" H 7400 2000 50  0001 C CNN
@@
 	7400 2000 7400 1950
 $Comp
-L power:+3V3 #PWR?
+L power:+3V3 #PWR016
 U 1 1 5DBDD44B
 P 7400 1200
-F 0 "#PWR?" H 7400 1050 50  0001 C CNN
+F 0 "#PWR016" H 7400 1050 50  0001 C CNN
 F 1 "+3V3" H 7415 1373 50  0000 C CNN
 F 2 "" H 7400 1200 50  0001 C CNN
@@
 	7400 1200 7400 1250
 $Comp
-L Amplifier_Operational:OPA356xxD U?
+L Amplifier_Operational:OPA356xxD U5
 U 1 1 5DBF673E
 P 10300 1700
-F 0 "U?" H 10350 2000 50  0000 L CNN
+F 0 "U5" H 10350 2000 50  0000 L CNN
 F 1 "OPA356xxD" H 10350 1900 50  0000 L CNN
 F 2 "Package_SO:SOIC-8_3.9x4.9mm_P1.27mm" H 10200 1500 50  0001 L CNN
@@
 $EndComp
 $Comp
-L Device:R R?
+L Device:R R6
 U 1 1 5DBF6744
 P 10200 2600
-F 0 "R?" V 9993 2600 50  0000 C CNN
+F 0 "R6" V 9993 2600 50  0000 C CNN
 F 1 "180" V 10084 2600 50  0000 C CNN
 F 2 "" V 10130 2600 50  0001 C CNN
@@
 	10350 2600 10600 2600
 $Comp
-L power:+3.3V #PWR?
+L power:+3.3V #PWR019
 U 1 1 5DBF674C
 P 10200 1350
-F 0 "#PWR?" H 10200 1200 50  0001 C CNN
+F 0 "#PWR019" H 10200 1200 50  0001 C CNN
 F 1 "+3.3V" H 10215 1523 50  0000 C CNN
 F 2 "" H 10200 1350 50  0001 C CNN
@@
 	10200 1350 10200 1400
 $Comp
-L power:GND #PWR?
+L power:GND #PWR023
 U 1 1 5DBF6753
 P 10200 2050
-F 0 "#PWR?" H 10200 1800 50  0001 C CNN
+F 0 "#PWR023" H 10200 1800 50  0001 C CNN
 F 1 "GND" H 10205 1877 50  0000 C CNN
 F 2 "" H 10200 2050 50  0001 C CNN
@@
 	9900 1800 10000 1800
 $Comp
-L power:+1V8 #PWR?
+L power:+1V8 #PWR025
 U 1 1 5DBF675D
 P 9350 2550
-F 0 "#PWR?" H 9350 2400 50  0001 C CNN
+F 0 "#PWR025" H 9350 2400 50  0001 C CNN
 F 1 "+1V8" H 9365 2723 50  0000 C CNN
 F 2 "" H 9350 2550 50  0001 C CNN
@@
 $EndComp
 $Comp
-L Device:R R?
+L Device:R R5
 U 1 1 5DBF6763
 P 9650 2600
-F 0 "R?" V 9443 2600 50  0000 C CNN
+F 0 "R5" V 9443 2600 50  0000 C CNN
 F 1 "1k" V 9534 2600 50  0000 C CNN
 F 2 "" V 9580 2600 50  0001 C CNN
@@
 Connection ~ 9900 2600
 $Comp
-L Device:R R?
+L Device:R R2
 U 1 1 5DBF6773
 P 9350 1800
-F 0 "R?" H 9420 1846 50  0000 L CNN
+F 0 "R2" H 9420 1846 50  0000 L CNN
 F 1 "1.8k" H 9420 1755 50  0000 L CNN
 F 2 "" V 9280 1800 50  0001 C CNN
@@
 	9350 1600 9350 1650
 $Comp
-L power:GND #PWR?
+L power:GND #PWR021
 U 1 1 5DBF677D
 P 9350 2000
-F 0 "#PWR?" H 9350 1750 50  0001 C CNN
+F 0 "#PWR021" H 9350 1750 50  0001 C CNN
 F 1 "GND" H 9355 1827 50  0000 C CNN
 F 2 "" H 9350 2000 50  0001 C CNN
@@
 	9350 2000 9350 1950
 $Comp
-L power:+3V3 #PWR?
+L power:+3V3 #PWR017
 U 1 1 5DBF6784
 P 9350 1200
-F 0 "#PWR?" H 9350 1050 50  0001 C CNN
+F 0 "#PWR017" H 9350 1050 50  0001 C CNN
 F 1 "+3V3" H 9365 1373 50  0000 C CNN
 F 2 "" H 9350 1200 50  0001 C CNN
@@
 	9350 1200 9350 1250
 $Comp
-L Device:Thermistor_NTC TH?
+L Device:Thermistor_NTC TH2
 U 1 1 5DBF7608
 P 9350 1400
-F 0 "TH?" H 9448 1446 50  0000 L CNN
+F 0 "TH2" H 9448 1446 50  0000 L CNN
 F 1 "Thermistor_NTC" H 9448 1355 50  0000 L CNN
 F 2 "" H 9350 1450 50  0001 C CNN

Commit message: MCU and Decoupling
Parts:
- removed U4, U5: OPA356xxD, Package_SO:SOIC-8_3.9x4.9mm_P1.27mm, symbol Amplifier_Operational:OPA356xxD
- added C10, C13, C15, C16, C17, C18, C7, C8, C9: 100n, Capacitor_SMD:C_0805_2012Metric, symbol Device:C
- added C11, C12: 2.2n, Capacitor_SMD:C_0805_2012Metric, symbol Device:C
- added C14: 1u, Capacitor_SMD:C_0805_2012Metric, symbol Device:C
- added C?: 4.7u, Capacitor_SMD:C_0805_2012Metric, symbol Device:C
- added U4, U5: OPA356xxDBV, Package_TO_SOT_SMD:SOT-23-5, symbol Amplifier_Operational:OPA356xxDBV
- added U6: STM32F405RGTx, Package_QFP:LQFP-64_10x10mm_P0.5mm, symbol MCU_ST_STM32F4:STM32F405RGTx
- R1, R2, R3, R4, R5, R6: footprint (none) -> Resistor_SMD:R_0805_2012Metric
Connections:
- net +1V8: now also C10.1, C9.1
- net +3V3: now also C13.1, C14.1, C15.1, C16.1, C17.1, C18.1, C7.1, C8.1, C?.1, U4.5 (V+), U5.5 (V+), U6.13 (VDDA), U6.19 (VDD), U6.32 (VDD), U6.48 (VDD), U6.64 (VDD)
- net GND: now also C10.2, C11.2, C12.2, C13.2, C14.2, C15.2, C16.2, C17.2, C18.2, C7.2, C8.2, C9.2, C?.2, U4.2 (V-), U5.2 (V-), U6.12 (VSSA), U6.18 (VSS), U6.63 (VSS)
- net Inverter_temp: now also U5.1
- net Motor_temp: now also U4.1
- net at R3.1, R4.2: now also U4.4 (-)
- net at R1.1, TH1.2: now also U4.3 (+)
- net at R5.1, R6.2: now also U5.4 (-)
- net at R2.1, TH2.2: now also U5.3 (+)
- new net VCAP_1: C11.1, U6.31 (VCAP_1)
- new net VCAP_2: C12.1, U6.47 (VCAP_2)
- no-connect marks 0 -> 1
Other:
- note added: "ADC"
- note added: "Decoupling"
- moved on the sheet: R1, R2, R3, R4, R5, R6, TH1, TH2

Commit message: IMU
Parts:
- added J1: Conn_01x10_Female, symbol Connector:Conn_01x10_Female
- gave numbers to parts that had none: 1
Connections:
- net +3V3: now also J1.1 (Pin_1)
- net GND: now also J1.2 (Pin_2), J1.5 (Pin_5)
- new net SPI1_CS_Accel: J1.8 (Pin_8)
- new net SPI1_CS_Gyro: J1.9 (Pin_9)
- new net SPI1_CS_Magnet: J1.10 (Pin_10)
- new net SPI1_MISO: J1.6 (Pin_6), J1.7 (Pin_7)
- new net SPI1_MOSI: J1.4 (Pin_4)
- new net SPI1_SCK: J1.3 (Pin_3)
Other:
- note added: "IMU"
Changed lines of the file:
@@
 $EndComp
 $Comp
-L Device:C C?
+L Device:C C19
 U 1 1 5DD27FA0
 P 4200 1250
-F 0 "C?" H 4315 1296 50  0000 L CNN
+F 0 "C19" H 4315 1296 50  0000 L CNN
 F 1 "4.7u" H 4315 1205 50  0000 L CNN
 F 2 "Capacitor_SMD:C_0805_2012Metric" H 4238 1100 50  0001 C CNN
@@
 Wire Wire Line
 	3000 1050 3400 1050
+$Comp
+L Connector:Conn_01x10_Female J1
+U 1 1 5DD2DFA2
+P 6000 7000
+F 0 "J1" H 6028 6976 50  0000 L CNN
+F 1 "Conn_01x10_Female" H 6028 6885 50  0000 L CNN
+F 2 "" H 6000 7000 50  0001 C CNN
+F 3 "~" H 6000 7000 50  0001 C CNN
+	1    6000 7000
+	1    0    0    -1
+$EndComp
+Text Notes 5650 6250 0    100  ~ 20
+IMU
+$Comp
+L power:+3V3 #PWR038
+U 1 1 5DD331B4
+P 5700 6550
+F 0 "#PWR038" H 5700 6400 50  0001 C CNN
+F 1 "+3V3" H 5715 6723 50  0000 C CNN
+F 2 "" H 5700 6550 50  0001 C CNN
+F 3 "" H 5700 6550 50  0001 C CNN
+	1    5700 6550
+	1    0    0    -1
+$EndComp
+Wire Wire Line
+	5700 6550 5700 6600
+Wire Wire Line
+	5700 6600 5800 6600
+$Comp
+L power:GND #PWR039
+U 1 1 5DD3B561
+P 5100 7000
+F 0 "#PWR039" H 5100 6750 50  0001 C CNN
+F 1 "GND" H 5105 6827 50  0000 C CNN
+F 2 "" H 5100 7000 50  0001 C CNN
+F 3 "" H 5100 7000 50  0001 C CNN
+	1    5100 7000
+	1    0    0    -1
+$EndComp
+Text Label 5800 6800 2    50   ~ 0
+SPI1_SCK
+Text Label 5800 6900 2    50   ~ 0
+SPI1_MOSI
+Text Label 5750 7150 2    50   ~ 0
+SPI1_MISO
+Wire Wire Line
+	5750 7150 5800 7150
+Wire Wire Line
+	5800 7150 5800 7100
+Wire Wire Line
+	5800 7200 5800 7150
+Connection ~ 5800 7150
+Text Label 5800 7300 2    50   ~ 0
+SPI1_CS_Accel
+Text Label 5800 7400 2    50   ~ 0
+SPI1_CS_Gyro
+Text Label 5800 7500 2    50   ~ 0
+SPI1_CS_Magnet
+Wire Wire Line
+	5100 7000 5800 7000
+Wire Wire Line
+	5100 7000 5100 6700
+Wire Wire Line
+	5100 6700 5800 6700
+Connection ~ 5100 7000
 $EndSCHEMATC

Commit message: Initialized STM32F405RGTx
Parts:
- added R7: 10k, Resistor_SMD:R_0805_2012Metric, symbol Device:R
- J1: footprint (none) -> Connector_PinSocket_2.54mm:PinSocket_1x10_P2.54mm_Vertical
- TH1, TH2: footprint (none) -> TerminalBlock_RND:TerminalBlock_RND_205-00012_1x02_P5.00mm_Horizontal
Connections:
- net +3V3: now also R7.1
- net GND: now also U6.60 (BOOT0)
- net reset: now reaches U6.7 (NRST)
- net reset: now also R7.2
Other:
- moved on the sheet: U6
Changed lines of the file:
@@
 F 0 "TH1" H 7247 1746 50  0000 L CNN
 F 1 "KTY81" H 7247 1655 50  0000 L CNN
-F 2 "" V 7350 1700 50  0001 C CNN
+F 2 "TerminalBlock_RND:TerminalBlock_RND_205-00012_1x02_P5.00mm_Horizontal" V 7350 1700 50  0001 C CNN
 F 3 "http://www.nxp.com/documents/data_sheet/KTY81_SER.pdf" H 7150 1650 50  0001 C CNN
 	1    7150 1700
@@
 F 0 "TH2" H 9198 1746 50  0000 L CNN
 F 1 "Thermistor_NTC" H 9198 1655 50  0000 L CNN
-F 2 "" H 9100 1750 50  0001 C CNN
+F 2 "TerminalBlock_RND:TerminalBlock_RND_205-00012_1x02_P5.00mm_Horizontal" H 9100 1750 50  0001 C CNN
 F 3 "~" H 9100 1750 50  0001 C CNN
 	1    9100 1700
@@
 L MCU_ST_STM32F4:STM32F405RGTx U6
 U 1 1 5DC72DB0
-P 1550 3900
-F 0 "U6" H 1850 2000 50  0000 C CNN
-F 1 "STM32F405RGTx" H 2100 2100 50  0000 C CNN
-F 2 "Package_QFP:LQFP-64_10x10mm_P0.5mm" H 950 2200 50  0001 R CNN
-F 3 "http://www.st.com/st-web-ui/static/active/en/resource/technical/document/datasheet/DM00037051.pdf" H 1550 3900 50  0001 C CNN
-	1    1550 3900
+P 1800 4100
+F 0 "U6" H 2100 2200 50  0000 C CNN
+F 1 "STM32F405RGTx" H 2350 2300 50  0000 C CNN
+F 2 "Package_QFP:LQFP-64_10x10mm_P0.5mm" H 1200 2400 50  0001 R CNN
+F 3 "http://www.st.com/st-web-ui/static/active/en/resource/technical/document/datasheet/DM00037051.pdf" H 1800 4100 50  0001 C CNN
+	1    1800 4100
 	1    0    0    -1
 $EndComp
@@
 $EndComp
 Wire Wire Line
-	1550 2000 1450 2000
-Wire Wire Line
-	1550 2000 1550 2100
-Connection ~ 1550 2000
-Wire Wire Line
-	1450 2000 1450 2100
-Wire Wire Line
-	1650 2100 1650 2000
-Wire Wire Line
-	1650 2000 1550 2000
-Wire Wire Line
-	1750 2100 1750 2000
-Wire Wire Line
-	1750 2000 1650 2000
-Connection ~ 1650 2000
-Wire Wire Line
-	1850 2100 1850 2000
-Wire Wire Line
-	1850 2000 1750 2000
-Connection ~ 1750 2000
+	1800 2200 1700 2200
+Wire Wire Line
+	1800 2200 1800 2300
+Connection ~ 1800 2200
+Wire Wire Line
+	1700 2200 1700 2300
+Wire Wire Line
+	1900 2300 1900 2200
+Wire Wire Line
+	1900 2200 1800 2200
+Wire Wire Line
+	2000 2300 2000 2200
+Wire Wire Line
+	2000 2200 1900 2200
+Connection ~ 1900 2200
+Wire Wire Line
+	2100 2300 2100 2200
+Wire Wire Line
+	2100 2200 2000 2200
+Connection ~ 2000 2200
 $Comp
 L power:GND #PWR027
 U 1 1 5DC7D7B5
-P 1550 5800
-F 0 "#PWR027" H 1550 5550 50  0001 C CNN
-F 1 "GND" H 1555 5627 50  0000 C CNN
-F 2 "" H 1550 5800 50  0001 C CNN
-F 3 "" H 1550 5800 50  0001 C CNN
-	1    1550 5800
-	1    0    0    -1
-$EndComp
-Wire Wire Line
-	1550 5800 1450 5800
-Wire Wire Line
-	1450 5800 1450 5700
-Wire Wire Line
-	1550 5700 1550 5800
-Connection ~ 1550 5800
-Wire Wire Line
-	1650 5700 1650 5800
-Wire Wire Line
-	1650 5800 1550 5800
+P 1800 6000
+F 0 "#PWR027" H 1800 5750 50  0001 C CNN
+F 1 "GND" H 1805 5827 50  0000 C CNN
+F 2 "" H 1800 6000 50  0001 C CNN
+F 3 "" H 1800 6000 50  0001 C CNN
+	1    1800 6000
+	1    0    0    -1
+$EndComp
+Wire Wire Line
+	1800 6000 1700 6000
+Wire Wire Line
+	1700 6000 1700 5900
+Wire Wire Line
+	1800 5900 1800 6000
+Connection ~ 1800 6000
+Wire Wire Line
+	1900 5900 1900 6000
+Wire Wire Line
+	1900 6000 1800 6000
 $Comp
 L Device:C C12
@@
 	1    0    0    -1
 $EndComp
-Text Label 850  2700 2    50   ~ 0
+Text Label 1100 2900 2    50   ~ 0
 VCAP_1
-Text Label 850  2800 2    50   ~ 0
+Text Label 1100 3000 2    50   ~ 0
 VCAP_2
 Text Label 850  1100 2    50   ~ 0
@@
 Text Notes 1700 1000 0    50   ~ 0
 ADC
-NoConn ~ 1350 2100
+NoConn ~ 1600 2300
 $Comp
 L Device:C C15
@@
 L power:+3V3 #PWR034
 U 1 1 5DCEBEA8
-P 1650 2000
-F 0 "#PWR034" H 1650 1850 50  0001 C CNN
-F 1 "+3V3" H 1665 2173 50  0000 C CNN
-F 2 "" H 1650 2000 50  0001 C CNN
-F 3 "" H 1650 2000 50  0001 C CNN
-	1    1650 2000
+P 1900 2200
+F 0 "#PWR034" H 1900 2050 50  0001 C CNN
+F 1 "+3V3" H 1915 2373 50  0000 C CNN
+F 2 "" H 1900 2200 50  0001 C CNN
+F 3 "" H 1900 2200 50  0001 C CNN
+	1    1900 2200
 	1    0    0    -1
 $EndComp
@@
 F 0 "J1" H 6028 6976 50  0000 L CNN
 F 1 "Conn_01x10_Female" H 6028 6885 50  0000 L CNN
-F 2 "" H 6000 7000 50  0001 C CNN
+F 2 "Connector_PinSocket_2.54mm:PinSocket_1x10_P2.54mm_Vertical" H 6000 7000 50  0001 C CNN
 F 3 "~" H 6000 7000 50  0001 C CNN
 	1    6000 7000
@@
 	5100 6700 5800 6700
 Connection ~ 5100 7000
+$Comp
+L power:GND #PWR041
+U 1 1 5DD53313
+P 700 2700
+F 0 "#PWR041" H 700 2450 50  0001 C CNN
+F 1 "GND" H 705 2527 50  0000 C CNN
+F 2 "" H 700 2700 50  0001 C CNN
+F 3 "" H 700 2700 50  0001 C CNN
+	1    700  2700
+	1    0    0    -1
+$EndComp
+Wire Wire Line
+	700  2700 1100 2700
+Text Label 950  2500 2    50   ~ 0
+reset
+$Comp
+L power:+3V3 #PWR040
+U 1 1 5DD5B29D
+P 1000 2050
+F 0 "#PWR040" H 1000 1900 50  0001 C CNN
+F 1 "+3V3" H 1015 2223 50  0000 C CNN
+F 2 "" H 1000 2050 50  0001 C CNN
+F 3 "" H 1000 2050 50  0001 C CNN
+	1    1000 2050
+	1    0    0    -1
+$EndComp
+$Comp
+L Device:R R7
+U 1 1 5DD5BE82
+P 1000 2250
+F 0 "R7" H 1070 2296 50  0000 L CNN
+F 1 "10k" H 1070 2205 50  0000 L CNN
+F 2 "Resistor_SMD:R_0805_2012Metric" V 930 2250 50  0001 C CNN
+F 3 "~" H 1000 2250 50  0001 C CNN
+	1    1000 2250
+	1    0    0    -1
+$EndComp
+Wire Wire Line
+	1000 2050 1000 2100
+Wire Wire Line
+	950  2500 1000 2500
+Wire Wire Line
+	1000 2400 1000 2500
+Connection ~ 1000 2500
+Wire Wire Line
+	1000 2500 1100 2500
 $EndSCHEMATC
