File: pcb/board/electric-FIAT.sch (KiCad schematic (older format))
At the start: 26 parts, among them J1 Conn_01x10_Female, U4 OPA356xxDBV, U5 OPA356xxDBV, U6 STM32F405RGTx

Commit message: Crystals
Parts:
- added C20, C21: 12p, Capacitor_SMD:C_0805_2012Metric, symbol Device:C
- added C22, C23: 30p, Capacitor_SMD:C_0805_2012Metric, symbol Device:C
- added Y1: 32.768MHz, Crystal:Crystal_SMD_3215-2Pin_3.2x1.5mm, symbol Device:Crystal
- added Y?: 25MHz, symbol Device:Crystal_GND24
Connections:
- net GND: now also C20.2, C21.2, C22.2, C23.2, Y?.2, Y?.4
- net SPI1_MOSI: now also U6.23 (PA7)
- net SPI1_SCK: now also U6.21 (PA5)
- new net: C20.1, Y1.1
- new net: C21.1, Y1.2
- new net: C22.1, Y?.1
- new net: C23.1, Y?.3
Other:
- note added: "Crystals"
Changed lines of the file:
@@
 Wire Wire Line
 	1000 2500 1100 2500
+Text Label 2500 3000 0    50   ~ 0
+SPI1_SCK
+Text Label 2500 3200 0    50   ~ 0
+SPI1_MOSI
+$Comp
+L Device:C C20
+U 1 1 5DC95CFF
+P 4800 1300
+F 0 "C20" H 4915 1346 50  0000 L CNN
+F 1 "12p" H 4915 1255 50  0000 L CNN
+F 2 "Capacitor_SMD:C_0805_2012Metric" H 4838 1150 50  0001 C CNN
+F 3 "~" H 4800 1300 50  0001 C CNN
+	1    4800 1300
+	1    0    0    -1
+$EndComp
+$Comp
+L Device:C C21
+U 1 1 5DC96103
+P 5200 1300
+F 0 "C21" H 5315 1346 50  0000 L CNN
+F 1 "12p" H 5315 1255 50  0000 L CNN
+F 2 "Capacitor_SMD:C_0805_2012Metric" H 5238 1150 50  0001 C CNN
+F 3 "~" H 5200 1300 50  0001 C CNN
+	1    5200 1300
+	1    0    0    -1
+$EndComp
+$Comp
+L Device:Crystal Y1
+U 1 1 5DC96831
+P 5000 1050
+F 0 "Y1" H 5000 1318 50  0000 C CNN
+F 1 "32.768MHz" H 5000 1227 50  0000 C CNN
+F 2 "Crystal:Crystal_SMD_3215-2Pin_3.2x1.5mm" H 5000 1050 50  0001 C CNN
+F 3 "~" H 5000 1050 50  0001 C CNN
+	1    5000 1050
+	1    0    0    -1
+$EndComp
+Wire Wire Line
+	4850 1050 4800 1050
+Wire Wire Line
+	4800 1050 4800 1150
+Wire Wire Line
+	5150 1050 5200 1050
+Wire Wire Line
+	5200 1050 5200 1150
+$Comp
+L power:GND #PWR042
+U 1 1 5DC9E145
+P 5000 1500
+F 0 "#PWR042" H 5000 1250 50  0001 C CNN
+F 1 "GND" H 5005 1327 50  0000 C CNN
+F 2 "" H 5000 1500 50  0001 C CNN
+F 3 "" H 5000 1500 50  0001 C CNN
+	1    5000 1500
+	1    0    0    -1
+$EndComp
+Wire Wire Line
+	5000 1500 4800 1500
+Wire Wire Line
+	4800 1500 4800 1450
+Wire Wire Line
+	5200 1450 5200 1500
+Wire Wire Line
+	5200 1500 5000 1500
+Connection ~ 5000 1500
+Text Notes 5250 700  0    100  ~ 20
+Crystals
+$Comp
+L Device:C C22
+U 1 1 5DCAD277
+P 5650 1300
+F 0 "C22" H 5765 1346 50  0000 L CNN
+F 1 "30p" H 5765 1255 50  0000 L CNN
+F 2 "Capacitor_SMD:C_0805_2012Metric" H 5688 1150 50  0001 C CNN
+F 3 "~" H 5650 1300 50  0001 C CNN
+	1    5650 1300
+	1    0    0    -1
+$EndComp
+$Comp
+L Device:C C23
+U 1 1 5DCAD27D
+P 6400 1300
+F 0 "C23" H 6515 1346 50  0000 L CNN
+F 1 "30p" H 6515 1255 50  0000 L CNN
+F 2 "Capacitor_SMD:C_0805_2012Metric" H 6438 1150 50  0001 C CNN
+F 3 "~" H 6400 1300 50  0001 C CNN
+	1    6400 1300
+	1    0    0    -1
+$EndComp
+Wire Wire Line
+	5900 1050 5650 1050
+Wire Wire Line
+	5650 1050 5650 1150
+Wire Wire Line
+	6200 1050 6400 1050
+Wire Wire Line
+	6400 1050 6400 1150
+$Comp
+L power:GND #PWR043
+U 1 1 5DCAD28D
+P 6000 1500
+F 0 "#PWR043" H 6000 1250 50  0001 C CNN
+F 1 "GND" H 6005 1327 50  0000 C CNN
+F 2 "" H 6000 1500 50  0001 C CNN
+F 3 "" H 6000 1500 50  0001 C CNN
+	1    6000 1500
+	1    0    0    -1
+$EndComp
+Wire Wire Line
+	6000 1500 5650 1500
+Wire Wire Line
+	5650 1500 5650 1450
+Wire Wire Line
+	6400 1450 6400 1500
+Wire Wire Line
+	6400 1500 6000 1500
+Connection ~ 6000 1500
+$Comp
+L Device:Crystal_GND24 Y?
+U 1 1 5DCB2832
+P 6050 1050
+F 0 "Y?" H 6250 1200 50  0000 L CNN
+F 1 "25MHz" H 6250 1100 50  0000 L CNN
+F 2 "" H 6050 1050 50  0001 C CNN
+F 3 "~" H 6050 1050 50  0001 C CNN
+	1    6050 1050
+	1    0    0    -1
+$EndComp
+$Comp
+L power:GND #PWR?
+U 1 1 5DCCBCED
+P 6050 1250
+F 0 "#PWR?" H 6050 1000 50  0001 C CNN
+F 1 "GND" H 6055 1077 50  0000 C CNN
+F 2 "" H 6050 1250 50  0001 C CNN
+F 3 "" H 6050 1250 50  0001 C CNN
+	1    6050 1250
+	1    0    0    -1
+$EndComp
+$Comp
+L power:GND #PWR?
+U 1 1 5DCCC2B5
+P 6200 600
+F 0 "#PWR?" H 6200 350 50  0001 C CNN
+F 1 "GND" H 6205 427 50  0000 C CNN
+F 2 "" H 6200 600 50  0001 C CNN
+F 3 "" H 6200 600 50  0001 C CNN
+	1    6200 600
+	1    0    0    -1
+$EndComp
+Wire Wire Line
+	6050 850  6050 600
+Wire Wire Line
+	6050 600  6200 600
 $EndSCHEMATC
