File: pcb/board/electric-FIAT.sch (KiCad schematic (older format))
At the start: 32 parts, among them J1 Conn_01x10_Female, U4 OPA356xxDBV, U5 OPA356xxDBV, U6 STM32F405RGTx, Y1 32.768MHz, Y2 25MHz

Commit message: Current Sensors connected to MCU
Connections:
- net Current_PH1: now reaches U6.14 (PA0)
- net Current_PH2: now reaches U6.15 (PA1)
- net Current_PH3: now reaches U6.16 (PA2)
Changed lines of the file:
@@
 	1    0    0    -1
 $EndComp
+Text Label 10450 3950 0    50   ~ 0
+Current_PH1
+Text Label 10450 4550 0    50   ~ 0
+Current_PH2
+Text Label 10450 5150 0    50   ~ 0
+Current_PH3
+Text Label 2500 2500 0    50   ~ 0
+Current_PH1
+Text Label 2500 2600 0    50   ~ 0
+Current_PH2
+Text Label 2500 2700 0    50   ~ 0
+Current_PH3
 $EndSCHEMATC
