File: pcb/board/current_sensor.sch (KiCad schematic (older format))
At the start: 3 parts, among them U1 ACS773ECB-200B-PFF

Commit message: MCU and Decoupling
Changed lines of the file:
@@
 EESchema Schematic File Version 4
+LIBS:electric-FIAT-cache
 EELAYER 30 0
 EELAYER END
 $Descr A4 11693 8268
 encoding utf-8
-Sheet 2 4
+Sheet 4 4
 Title ""
 Date ""
@@
 F 3 "https://www.allegromicro.com/-/media/Files/Datasheets/ACS773-Datasheet.ashx" H 5600 3950 50  0001 C CNN
 	1    5600 3950
-	1    0    0    -1
-$EndComp
-$Comp
-L power:+3.3V #PWR?
-U 1 1 5DC6FAA0
-P 5600 3600
-AR Path="/5DC7202D/5DC6FAA0" Ref="#PWR?"  Part="1"
-AR Path="/5DC75544/5DC6FAA0" Ref="#PWR?"  Part="1"
-AR Path="/5DC755EE/5DC6FAA0" Ref="#PWR?"  Part="1"
-AR Path="/5DC773B5/5DC6FAA0" Ref="#PWR01"  Part="1"
-AR Path="/5DC77C5E/5DC6FAA0" Ref="#PWR06"  Part="1"
-AR Path="/5DC77D5C/5DC6FAA0" Ref="#PWR011"  Part="1"
-F 0 "#PWR011" H 5600 3450 50  0001 C CNN
-F 1 "+3.3V" H 5615 3773 50  0000 C CNN
-F 2 "" H 5600 3600 50  0001 C CNN
-F 3 "" H 5600 3600 50  0001 C CNN
-	1    5600 3600
 	1    0    0    -1
 $EndComp
@@
 Text HLabel 6100 3950 2    50   Output ~ 0
 out
+$Comp
+L power:+3V3 #PWR035
+U 1 1 5DCEB1D3
+P 5600 3600
+AR Path="/5DC773B5/5DCEB1D3" Ref="#PWR035"  Part="1"
+AR Path="/5DC77C5E/5DCEB1D3" Ref="#PWR036"  Part="1"
+AR Path="/5DC77D5C/5DCEB1D3" Ref="#PWR037"  Part="1"
+F 0 "#PWR037" H 5600 3450 50  0001 C CNN
+F 1 "+3V3" H 5615 3773 50  0000 C CNN
+F 2 "" H 5600 3600 50  0001 C CNN
+F 3 "" H 5600 3600 50  0001 C CNN
+	1    5600 3600
+	1    0    0    -1
+$EndComp
 $EndSCHEMATC

Commit message: Initialized STM32F405RGTx
Other:
- moved on the sheet: C1, C2, U1
Changed lines of the file:
@@
 $Descr A4 11693 8268
 encoding utf-8
-Sheet 4 4
+Sheet 2 4
 Title ""
 Date ""
@@
 L fiat:ACS773ECB-200B-PFF U?
 U 1 1 5DC6FA9A
-P 5600 3950
+P 6250 4000
 AR Path="/5DC7202D/5DC6FA9A" Ref="U?"  Part="1"
 AR Path="/5DC75544/5DC6FA9A" Ref="U?"  Part="1"
@@
 AR Path="/5DC77C5E/5DC6FA9A" Ref="U2"  Part="1"
 AR Path="/5DC77D5C/5DC6FA9A" Ref="U3"  Part="1"
-F 0 "U3" H 5750 4350 50  0000 L CNN
-F 1 "ACS773ECB-200B-PFF" H 5750 4250 50  0000 L CNN
-F 2 "Sensor_Current:Allegro_CB_PFF" H 5600 3950 50  0001 C CNN
-F 3 "https://www.allegromicro.com/-/media/Files/Datasheets/ACS773-Datasheet.ashx" H 5600 3950 50  0001 C CNN
-	1    5600 3950
+F 0 "U1" H 6400 4400 50  0000 L CNN
+F 1 "ACS773ECB-200B-PFF" H 6400 4300 50  0000 L CNN
+F 2 "Sensor_Current:Allegro_CB_PFF" H 6250 4000 50  0001 C CNN
+F 3 "https://www.allegromicro.com/-/media/Files/Datasheets/ACS773-Datasheet.ashx" H 6250 4000 50  0001 C CNN
+	1    6250 4000
 	1    0    0    -1
 $EndComp
 Wire Wire Line
-	5600 3600 5600 3650
+	6250 3650 6250 3700
 $Comp
 L power:GND #PWR?
 U 1 1 5DC6FAA7
-P 5600 4300
+P 6250 4350
 AR Path="/5DC7202D/5DC6FAA7" Ref="#PWR?"  Part="1"
 AR Path="/5DC75544/5DC6FAA7" Ref="#PWR?"  Part="1"
@@
 AR Path="/5DC77C5E/5DC6FAA7" Ref="#PWR09"  Part="1"
 AR Path="/5DC77D5C/5DC6FAA7" Ref="#PWR014"  Part="1"
-F 0 "#PWR014" H 5600 4050 50  0001 C CNN
-F 1 "GND" H 5605 4127 50  0000 C CNN
-F 2 "" H 5600 4300 50  0001 C CNN
-F 3 "" H 5600 4300 50  0001 C CNN
-	1    5600 4300
+F 0 "#PWR014" H 6250 4100 50  0001 C CNN
+F 1 "GND" H 6255 4177 50  0000 C CNN
+F 2 "" H 6250 4350 50  0001 C CNN
+F 3 "" H 6250 4350 50  0001 C CNN
+	1    6250 4350
 	1    0    0    -1
 $EndComp
 Wire Wire Line
-	5600 4300 5600 4250
-Text HLabel 5200 3850 0    50   Input ~ 0
+	6250 4350 6250 4300
+Text HLabel 5850 3900 0    50   Input ~ 0
 IGBT_PH1
-Text HLabel 5200 4050 0    50   Output ~ 0
+Text HLabel 5850 4100 0    50   Output ~ 0
 Motor_PH1
-Text Notes 3450 3500 0    100  ~ 20
+Text Notes 4100 3550 0    100  ~ 20
 Decoupling
 $Comp
 L Device:C C?
 U 1 1 5DC71A7F
-P 3850 4050
+P 4500 4100
 AR Path="/5DC7202D/5DC71A7F" Ref="C?"  Part="1"
 AR Path="/5DC75544/5DC71A7F" Ref="C?"  Part="1"
@@
 AR Path="/5DC77C5E/5DC71A7F" Ref="C3"  Part="1"
 AR Path="/5DC77D5C/5DC71A7F" Ref="C5"  Part="1"
-F 0 "C5" H 3965 4096 50  0000 L CNN
-F 1 "100n" H 3965 4005 50  0000 L CNN
-F 2 "Capacitor_SMD:C_0805_2012Metric" H 3888 3900 50  0001 C CNN
-F 3 "~" H 3850 4050 50  0001 C CNN
-	1    3850 4050
+F 0 "C1" H 4615 4146 50  0000 L CNN
+F 1 "100n" H 4615 4055 50  0000 L CNN
+F 2 "Capacitor_SMD:C_0805_2012Metric" H 4538 3950 50  0001 C CNN
+F 3 "~" H 4500 4100 50  0001 C CNN
+	1    4500 4100
 	1    0    0    -1
 $EndComp
@@
 L power:+3.3V #PWR?
 U 1 1 5DC71F2C
-P 3850 3850
+P 4500 3900
 AR Path="/5DC7202D/5DC71F2C" Ref="#PWR?"  Part="1"
 AR Path="/5DC75544/5DC71F2C" Ref="#PWR?"  Part="1"
@@
 AR Path="/5DC77C5E/5DC71F2C" Ref="#PWR07"  Part="1"
 AR Path="/5DC77D5C/5DC71F2C" Ref="#PWR012"  Part="1"
-F 0 "#PWR012" H 3850 3700 50  0001 C CNN
-F 1 "+3.3V" H 3865 4023 50  0000 C CNN
-F 2 "" H 3850 3850 50  0001 C CNN
-F 3 "" H 3850 3850 50  0001 C CNN
-	1    3850 3850
+F 0 "#PWR012" H 4500 3750 50  0001 C CNN
+F 1 "+3.3V" H 4515 4073 50  0000 C CNN
+F 2 "" H 4500 3900 50  0001 C CNN
+F 3 "" H 4500 3900 50  0001 C CNN
+	1    4500 3900
 	1    0    0    -1
 $EndComp
 Wire Wire Line
-	3850 3850 3850 3900
+	4500 3900 4500 3950
 $Comp
 L power:GND #PWR?
 U 1 1 5DC7230E
-P 3850 4250
+P 4500 4300
 AR Path="/5DC7202D/5DC7230E" Ref="#PWR?"  Part="1"
 AR Path="/5DC75544/5DC7230E" Ref="#PWR?"  Part="1"
@@
 AR Path="/5DC77C5E/5DC7230E" Ref="#PWR08"  Part="1"
 AR Path="/5DC77D5C/5DC7230E" Ref="#PWR013"  Part="1"
-F 0 "#PWR013" H 3850 4000 50  0001 C CNN
-F 1 "GND" H 3855 4077 50  0000 C CNN
-F 2 "" H 3850 4250 50  0001 C CNN
-F 3 "" H 3850 4250 50  0001 C CNN
-	1    3850 4250
+F 0 "#PWR013" H 4500 4050 50  0001 C CNN
+F 1 "GND" H 4505 4127 50  0000 C CNN
+F 2 "" H 4500 4300 50  0001 C CNN
+F 3 "" H 4500 4300 50  0001 C CNN
+	1    4500 4300
 	1    0    0    -1
 $EndComp
 Wire Wire Line
-	3850 4250 3850 4200
+	4500 4300 4500 4250
 $Comp
 L Device:C C?
 U 1 1 5DC730E7
-P 6100 4150
+P 6750 4200
 AR Path="/5DC7202D/5DC730E7" Ref="C?"  Part="1"
 AR Path="/5DC75544/5DC730E7" Ref="C?"  Part="1"
@@
 AR Path="/5DC77C5E/5DC730E7" Ref="C4"  Part="1"
 AR Path="/5DC77D5C/5DC730E7" Ref="C6"  Part="1"
-F 0 "C6" H 6215 4196 50  0000 L CNN
-F 1 "1n" H 6215 4105 50  0000 L CNN
-F 2 "Capacitor_SMD:C_0805_2012Metric" H 6138 4000 50  0001 C CNN
-F 3 "~" H 6100 4150 50  0001 C CNN
-	1    6100 4150
+F 0 "C2" H 6865 4246 50  0000 L CNN
+F 1 "1n" H 6865 4155 50  0000 L CNN
+F 2 "Capacitor_SMD:C_0805_2012Metric" H 6788 4050 50  0001 C CNN
+F 3 "~" H 6750 4200 50  0001 C CNN
+	1    6750 4200
 	1    0    0    -1
 $EndComp
@@
 L power:GND #PWR?
 U 1 1 5DC7443D
-P 6100 4350
+P 6750 4400
 AR Path="/5DC7202D/5DC7443D" Ref="#PWR?"  Part="1"
 AR Path="/5DC75544/5DC7443D" Ref="#PWR?"  Part="1"
@@
 AR Path="/5DC77C5E/5DC7443D" Ref="#PWR010"  Part="1"
 AR Path="/5DC77D5C/5DC7443D" Ref="#PWR015"  Part="1"
-F 0 "#PWR015" H 6100 4100 50  0001 C CNN
-F 1 "GND" H 6105 4177 50  0000 C CNN
-F 2 "" H 6100 4350 50  0001 C CNN
-F 3 "" H 6100 4350 50  0001 C CNN
-	1    6100 4350
+F 0 "#PWR015" H 6750 4150 50  0001 C CNN
+F 1 "GND" H 6755 4227 50  0000 C CNN
+F 2 "" H 6750 4400 50  0001 C CNN
+F 3 "" H 6750 4400 50  0001 C CNN
+	1    6750 4400
 	1    0    0    -1
 $EndComp
 Wire Wire Line
-	6100 4350 6100 4300
+	6750 4400 6750 4350
 Wire Wire Line
-	6100 4000 6100 3950
+	6750 4050 6750 4000
 Wire Wire Line
-	6100 3950 6000 3950
-Text HLabel 6100 3950 2    50   Output ~ 0
+	6750 4000 6650 4000
+Text HLabel 6750 4000 2    50   Output ~ 0
 out
 $Comp
 L power:+3V3 #PWR035
 U 1 1 5DCEB1D3
-P 5600 3600
+P 6250 3650
 AR Path="/5DC773B5/5DCEB1D3" Ref="#PWR035"  Part="1"
 AR Path="/5DC77C5E/5DCEB1D3" Ref="#PWR036"  Part="1"
 AR Path="/5DC77D5C/5DCEB1D3" Ref="#PWR037"  Part="1"
-F 0 "#PWR037" H 5600 3450 50  0001 C CNN
-F 1 "+3V3" H 5615 3773 50  0000 C CNN
-F 2 "" H 5600 3600 50  0001 C CNN
-F 3 "" H 5600 3600 50  0001 C CNN
-	1    5600 3600
+F 0 "#PWR037" H 6250 3500 50  0001 C CNN
+F 1 "+3V3" H 6265 3823 50  0000 C CNN
+F 2 "" H 6250 3650 50  0001 C CNN
+F 3 "" H 6250 3650 50  0001 C CNN
+	1    6250 3650
 	1    0    0    -1
 $EndComp
