File: hardware/motor_controller/ac_sensor.sch (KiCad schematic (older format))
At the start: 13 parts

Commit message: Anotation
Parts:
- gave numbers to parts that had none: 13
