File: hardware/motor_controller/ac_sensor.sch (KiCad schematic (older format))
At the start: 13 parts, among them U15 ACPL-C87A, U16 OPA356xxDBV

Commit message: SD Card and other pins
Parts:
- renumbered C39 to C59, C40 to C60, C41 to C61, C42 to C62, C43 to C63, R27 to R34, R28 to R35, R29 to R36, R30 to R37, R31 to R38, R32 to R39, U15 to U17, U16 to U18

Commit message: Voltage Sensors corrected
Parts:
- removed R35: 75k, symbol Device:R
- added R? (x9): 200k, symbol Device:R
Connections:
- net +3V3: no longer C61.1, U17.1 (VDD1)
- net ac_phase: now also R?.1
- net at C60.1, R37.1, U17.2 (IN): now also R?.2
- new net: R?.2, R?.2 (x4)
- new net: R?.1, R?.1 (x4)
- new net +5V: C61.1, U17.1 (VDD1)
Other:
- moved on the sheet: C49, C50, C51, C52, C53, R22, R24, R25, R26, R27, U13, U14
