File: hardware/motor_controller/current_sensor.sch (KiCad schematic (older format))
At the start: 3 parts, among them U1 ACS773ECB-200B-PFF

Commit message: FOC controller, CAN and IGBTs
Parts:
- removed U1: ACS773ECB-200B-PFF, Sensor_Current:Allegro_CB_PFF, symbol fiat:ACS773ECB-200B-PFF
- added U2: ACS759xCB-200B-PFF, Sensor_Current:Allegro_CB_PFF, symbol Sensor_Current:ACS759xCB-200B-PFF
Changed lines of the file:
@@
 Comment4 ""
 $EndDescr
-$Comp
-L fiat:ACS773ECB-200B-PFF U?
-U 1 1 5DC6FA9A
-P 6250 4000
-AR Path="/5DC7202D/5DC6FA9A" Ref="U?"  Part="1"
-AR Path="/5DC75544/5DC6FA9A" Ref="U?"  Part="1"
-AR Path="/5DC755EE/5DC6FA9A" Ref="U?"  Part="1"
-AR Path="/5DC773B5/5DC6FA9A" Ref="U1"  Part="1"
-AR Path="/5DC77C5E/5DC6FA9A" Ref="U2"  Part="1"
-AR Path="/5DC77D5C/5DC6FA9A" Ref="U3"  Part="1"
-F 0 "U1" H 6400 4400 50  0000 L CNN
-F 1 "ACS773ECB-200B-PFF" H 6400 4300 50  0000 L CNN
-F 2 "Sensor_Current:Allegro_CB_PFF" H 6250 4000 50  0001 C CNN
-F 3 "https://www.allegromicro.com/-/media/Files/Datasheets/ACS773-Datasheet.ashx" H 6250 4000 50  0001 C CNN
-	1    6250 4000
-	1    0    0    -1
-$EndComp
 Wire Wire Line
 	6250 3650 6250 3700
@@
 AR Path="/5DC77C5E/5DC6FAA7" Ref="#PWR09"  Part="1"
 AR Path="/5DC77D5C/5DC6FAA7" Ref="#PWR014"  Part="1"
-F 0 "#PWR014" H 6250 4100 50  0001 C CNN
+F 0 "#PWR04" H 6250 4100 50  0001 C CNN
 F 1 "GND" H 6255 4177 50  0000 C CNN
 F 2 "" H 6250 4350 50  0001 C CNN
@@
 AR Path="/5DC77C5E/5DC71F2C" Ref="#PWR07"  Part="1"
 AR Path="/5DC77D5C/5DC71F2C" Ref="#PWR012"  Part="1"
-F 0 "#PWR012" H 4500 3750 50  0001 C CNN
+F 0 "#PWR02" H 4500 3750 50  0001 C CNN
 F 1 "+3.3V" H 4515 4073 50  0000 C CNN
 F 2 "" H 4500 3900 50  0001 C CNN
@@
 AR Path="/5DC77C5E/5DC7230E" Ref="#PWR08"  Part="1"
 AR Path="/5DC77D5C/5DC7230E" Ref="#PWR013"  Part="1"
-F 0 "#PWR013" H 4500 4050 50  0001 C CNN
+F 0 "#PWR03" H 4500 4050 50  0001 C CNN
 F 1 "GND" H 4505 4127 50  0000 C CNN
 F 2 "" H 4500 4300 50  0001 C CNN
@@
 AR Path="/5DC77C5E/5DC7443D" Ref="#PWR010"  Part="1"
 AR Path="/5DC77D5C/5DC7443D" Ref="#PWR015"  Part="1"
-F 0 "#PWR015" H 6750 4150 50  0001 C CNN
+F 0 "#PWR05" H 6750 4150 50  0001 C CNN
 F 1 "GND" H 6755 4227 50  0000 C CNN
 F 2 "" H 6750 4400 50  0001 C CNN
@@
 AR Path="/5DC77C5E/5DCEB1D3" Ref="#PWR036"  Part="1"
 AR Path="/5DC77D5C/5DCEB1D3" Ref="#PWR037"  Part="1"
-F 0 "#PWR037" H 6250 3500 50  0001 C CNN
+F 0 "#PWR035" H 6250 3500 50  0001 C CNN
 F 1 "+3V3" H 6265 3823 50  0000 C CNN
 F 2 "" H 6250 3650 50  0001 C CNN
@@
 	1    0    0    -1
 $EndComp
+$Comp
+L Sensor_Current:ACS759xCB-200B-PFF U2
+U 1 1 5DCAFD9E
+P 6250 4000
+AR Path="/5DC773B5/5DCAFD9E" Ref="U2"  Part="1"
+AR Path="/5DC77C5E/5DCAFD9E" Ref="U3"  Part="1"
+AR Path="/5DC77D5C/5DCAFD9E" Ref="U7"  Part="1"
+F 0 "U2" H 6350 4350 50  0000 L CNN
+F 1 "ACS759xCB-200B-PFF" H 6350 4250 50  0000 L CNN
+F 2 "Sensor_Current:Allegro_CB_PFF" H 6250 4000 50  0001 C CNN
+F 3 "http://www.allegromicro.com/~/media/Files/Datasheets/ACS759-Datasheet.ashx?la=en" H 6250 4000 50  0001 C CNN
+	1    6250 4000
+	1    0    0    -1
+$EndComp

Commit message: Anotation
Changed lines of the file:
@@
 AR Path="/5DC77C5E/5DC6FAA7" Ref="#PWR09"  Part="1"
 AR Path="/5DC77D5C/5DC6FAA7" Ref="#PWR014"  Part="1"
-F 0 "#PWR04" H 6250 4100 50  0001 C CNN
+F 0 "#PWR014" H 6250 4100 50  0001 C CNN
 F 1 "GND" H 6255 4177 50  0000 C CNN
 F 2 "" H 6250 4350 50  0001 C CNN
@@
 AR Path="/5DC77C5E/5DC71A7F" Ref="C3"  Part="1"
 AR Path="/5DC77D5C/5DC71A7F" Ref="C5"  Part="1"
-F 0 "C1" H 4615 4146 50  0000 L CNN
+F 0 "C5" H 4615 4146 50  0000 L CNN
 F 1 "100n" H 4615 4055 50  0000 L CNN
 F 2 "Capacitor_SMD:C_0805_2012Metric" H 4538 3950 50  0001 C CNN
@@
 AR Path="/5DC77C5E/5DC71F2C" Ref="#PWR07"  Part="1"
 AR Path="/5DC77D5C/5DC71F2C" Ref="#PWR012"  Part="1"
-F 0 "#PWR02" H 4500 3750 50  0001 C CNN
+F 0 "#PWR012" H 4500 3750 50  0001 C CNN
 F 1 "+3.3V" H 4515 4073 50  0000 C CNN
 F 2 "" H 4500 3900 50  0001 C CNN
@@
 AR Path="/5DC77C5E/5DC7230E" Ref="#PWR08"  Part="1"
 AR Path="/5DC77D5C/5DC7230E" Ref="#PWR013"  Part="1"
-F 0 "#PWR03" H 4500 4050 50  0001 C CNN
+F 0 "#PWR013" H 4500 4050 50  0001 C CNN
 F 1 "GND" H 4505 4127 50  0000 C CNN
 F 2 "" H 4500 4300 50  0001 C CNN
@@
 AR Path="/5DC77C5E/5DC730E7" Ref="C4"  Part="1"
 AR Path="/5DC77D5C/5DC730E7" Ref="C6"  Part="1"
-F 0 "C2" H 6865 4246 50  0000 L CNN
+F 0 "C6" H 6865 4246 50  0000 L CNN
 F 1 "1n" H 6865 4155 50  0000 L CNN
 F 2 "Capacitor_SMD:C_0805_2012Metric" H 6788 4050 50  0001 C CNN
@@
 AR Path="/5DC77C5E/5DC7443D" Ref="#PWR010"  Part="1"
 AR Path="/5DC77D5C/5DC7443D" Ref="#PWR015"  Part="1"
-F 0 "#PWR05" H 6750 4150 50  0001 C CNN
+F 0 "#PWR015" H 6750 4150 50  0001 C CNN
 F 1 "GND" H 6755 4227 50  0000 C CNN
 F 2 "" H 6750 4400 50  0001 C CNN
@@
 AR Path="/5DC77C5E/5DCEB1D3" Ref="#PWR036"  Part="1"
 AR Path="/5DC77D5C/5DCEB1D3" Ref="#PWR037"  Part="1"
-F 0 "#PWR035" H 6250 3500 50  0001 C CNN
+F 0 "#PWR037" H 6250 3500 50  0001 C CNN
 F 1 "+3V3" H 6265 3823 50  0000 C CNN
 F 2 "" H 6250 3650 50  0001 C CNN
@@
 AR Path="/5DC77C5E/5DCAFD9E" Ref="U3"  Part="1"
 AR Path="/5DC77D5C/5DCAFD9E" Ref="U7"  Part="1"
-F 0 "U2" H 6350 4350 50  0000 L CNN
+F 0 "U7" H 6350 4350 50  0000 L CNN
 F 1 "ACS759xCB-200B-PFF" H 6350 4250 50  0000 L CNN
 F 2 "Sensor_Current:Allegro_CB_PFF" H 6250 4000 50  0001 C CNN

Commit message: DC/DC converters added
Parts:
- added R33: 4.7k, symbol Device:R
Connections:
- net out: now also R33.1; no longer U2.3 (VIOUT)
- new net: R33.2, U2.3 (VIOUT)
Other:
- moved on the sheet: C2
Changed lines of the file:
@@
 EESchema Schematic File Version 4
+LIBS:electric-FIAT-cache
 EELAYER 30 0
 EELAYER END
@@
 AR Path="/5DC77C5E/5DC6FAA7" Ref="#PWR09"  Part="1"
 AR Path="/5DC77D5C/5DC6FAA7" Ref="#PWR014"  Part="1"
-F 0 "#PWR014" H 6250 4100 50  0001 C CNN
+F 0 "#PWR04" H 6250 4100 50  0001 C CNN
 F 1 "GND" H 6255 4177 50  0000 C CNN
 F 2 "" H 6250 4350 50  0001 C CNN
@@
 AR Path="/5DC77C5E/5DC71A7F" Ref="C3"  Part="1"
 AR Path="/5DC77D5C/5DC71A7F" Ref="C5"  Part="1"
-F 0 "C5" H 4615 4146 50  0000 L CNN
+F 0 "C1" H 4615 4146 50  0000 L CNN
 F 1 "100n" H 4615 4055 50  0000 L CNN
 F 2 "Capacitor_SMD:C_0805_2012Metric" H 4538 3950 50  0001 C CNN
@@
 AR Path="/5DC77C5E/5DC71F2C" Ref="#PWR07"  Part="1"
 AR Path="/5DC77D5C/5DC71F2C" Ref="#PWR012"  Part="1"
-F 0 "#PWR012" H 4500 3750 50  0001 C CNN
+F 0 "#PWR02" H 4500 3750 50  0001 C CNN
 F 1 "+3.3V" H 4515 4073 50  0000 C CNN
 F 2 "" H 4500 3900 50  0001 C CNN
@@
 AR Path="/5DC77C5E/5DC7230E" Ref="#PWR08"  Part="1"
 AR Path="/5DC77D5C/5DC7230E" Ref="#PWR013"  Part="1"
-F 0 "#PWR013" H 4500 4050 50  0001 C CNN
+F 0 "#PWR03" H 4500 4050 50  0001 C CNN
 F 1 "GND" H 4505 4127 50  0000 C CNN
 F 2 "" H 4500 4300 50  0001 C CNN
@@
 L Device:C C?
 U 1 1 5DC730E7
-P 6750 4200
+P 7100 4200
 AR Path="/5DC7202D/5DC730E7" Ref="C?"  Part="1"
 AR Path="/5DC75544/5DC730E7" Ref="C?"  Part="1"
@@
 AR Path="/5DC77C5E/5DC730E7" Ref="C4"  Part="1"
 AR Path="/5DC77D5C/5DC730E7" Ref="C6"  Part="1"
-F 0 "C6" H 6865 4246 50  0000 L CNN
-F 1 "1n" H 6865 4155 50  0000 L CNN
-F 2 "Capacitor_SMD:C_0805_2012Metric" H 6788 4050 50  0001 C CNN
-F 3 "~" H 6750 4200 50  0001 C CNN
-	1    6750 4200
+F 0 "C2" H 7215 4246 50  0000 L CNN
+F 1 "1n" H 7215 4155 50  0000 L CNN
+F 2 "Capacitor_SMD:C_0805_2012Metric" H 7138 4050 50  0001 C CNN
+F 3 "~" H 7100 4200 50  0001 C CNN
+	1    7100 4200
 	1    0    0    -1
 $EndComp
@@
 L power:GND #PWR?
 U 1 1 5DC7443D
-P 6750 4400
+P 7100 4400
 AR Path="/5DC7202D/5DC7443D" Ref="#PWR?"  Part="1"
 AR Path="/5DC75544/5DC7443D" Ref="#PWR?"  Part="1"
@@
 AR Path="/5DC77C5E/5DC7443D" Ref="#PWR010"  Part="1"
 AR Path="/5DC77D5C/5DC7443D" Ref="#PWR015"  Part="1"
-F 0 "#PWR015" H 6750 4150 50  0001 C CNN
-F 1 "GND" H 6755 4227 50  0000 C CNN
-F 2 "" H 6750 4400 50  0001 C CNN
-F 3 "" H 6750 4400 50  0001 C CNN
-	1    6750 4400
+F 0 "#PWR05" H 7100 4150 50  0001 C CNN
+F 1 "GND" H 7105 4227 50  0000 C CNN
+F 2 "" H 7100 4400 50  0001 C CNN
+F 3 "" H 7100 4400 50  0001 C CNN
+	1    7100 4400
 	1    0    0    -1
 $EndComp
 Wire Wire Line
-	6750 4400 6750 4350
+	7100 4400 7100 4350
 Wire Wire Line
-	6750 4050 6750 4000
+	7100 4050 7100 4000
 Wire Wire Line
-	6750 4000 6650 4000
-Text HLabel 6750 4000 2    50   Output ~ 0
+	7100 4000 7000 4000
+Text HLabel 7100 4000 2    50   Output ~ 0
 out
 $Comp
@@
 AR Path="/5DC77C5E/5DCEB1D3" Ref="#PWR036"  Part="1"
 AR Path="/5DC77D5C/5DCEB1D3" Ref="#PWR037"  Part="1"
-F 0 "#PWR037" H 6250 3500 50  0001 C CNN
+F 0 "#PWR035" H 6250 3500 50  0001 C CNN
 F 1 "+3V3" H 6265 3823 50  0000 C CNN
 F 2 "" H 6250 3650 50  0001 C CNN
@@
 AR Path="/5DC77C5E/5DCAFD9E" Ref="U3"  Part="1"
 AR Path="/5DC77D5C/5DCAFD9E" Ref="U7"  Part="1"
-F 0 "U7" H 6350 4350 50  0000 L CNN
+F 0 "U2" H 6350 4350 50  0000 L CNN
 F 1 "ACS759xCB-200B-PFF" H 6350 4250 50  0000 L CNN
 F 2 "Sensor_Current:Allegro_CB_PFF" H 6250 4000 50  0001 C CNN
@@
 	1    0    0    -1
 $EndComp
+$Comp
+L Device:R R33
+U 1 1 5DE77132
+P 6850 4000
+AR Path="/5DC773B5/5DE77132" Ref="R33"  Part="1"
+AR Path="/5DC77C5E/5DE77132" Ref="R34"  Part="1"
+AR Path="/5DC77D5C/5DE77132" Ref="R35"  Part="1"
+F 0 "R33" V 6643 4000 50  0000 C CNN
+F 1 "4.7k" V 6734 4000 50  0000 C CNN
+F 2 "" V 6780 4000 50  0001 C CNN
+F 3 "~" H 6850 4000 50  0001 C CNN
+	1    6850 4000
+	0    1    1    0
+$EndComp
+Wire Wire Line
+	6650 4000 6700 4000
 $EndSCHEMATC

Commit message: DC/DC converters updated
Changed lines of the file:
@@
 AR Path="/5DC77C5E/5DC6FAA7" Ref="#PWR09"  Part="1"
 AR Path="/5DC77D5C/5DC6FAA7" Ref="#PWR014"  Part="1"
-F 0 "#PWR04" H 6250 4100 50  0001 C CNN
+F 0 "#PWR014" H 6250 4100 50  0001 C CNN
 F 1 "GND" H 6255 4177 50  0000 C CNN
 F 2 "" H 6250 4350 50  0001 C CNN
@@
 AR Path="/5DC77C5E/5DC71A7F" Ref="C3"  Part="1"
 AR Path="/5DC77D5C/5DC71A7F" Ref="C5"  Part="1"
-F 0 "C1" H 4615 4146 50  0000 L CNN
+F 0 "C5" H 4615 4146 50  0000 L CNN
 F 1 "100n" H 4615 4055 50  0000 L CNN
 F 2 "Capacitor_SMD:C_0805_2012Metric" H 4538 3950 50  0001 C CNN
@@
 AR Path="/5DC77C5E/5DC71F2C" Ref="#PWR07"  Part="1"
 AR Path="/5DC77D5C/5DC71F2C" Ref="#PWR012"  Part="1"
-F 0 "#PWR02" H 4500 3750 50  0001 C CNN
+F 0 "#PWR012" H 4500 3750 50  0001 C CNN
 F 1 "+3.3V" H 4515 4073 50  0000 C CNN
 F 2 "" H 4500 3900 50  0001 C CNN
@@
 AR Path="/5DC77C5E/5DC7230E" Ref="#PWR08"  Part="1"
 AR Path="/5DC77D5C/5DC7230E" Ref="#PWR013"  Part="1"
-F 0 "#PWR03" H 4500 4050 50  0001 C CNN
+F 0 "#PWR013" H 4500 4050 50  0001 C CNN
 F 1 "GND" H 4505 4127 50  0000 C CNN
 F 2 "" H 4500 4300 50  0001 C CNN
@@
 AR Path="/5DC77C5E/5DC730E7" Ref="C4"  Part="1"
 AR Path="/5DC77D5C/5DC730E7" Ref="C6"  Part="1"
-F 0 "C2" H 7215 4246 50  0000 L CNN
+F 0 "C6" H 7215 4246 50  0000 L CNN
 F 1 "1n" H 7215 4155 50  0000 L CNN
 F 2 "Capacitor_SMD:C_0805_2012Metric" H 7138 4050 50  0001 C CNN
@@
 AR Path="/5DC77C5E/5DC7443D" Ref="#PWR010"  Part="1"
 AR Path="/5DC77D5C/5DC7443D" Ref="#PWR015"  Part="1"
-F 0 "#PWR05" H 7100 4150 50  0001 C CNN
+F 0 "#PWR015" H 7100 4150 50  0001 C CNN
 F 1 "GND" H 7105 4227 50  0000 C CNN
 F 2 "" H 7100 4400 50  0001 C CNN
@@
 AR Path="/5DC77C5E/5DCEB1D3" Ref="#PWR036"  Part="1"
 AR Path="/5DC77D5C/5DCEB1D3" Ref="#PWR037"  Part="1"
-F 0 "#PWR035" H 6250 3500 50  0001 C CNN
+F 0 "#PWR037" H 6250 3500 50  0001 C CNN
 F 1 "+3V3" H 6265 3823 50  0000 C CNN
 F 2 "" H 6250 3650 50  0001 C CNN
@@
 AR Path="/5DC77C5E/5DCAFD9E" Ref="U3"  Part="1"
 AR Path="/5DC77D5C/5DCAFD9E" Ref="U7"  Part="1"
-F 0 "U2" H 6350 4350 50  0000 L CNN
+F 0 "U7" H 6350 4350 50  0000 L CNN
 F 1 "ACS759xCB-200B-PFF" H 6350 4250 50  0000 L CNN
 F 2 "Sensor_Current:Allegro_CB_PFF" H 6250 4000 50  0001 C CNN
@@
 AR Path="/5DC77C5E/5DE77132" Ref="R34"  Part="1"
 AR Path="/5DC77D5C/5DE77132" Ref="R35"  Part="1"
-F 0 "R33" V 6643 4000 50  0000 C CNN
+F 0 "R35" V 6643 4000 50  0000 C CNN
 F 1 "4.7k" V 6734 4000 50  0000 C CNN
 F 2 "" V 6780 4000 50  0001 C CNN
