File: hardware/motor_controller/current_sensor.sch (KiCad schematic (older format))
At the start: 4 parts, among them U2 ACS759xCB-200B-PFF

Commit message: RTMI + Pedal Sensor + DC Current Sensor
Changed lines of the file:
@@
 EESchema Schematic File Version 4
+LIBS:electric-FIAT-cache
 EELAYER 30 0
 EELAYER END
 $Descr A4 11693 8268
 encoding utf-8
-Sheet 2 13
+Sheet 14 14
 Title ""
 Date ""
@@
 AR Path="/5DC77C5E/5DC6FAA7" Ref="#PWR09"  Part="1"
 AR Path="/5DC77D5C/5DC6FAA7" Ref="#PWR014"  Part="1"
-F 0 "#PWR014" H 6250 4100 50  0001 C CNN
+AR Path="/5E0A8F27/5DC6FAA7" Ref="#PWR?"  Part="1"
+F 0 "#PWR?" H 6250 4100 50  0001 C CNN
 F 1 "GND" H 6255 4177 50  0000 C CNN
 F 2 "" H 6250 4350 50  0001 C CNN
@@
 AR Path="/5DC77C5E/5DC71A7F" Ref="C3"  Part="1"
 AR Path="/5DC77D5C/5DC71A7F" Ref="C5"  Part="1"
-F 0 "C5" H 4615 4146 50  0000 L CNN
+AR Path="/5E0A8F27/5DC71A7F" Ref="C?"  Part="1"
+F 0 "C?" H 4615 4146 50  0000 L CNN
 F 1 "100n" H 4615 4055 50  0000 L CNN
 F 2 "Capacitor_SMD:C_0805_2012Metric" H 4538 3950 50  0001 C CNN
@@
 AR Path="/5DC77C5E/5DC71F2C" Ref="#PWR07"  Part="1"
 AR Path="/5DC77D5C/5DC71F2C" Ref="#PWR012"  Part="1"
-F 0 "#PWR012" H 4500 3750 50  0001 C CNN
+AR Path="/5E0A8F27/5DC71F2C" Ref="#PWR?"  Part="1"
+F 0 "#PWR?" H 4500 3750 50  0001 C CNN
 F 1 "+3.3V" H 4515 4073 50  0000 C CNN
 F 2 "" H 4500 3900 50  0001 C CNN
@@
 AR Path="/5DC77C5E/5DC7230E" Ref="#PWR08"  Part="1"
 AR Path="/5DC77D5C/5DC7230E" Ref="#PWR013"  Part="1"
-F 0 "#PWR013" H 4500 4050 50  0001 C CNN
+AR Path="/5E0A8F27/5DC7230E" Ref="#PWR?"  Part="1"
+F 0 "#PWR?" H 4500 4050 50  0001 C CNN
 F 1 "GND" H 4505 4127 50  0000 C CNN
 F 2 "" H 4500 4300 50  0001 C CNN
@@
 AR Path="/5DC77C5E/5DC730E7" Ref="C4"  Part="1"
 AR Path="/5DC77D5C/5DC730E7" Ref="C6"  Part="1"
-F 0 "C6" H 7215 4246 50  0000 L CNN
+AR Path="/5E0A8F27/5DC730E7" Ref="C?"  Part="1"
+F 0 "C?" H 7215 4246 50  0000 L CNN
 F 1 "1n" H 7215 4155 50  0000 L CNN
 F 2 "Capacitor_SMD:C_0805_2012Metric" H 7138 4050 50  0001 C CNN
@@
 AR Path="/5DC77C5E/5DC7443D" Ref="#PWR010"  Part="1"
 AR Path="/5DC77D5C/5DC7443D" Ref="#PWR015"  Part="1"
-F 0 "#PWR015" H 7100 4150 50  0001 C CNN
+AR Path="/5E0A8F27/5DC7443D" Ref="#PWR?"  Part="1"
+F 0 "#PWR?" H 7100 4150 50  0001 C CNN
 F 1 "GND" H 7105 4227 50  0000 C CNN
 F 2 "" H 7100 4400 50  0001 C CNN
@@
 AR Path="/5DC77C5E/5DCEB1D3" Ref="#PWR036"  Part="1"
 AR Path="/5DC77D5C/5DCEB1D3" Ref="#PWR037"  Part="1"
-F 0 "#PWR037" H 6250 3500 50  0001 C CNN
+AR Path="/5E0A8F27/5DCEB1D3" Ref="#PWR?"  Part="1"
+F 0 "#PWR?" H 6250 3500 50  0001 C CNN
 F 1 "+3V3" H 6265 3823 50  0000 C CNN
 F 2 "" H 6250 3650 50  0001 C CNN
@@
 AR Path="/5DC77C5E/5DCAFD9E" Ref="U3"  Part="1"
 AR Path="/5DC77D5C/5DCAFD9E" Ref="U7"  Part="1"
-F 0 "U7" H 6350 4350 50  0000 L CNN
+AR Path="/5E0A8F27/5DCAFD9E" Ref="U?"  Part="1"
+F 0 "U?" H 6350 4350 50  0000 L CNN
 F 1 "ACS759xCB-200B-PFF" H 6350 4250 50  0000 L CNN
 F 2 "Sensor_Current:Allegro_CB_PFF" H 6250 4000 50  0001 C CNN
@@
 AR Path="/5DC77C5E/5DE77132" Ref="R34"  Part="1"
 AR Path="/5DC77D5C/5DE77132" Ref="R35"  Part="1"
-F 0 "R35" V 6643 4000 50  0000 C CNN
+AR Path="/5E0A8F27/5DE77132" Ref="R?"  Part="1"
+F 0 "R?" V 6643 4000 50  0000 C CNN
 F 1 "4.7k" V 6734 4000 50  0000 C CNN
 F 2 "" V 6780 4000 50  0001 C CNN

Commit message: SD Card and other pins
Parts:
- renumbered C1 to C43, C2 to C44, R33 to R19, U2 to U10
Connections:
- net IGBT_PH1 renamed IP+
- net Motor_PH1 renamed IP-
Changed lines of the file:
@@
 EESchema Schematic File Version 4
-LIBS:electric-FIAT-cache
 EELAYER 30 0
 EELAYER END
@@
 AR Path="/5DC75544/5DC6FAA7" Ref="#PWR?"  Part="1"
 AR Path="/5DC755EE/5DC6FAA7" Ref="#PWR?"  Part="1"
-AR Path="/5DC773B5/5DC6FAA7" Ref="#PWR04"  Part="1"
-AR Path="/5DC77C5E/5DC6FAA7" Ref="#PWR09"  Part="1"
-AR Path="/5DC77D5C/5DC6FAA7" Ref="#PWR014"  Part="1"
-AR Path="/5E0A8F27/5DC6FAA7" Ref="#PWR?"  Part="1"
-F 0 "#PWR?" H 6250 4100 50  0001 C CNN
+AR Path="/5DC773B5/5DC6FAA7" Ref="#PWR075"  Part="1"
+AR Path="/5DC77C5E/5DC6FAA7" Ref="#PWR080"  Part="1"
+AR Path="/5DC77D5C/5DC6FAA7" Ref="#PWR085"  Part="1"
+AR Path="/5E0A8F27/5DC6FAA7" Ref="#PWR0123"  Part="1"
+F 0 "#PWR0123" H 6250 4100 50  0001 C CNN
 F 1 "GND" H 6255 4177 50  0000 C CNN
 F 2 "" H 6250 4350 50  0001 C CNN
@@
 	6250 4350 6250 4300
 Text HLabel 5850 3900 0    50   Input ~ 0
-IGBT_PH1
+IP+
 Text HLabel 5850 4100 0    50   Output ~ 0
-Motor_PH1
+IP-
 Text Notes 4100 3550 0    100  ~ 20
 Decoupling
@@
 AR Path="/5DC75544/5DC71A7F" Ref="C?"  Part="1"
 AR Path="/5DC755EE/5DC71A7F" Ref="C?"  Part="1"
-AR Path="/5DC773B5/5DC71A7F" Ref="C1"  Part="1"
-AR Path="/5DC77C5E/5DC71A7F" Ref="C3"  Part="1"
-AR Path="/5DC77D5C/5DC71A7F" Ref="C5"  Part="1"
-AR Path="/5E0A8F27/5DC71A7F" Ref="C?"  Part="1"
-F 0 "C?" H 4615 4146 50  0000 L CNN
+AR Path="/5DC773B5/5DC71A7F" Ref="C43"  Part="1"
+AR Path="/5DC77C5E/5DC71A7F" Ref="C45"  Part="1"
+AR Path="/5DC77D5C/5DC71A7F" Ref="C47"  Part="1"
+AR Path="/5E0A8F27/5DC71A7F" Ref="C64"  Part="1"
+F 0 "C64" H 4615 4146 50  0000 L CNN
 F 1 "100n" H 4615 4055 50  0000 L CNN
 F 2 "Capacitor_SMD:C_0805_2012Metric" H 4538 3950 50  0001 C CNN
@@
 AR Path="/5DC75544/5DC71F2C" Ref="#PWR?"  Part="1"
 AR Path="/5DC755EE/5DC71F2C" Ref="#PWR?"  Part="1"
-AR Path="/5DC773B5/5DC71F2C" Ref="#PWR02"  Part="1"
-AR Path="/5DC77C5E/5DC71F2C" Ref="#PWR07"  Part="1"
-AR Path="/5DC77D5C/5DC71F2C" Ref="#PWR012"  Part="1"
-AR Path="/5E0A8F27/5DC71F2C" Ref="#PWR?"  Part="1"
-F 0 "#PWR?" H 4500 3750 50  0001 C CNN
+AR Path="/5DC773B5/5DC71F2C" Ref="#PWR073"  Part="1"
+AR Path="/5DC77C5E/5DC71F2C" Ref="#PWR078"  Part="1"
+AR Path="/5DC77D5C/5DC71F2C" Ref="#PWR083"  Part="1"
+AR Path="/5E0A8F27/5DC71F2C" Ref="#PWR0121"  Part="1"
+F 0 "#PWR0121" H 4500 3750 50  0001 C CNN
 F 1 "+3.3V" H 4515 4073 50  0000 C CNN
 F 2 "" H 4500 3900 50  0001 C CNN
@@
 AR Path="/5DC75544/5DC7230E" Ref="#PWR?"  Part="1"
 AR Path="/5DC755EE/5DC7230E" Ref="#PWR?"  Part="1"
-AR Path="/5DC773B5/5DC7230E" Ref="#PWR03"  Part="1"
-AR Path="/5DC77C5E/5DC7230E" Ref="#PWR08"  Part="1"
-AR Path="/5DC77D5C/5DC7230E" Ref="#PWR013"  Part="1"
-AR Path="/5E0A8F27/5DC7230E" Ref="#PWR?"  Part="1"
-F 0 "#PWR?" H 4500 4050 50  0001 C CNN
+AR Path="/5DC773B5/5DC7230E" Ref="#PWR074"  Part="1"
+AR Path="/5DC77C5E/5DC7230E" Ref="#PWR079"  Part="1"
+AR Path="/5DC77D5C/5DC7230E" Ref="#PWR084"  Part="1"
+AR Path="/5E0A8F27/5DC7230E" Ref="#PWR0122"  Part="1"
+F 0 "#PWR0122" H 4500 4050 50  0001 C CNN
 F 1 "GND" H 4505 4127 50  0000 C CNN
 F 2 "" H 4500 4300 50  0001 C CNN
@@
 AR Path="/5DC75544/5DC730E7" Ref="C?"  Part="1"
 AR Path="/5DC755EE/5DC730E7" Ref="C?"  Part="1"
-AR Path="/5DC773B5/5DC730E7" Ref="C2"  Part="1"
-AR Path="/5DC77C5E/5DC730E7" Ref="C4"  Part="1"
-AR Path="/5DC77D5C/5DC730E7" Ref="C6"  Part="1"
-AR Path="/5E0A8F27/5DC730E7" Ref="C?"  Part="1"
-F 0 "C?" H 7215 4246 50  0000 L CNN
+AR Path="/5DC773B5/5DC730E7" Ref="C44"  Part="1"
+AR Path="/5DC77C5E/5DC730E7" Ref="C46"  Part="1"
+AR Path="/5DC77D5C/5DC730E7" Ref="C48"  Part="1"
+AR Path="/5E0A8F27/5DC730E7" Ref="C65"  Part="1"
+F 0 "C65" H 7215 4246 50  0000 L CNN
 F 1 "1n" H 7215 4155 50  0000 L CNN
 F 2 "Capacitor_SMD:C_0805_2012Metric" H 7138 4050 50  0001 C CNN
@@
 AR Path="/5DC75544/5DC7443D" Ref="#PWR?"  Part="1"
 AR Path="/5DC755EE/5DC7443D" Ref="#PWR?"  Part="1"
-AR Path="/5DC773B5/5DC7443D" Ref="#PWR05"  Part="1"
-AR Path="/5DC77C5E/5DC7443D" Ref="#PWR010"  Part="1"
-AR Path="/5DC77D5C/5DC7443D" Ref="#PWR015"  Part="1"
-AR Path="/5E0A8F27/5DC7443D" Ref="#PWR?"  Part="1"
-F 0 "#PWR?" H 7100 4150 50  0001 C CNN
+AR Path="/5DC773B5/5DC7443D" Ref="#PWR076"  Part="1"
+AR Path="/5DC77C5E/5DC7443D" Ref="#PWR081"  Part="1"
+AR Path="/5DC77D5C/5DC7443D" Ref="#PWR086"  Part="1"
+AR Path="/5E0A8F27/5DC7443D" Ref="#PWR0124"  Part="1"
+F 0 "#PWR0124" H 7100 4150 50  0001 C CNN
 F 1 "GND" H 7105 4227 50  0000 C CNN
 F 2 "" H 7100 4400 50  0001 C CNN
@@
 out
 $Comp
-L power:+3V3 #PWR035
+L power:+3V3 #PWR072
 U 1 1 5DCEB1D3
 P 6250 3650
-AR Path="/5DC773B5/5DCEB1D3" Ref="#PWR035"  Part="1"
-AR Path="/5DC77C5E/5DCEB1D3" Ref="#PWR036"  Part="1"
-AR Path="/5DC77D5C/5DCEB1D3" Ref="#PWR037"  Part="1"
-AR Path="/5E0A8F27/5DCEB1D3" Ref="#PWR?"  Part="1"
-F 0 "#PWR?" H 6250 3500 50  0001 C CNN
+AR Path="/5DC773B5/5DCEB1D3" Ref="#PWR072"  Part="1"
+AR Path="/5DC77C5E/5DCEB1D3" Ref="#PWR077"  Part="1"
+AR Path="/5DC77D5C/5DCEB1D3" Ref="#PWR082"  Part="1"
+AR Path="/5E0A8F27/5DCEB1D3" Ref="#PWR0120"  Part="1"
+F 0 "#PWR0120" H 6250 3500 50  0001 C CNN
 F 1 "+3V3" H 6265 3823 50  0000 C CNN
 F 2 "" H 6250 3650 50  0001 C CNN
@@
 $EndComp
 $Comp
-L Sensor_Current:ACS759xCB-200B-PFF U2
+L Sensor_Current:ACS759xCB-200B-PFF U10
 U 1 1 5DCAFD9E
 P 6250 4000
-AR Path="/5DC773B5/5DCAFD9E" Ref="U2"  Part="1"
-AR Path="/5DC77C5E/5DCAFD9E" Ref="U3"  Part="1"
-AR Path="/5DC77D5C/5DCAFD9E" Ref="U7"  Part="1"
-AR Path="/5E0A8F27/5DCAFD9E" Ref="U?"  Part="1"
-F 0 "U?" H 6350 4350 50  0000 L CNN
+AR Path="/5DC773B5/5DCAFD9E" Ref="U10"  Part="1"
+AR Path="/5DC77C5E/5DCAFD9E" Ref="U11"  Part="1"
+AR Path="/5DC77D5C/5DCAFD9E" Ref="U12"  Part="1"
+AR Path="/5E0A8F27/5DCAFD9E" Ref="U19"  Part="1"
+F 0 "U19" H 6350 4350 50  0000 L CNN
 F 1 "ACS759xCB-200B-PFF" H 6350 4250 50  0000 L CNN
 F 2 "Sensor_Current:Allegro_CB_PFF" H 6250 4000 50  0001 C CNN
@@
 $EndComp
 $Comp
-L Device:R R33
+L Device:R R19
 U 1 1 5DE77132
 P 6850 4000
-AR Path="/5DC773B5/5DE77132" Ref="R33"  Part="1"
-AR Path="/5DC77C5E/5DE77132" Ref="R34"  Part="1"
-AR Path="/5DC77D5C/5DE77132" Ref="R35"  Part="1"
-AR Path="/5E0A8F27/5DE77132" Ref="R?"  Part="1"
-F 0 "R?" V 6643 4000 50  0000 C CNN
+AR Path="/5DC773B5/5DE77132" Ref="R19"  Part="1"
+AR Path="/5DC77C5E/5DE77132" Ref="R20"  Part="1"
+AR Path="/5DC77D5C/5DE77132" Ref="R21"  Part="1"
+AR Path="/5E0A8F27/5DE77132" Ref="R52"  Part="1"
+F 0 "R52" V 6643 4000 50  0000 C CNN
 F 1 "4.7k" V 6734 4000 50  0000 C CNN
 F 2 "" V 6780 4000 50  0001 C CNN
