File: hardware/motor_controller/electric-FIAT.sch (KiCad schematic (older format))
At the start: 32 parts, among them J1 Conn_01x10_Female, U4 OPA356xxDBV, U5 OPA356xxDBV, U6 STM32F405RGTx, Y1 32.768MHz, Y2 25MHz

Commit message: Added FOC controller
Parts:
- added U?: TMC4671-ES, trinamic-footprints:QFN76P, symbol fiat:TMC4671-ES
Changed lines of the file:
@@
 Text Label 2500 2700 0    50   ~ 0
 Current_PH3
+$Comp
+L fiat:TMC4671-ES U?
+U 1 1 5DC9033A
+P 5350 4700
+F 0 "U?" H 5350 2419 40  0000 C CNN
+F 1 "TMC4671-ES" H 5350 2343 40  0000 C CNN
+F 2 "trinamic-footprints:QFN76P" H 6400 4900 60  0001 L CNN
+F 3 "https://www.trinamic.com/fileadmin/assets/Products/ICs_Documents/TMC4671_datasheet_v1.03.pdf" H 6400 5000 60  0001 L CNN
+F 4 "1460-1302-ND" H 6400 5100 60  0001 L CNN "Digi-Key_PN"
+F 5 "TMC4671-ES" H 6400 5200 60  0001 L CNN "MPN"
+F 6 "Integrated Circuits (ICs)" H 6400 5300 60  0001 L CNN "Category"
+F 7 "PMIC - Motor Drivers, Controllers" H 6400 5400 60  0001 L CNN "Family"
+F 8 "https://www.trinamic.com/fileadmin/assets/Products/ICs_Documents/TMC4671_datasheet_v1.03.pdf" H 6400 5500 60  0001 L CNN "DK_Datasheet_Link"
+F 9 "/product-detail/en/trinamic-motion-control-gmbh/TMC4671-ES/1460-1302-ND/9450492" H 6400 5600 60  0001 L CNN "DK_Detail_Page"
+F 10 "IC MOTOR DRIVER MULTIPHASE 76QFN" H 6400 5700 60  0001 L CNN "Description"
+F 11 "Trinamic Motion Control GmbH" H 6400 5800 60  0001 L CNN "Manufacturer"
+F 12 "Active" H 6400 5900 60  0001 L CNN "Status"
+	1    5350 4700
+	1    0    0    -1
+$EndComp
 $EndSCHEMATC

Commit message: Connected Crystals
Parts:
- gave numbers to parts that had none: 1
Connections:
- net LSE_IN: now reaches U6.3 (PC14)
- net LSE_IN: now also C20.1, Y1.1
- net LSE_OUT: now reaches U6.4 (PC15)
- net LSE_OUT: now also C21.1, Y1.2
- net HSE_IN: now reaches U6.5 (PH0)
- net HSE_IN: now also C22.1, Y2.1
- net HSE_OUT: now reaches C23.1, Y2.3
Changed lines of the file:
@@
 	1    0    0    -1
 $EndComp
-$Comp
-L power:GND #PWR044
-U 1 1 5DCCC2B5
-P 6200 600
-F 0 "#PWR044" H 6200 350 50  0001 C CNN
-F 1 "GND" H 6205 427 50  0000 C CNN
-F 2 "" H 6200 600 50  0001 C CNN
-F 3 "" H 6200 600 50  0001 C CNN
-	1    6200 600
-	1    0    0    -1
-$EndComp
-Wire Wire Line
-	6050 850  6050 600
-Wire Wire Line
-	6050 600  6200 600
 Text Label 2500 3100 0    50   ~ 0
 SPI1_MISO
@@
 Inverter_temp
 NoConn ~ 10400 -1700
-$Comp
-L Device:Crystal_GND24 Y2
-U 1 1 5DCB2832
-P 6050 1050
-F 0 "Y2" H 6250 1200 50  0000 L CNN
-F 1 "25MHz" H 6250 1100 50  0000 L CNN
-F 2 "Crystal:Crystal_SMD_3225-4Pin_3.2x2.5mm" H 6050 1050 50  0001 C CNN
-F 3 "~" H 6050 1050 50  0001 C CNN
-	1    6050 1050
-	1    0    0    -1
-$EndComp
 Text Label 10450 3950 0    50   ~ 0
 Current_PH1
@@
 Text Label 2500 2700 0    50   ~ 0
 Current_PH3
+Text Label 5200 1050 0    50   ~ 0
+LSE_OUT
+Text Label 4800 1050 2    50   ~ 0
+LSE_IN
+Text Label 5850 1050 2    50   ~ 0
+HSE_IN
+Wire Wire Line
+	6050 850  6050 800
+Wire Wire Line
+	6050 800  6300 800
 $Comp
-L fiat:TMC4671-ES U?
+L power:GND #PWR044
+U 1 1 5DCCC2B5
+P 6300 800
+F 0 "#PWR044" H 6300 550 50  0001 C CNN
+F 1 "GND" H 6305 627 50  0000 C CNN
+F 2 "" H 6300 800 50  0001 C CNN
+F 3 "" H 6300 800 50  0001 C CNN
+	1    6300 800
+	1    0    0    -1
+$EndComp
+$Comp
+L Device:Crystal_GND24 Y2
+U 1 1 5DCB2832
+P 6050 1050
+F 0 "Y2" H 5650 1300 50  0000 L CNN
+F 1 "25MHz" H 5650 1200 50  0000 L CNN
+F 2 "Crystal:Crystal_SMD_3225-4Pin_3.2x2.5mm" H 6050 1050 50  0001 C CNN
+F 3 "~" H 6050 1050 50  0001 C CNN
+	1    6050 1050
+	1    0    0    -1
+$EndComp
+Text Label 6400 1050 0    50   ~ 0
+HSE_OUT
+Text Label 1100 5700 2    50   ~ 0
+LSE_OUT
+Text Label 1100 5600 2    50   ~ 0
+LSE_IN
+$Comp
+L fiat:TMC4671-ES U7
 U 1 1 5DC9033A
 P 5350 4700
-F 0 "U?" H 5350 2419 40  0000 C CNN
+F 0 "U7" H 5350 2419 40  0000 C CNN
 F 1 "TMC4671-ES" H 5350 2343 40  0000 C CNN
 F 2 "trinamic-footprints:QFN76P" H 6400 4900 60  0001 L CNN
@@
 	1    0    0    -1
 $EndComp
+Text Label 1100 3700 2    50   ~ 0
+HSE_IN
+Text Label 1150 3800 2    50   ~ 0
+HSE_OUT
 $EndSCHEMATC

Commit message: FOC controller, CAN and IGBTs
Parts:
- removed U7: TMC4671-ES, trinamic-footprints:QFN76P, symbol fiat:TMC4671-ES
- added J2: Conn_02x13_Odd_Even, Connector_IDC:IDC-Header_2x13_P2.54mm_Vertical_Lock, symbol Connector_Generic:Conn_02x13_Odd_Even
- added J3: Conn_01x02_Male, Connector_Phoenix_MSTB:PhoenixContact_MSTBVA_2,5_2-G-5,08_1x02_P5.08mm_Vertical, symbol Connector:Conn_01x02_Male
- added U1: TMC4671-ES, trinamic:TMC4671-ES, symbol fiat:TMC4671-ES
- added U8: MCP2562-E-SN, Package_SO:SOIC-8_3.9x4.9mm_P1.27mm, symbol Interface_CAN_LIN:MCP2562-E-SN
Connections:
- net +3V3: now also U8.5 (Vio)
- net GND: now also J2.18 (Pin_18), J2.19 (Pin_19), J2.21 (Pin_21), J2.23 (Pin_23), J2.25 (Pin_25), U1.14 (GNDIO2), U1.24 (GNDA), U1.3 (GNDIO1), U1.44 (GNDIO3), U1.53 (GNDIO4), U1.62 (GNDIO5), U1.73 (GNDIO6), U1.77 (PAD), U8.2 (VSS)
- net HSE_OUT: now also U6.6 (PH1)
- net SPI2_NSS: now reaches U6.33 (PB12)
- net SPI2_NSS: now also U1.6 (SPI_nSCS)
- net SPI2_SCK: now reaches U6.34 (PB13)
- net SPI2_SCK: now also U1.7 (SPI_SCK)
- net SPI2_MISO: now reaches U6.35 (PB14)
- net SPI2_MISO: now also U1.9 (SPI_MISO)
- net SPI2_MOSI: now reaches U6.36 (PB15)
- net SPI2_MOSI: now also U1.8 (SPI_MOSI)
- net FOC_Status: now reaches U6.37 (PC6)
- net FOC_Status: now also U1.12 (STATUS)
- net CAN_STBY: now reaches U6.43 (PA10)
- net CAN_STBY: now also U8.8 (STBY)
- net CAN_RX: now reaches U6.44 (PA11)
- net CAN_RX: now also U8.1 (TXD)
- net CAN_TX: now reaches U6.45 (PA12)
- net CAN_TX: now also U8.4 (RXD)
- new net: J3.1 (Pin_1), U8.6 (CANL)
- new net: J3.2 (Pin_2), U8.7 (CANH)
- new net +24V: J2.14 (Pin_14), J2.15 (Pin_15)
- new net +5V: U8.3 (VDD)
- no-connect marks 2 -> 12
Other:
- note added: "CAN Interface"
- note added: "FOC Controller"
- note added: "IGBT Connector"
- moved on the sheet: C11, C12, C13, C14, C15, C16, C17, C18, C19, R7, U6

Commit message: Added Voltage sensors
Parts:
- added C? (x2): 1n, symbol Device:C
- added C?: 10n, symbol Device:C
- added C? (x2): 0.1u, symbol Device:C
- added R?: 300k, symbol Device:R
- added R?: 2k, symbol Device:R
- added R?: 39, symbol Device:R
- added R? (x2): 20k, symbol Device:R
- added R? (x2): 220, symbol Device:R
- added U?: ACPL-C87A, Package_SO:SSO-8_6.8x5.9mm_P1.27mm_Clearance8mm, symbol Isolator_Analog:ACPL-C87A
- added U?: OPA356xxDBV, Package_TO_SOT_SMD:SOT-23-5, symbol Amplifier_Operational:OPA356xxDBV
Connections:
- net +3V3: now also C?.1, C?.1, U?.1 (VDD1), U?.5 (V+), U?.8 (VDD2)
- net GND: now also C?.2, C?.2, C?.2, C?.2, R?.2, R?.2, U?.2 (V-), U?.3 (IN-), U?.4 (GND1), U?.5 (GND2)
- new net: C?.1, R?.1, U?.2 (IN)
- new net: R?.1, U?.6 (OUT-)
- new net: R?.2, U?.7 (OUT+)
- new net: R?.1, R?.2, R?.2
- new net: C?.1, C?.1, R?.1, R?.1, R?.2, U?.4 (-)
- new net: R?.1, U?.3 (+)
- new net: C?.2, R?.2, U?.1
- new net +BATT: R?.1
Other:
- note added: "AC Phase Voltage Sensors"
- note added: "DC-Link Voltage Sensor"
- moved on the sheet: C10, C11, C12, C13, C14, C15, C16, C17, C18, C19, C20, C21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

Commit message: Anotation
Parts:
- gave numbers to parts that had none: 14
Other:
- moved on the sheet: C24, C25, C26, C27, C28, R10, R11, R12, R13, R14, R8, R9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

Commit message: DC/DC converters added
Parts:
- added C?: 220p, symbol Device:C
- added C?: 4.7u, symbol Device:C
- added C? (x2): 470u, symbol Device:C
- added C?: 100u, symbol Device:C
- added C?: 10u, symbol Device:C
- added C?: 1000p, symbol Device:C
- added L?: 4.7u, symbol Device:L
- added L?: 6.4u, symbol Device:L
- added L?: 398u, symbol Device:L_Core_Iron_Coupled
- added PS?: ITX1205SA, Converter_DCDC:Converter_DCDC_XP_POWER-ITXxxxxSA_THT, symbol Converter_DCDC:ITX1205SA
- added PS?: IU1203SA, Converter_DCDC:Converter_DCDC_XP_POWER-ITXxxxxSA_THT, symbol Converter_DCDC:ITX1203SA
- added U?: TEN40-1215, Converter_DCDC:Converter_DCDC_TRACO_TEN20-xxxx_THT, symbol Converter_DCDC:TEN20-2412WIN
- added U?: SR05S1V8, Converter_DCDC:Converter_DCDC_muRata_OKI-78SR_Vertical, symbol Converter_DCDC:OKI-78SR-3.3_1.5-W36-C
Connections:
- net labels added: +12V
- wire segments 200 -> 241
Other:
- note added: "12V/1.8V\n"
- note added: "12V/24V"
- note added: "12V/3.3V\n"
- note added: "12V/5V\n"
- note added: "DC/DC Converters\n"

Commit message: DC/DC converters updated
Parts:
- removed L?: 4.7u, symbol Device:L
- removed L?: 6.4u, symbol Device:L
- removed L?: 398u, symbol Device:L_Core_Iron_Coupled
- added C45: 270u, symbol Device:C
- added C47: 470p, symbol Device:C
- added C50: 680p, symbol Device:C
- C44, C51: renamed from C?; Note (none) -> 50V
- C48, C49: renamed from C?; Note (none) -> 35V
- C52: renamed from C?; Note (none) -> 3kV
- gave numbers to parts that had none: 6
Connections:
- wire segments 241 -> 243
Other:
- moved on the sheet: C48, C49, C51, C52, C53
