File: hardware/motor_controller/electric-FIAT.sch (KiCad schematic (older format))
At the start: 84 parts, among them J1 Conn_02x13_Odd_Even, J2 Conn_01x02_Male, J3 Micro_SD_Card_Det, J4 RTMI, J5 Conn_01x10_Female, U1 TEN40-1215, U2 OPA356xxDBV, U3 OPA356xxDBV, U4 74LS04, U5 ACPL-C87A, U6 OPA356xxDBV, U7 TMC4671-ES, U8 STM32F405RGTx, U9 MCP2562-E-SN, Y1 32.768MHz, Y2 25MHz

Commit message: Pedal Sensor + Program/Debug
Parts:
- added J6: Program/Debug, symbol Connector:Conn_01x06_Male
- added R53: 1k, symbol Device:R
- Pedal_Sensor1: renamed from RV1; value Pedal Sensor -> 5.1k
Connections:
- net +3V3: now also J6.1 (Pin_1), R53.1; no longer Pedal_Sensor1.1
- net GND: now also J6.6 (Pin_6)
- net GPIO0: now also J4.2 (Pin_2), U7.71 (GPIO1/ADC_I1_MCD)
- net GPIO1: now also J4.4 (Pin_4), U7.70 (GPIO0/ADC_I0_MCD)
- net reset: now also R9.1, U7.50 (nRST), J6.5 (Pin_5)
- net SWDIO: now reaches U8.46 (PA13)
- net SWDIO: now also J6.2 (Pin_2)
- net SWCLK: now reaches U8.49 (PA14)
- net SWCLK: now also J6.3 (Pin_3)
- net SWO: now reaches U8.55 (PB3)
- net SWO: now also J6.4 (Pin_4)
- new net: Pedal_Sensor1.1, R53.2
- no-connect marks 35 -> 33
Other:
- moved on the sheet: R9
Changed lines of the file:
@@
 EESchema Schematic File Version 4
+LIBS:electric-FIAT-cache
 EELAYER 30 0
 EELAYER END
@@
 SPI2_NSS
 NoConn ~ 6700 4700
-NoConn ~ 6700 4800
-NoConn ~ 6700 4900
 $Comp
 L Connector_Generic:Conn_02x13_Odd_Even J1
@@
 L power:GND #PWR040
 U 1 1 5DFE6F2E
-P 3900 3300
-F 0 "#PWR040" H 3900 3050 50  0001 C CNN
-F 1 "GND" H 3905 3127 50  0000 C CNN
-F 2 "" H 3900 3300 50  0001 C CNN
-F 3 "" H 3900 3300 50  0001 C CNN
-	1    3900 3300
+P 3750 3300
+F 0 "#PWR040" H 3750 3050 50  0001 C CNN
+F 1 "GND" H 3755 3127 50  0000 C CNN
+F 2 "" H 3750 3300 50  0001 C CNN
+F 3 "" H 3750 3300 50  0001 C CNN
+	1    3750 3300
 	1    0    0    -1
 $EndComp
@@
 L Device:R R9
 U 1 1 5DEE358A
-P 4250 3400
-F 0 "R9" V 4043 3400 50  0000 C CNN
-F 1 "10k" V 4134 3400 50  0000 C CNN
-F 2 "Resistor_SMD:R_0805_2012Metric" V 4180 3400 50  0001 C CNN
-F 3 "~" H 4250 3400 50  0001 C CNN
-	1    4250 3400
+P 4100 3400
+F 0 "R9" V 3893 3400 50  0000 C CNN
+F 1 "10k" V 3984 3400 50  0000 C CNN
+F 2 "Resistor_SMD:R_0805_2012Metric" V 4030 3400 50  0001 C CNN
+F 3 "~" H 4100 3400 50  0001 C CNN
+	1    4100 3400
 	0    1    1    0
 $EndComp
 Wire Wire Line
-	3900 3300 4050 3300
-Wire Wire Line
-	4100 3400 4050 3400
-Wire Wire Line
-	4050 3400 4050 3300
-Connection ~ 4050 3300
-Wire Wire Line
-	4050 3300 4400 3300
+	3750 3300 3900 3300
+Wire Wire Line
+	3950 3400 3900 3400
+Wire Wire Line
+	3900 3400 3900 3300
+Connection ~ 3900 3300
 NoConn ~ 4400 4800
 NoConn ~ 4400 4900
@@
 SD_DAT1
 $Comp
-L Device:R_POT RV1
+L Device:R_POT Pedal_Sensor1
 U 1 1 5DF3A930
 P 1150 10400
-F 0 "RV1" H 1080 10446 50  0000 R CNN
-F 1 "Pedal Sensor" H 1080 10355 50  0000 R CNN
+F 0 "Pedal_Sensor1" H 1080 10446 50  0000 R CNN
+F 1 "5.1k" H 1080 10355 50  0000 R CNN
 F 2 "" H 1150 10400 50  0001 C CNN
 F 3 "~" H 1150 10400 50  0001 C CNN
@@
 L power:+3V3 #PWR067
 U 1 1 5DF5758D
-P 1150 10250
-F 0 "#PWR067" H 1150 10100 50  0001 C CNN
-F 1 "+3V3" H 1165 10423 50  0000 C CNN
-F 2 "" H 1150 10250 50  0001 C CNN
-F 3 "" H 1150 10250 50  0001 C CNN
-	1    1150 10250
+P 1150 9750
+F 0 "#PWR067" H 1150 9600 50  0001 C CNN
+F 1 "+3V3" H 1165 9923 50  0000 C CNN
+F 2 "" H 1150 9750 50  0001 C CNN
+F 3 "" H 1150 9750 50  0001 C CNN
+	1    1150 9750
 	1    0    0    -1
 $EndComp
@@
 Text Label 2900 10300 2    50   ~ 0
 DBGSPI_nSCS
-Text Label 6800 4800 0    50   ~ 0
+Text Label 6700 4800 0    50   ~ 0
 GPIO0
-Text Label 6800 4900 0    50   ~ 0
-GPIO1
-Text Label 3500 10200 0    50   ~ 0
+Text Label 3400 10200 0    50   ~ 0
 GPIO0
-Text Label 3500 10300 0    50   ~ 0
+Text Label 3400 10300 0    50   ~ 0
 GPIO1
 Text Label 1300 10400 0    50   ~ 0
@@
 Wire Wire Line
 	4200 9600 4900 9600
+$Comp
+L Device:R R53
+U 1 1 5DF06CCF
+P 1150 10000
+F 0 "R53" H 1220 10046 50  0000 L CNN
+F 1 "1k" H 1220 9955 50  0000 L CNN
+F 2 "" V 1080 10000 50  0001 C CNN
+F 3 "~" H 1150 10000 50  0001 C CNN
+	1    1150 10000
+	1    0    0    -1
+$EndComp
+Wire Wire Line
+	1150 10250 1150 10150
+Wire Wire Line
+	1150 9750 1150 9850
+Text Label 6700 4900 0    50   ~ 0
+GPIO1
+$Comp
+L Connector:Conn_01x06_Male J6
+U 1 1 5DFBD3CB
+P 7650 10350
+F 0 "J6" H 7758 10731 50  0000 C CNN
+F 1 "Program/Debug" H 7758 10640 50  0000 C CNN
+F 2 "" H 7650 10350 50  0001 C CNN
+F 3 "~" H 7650 10350 50  0001 C CNN
+	1    7650 10350
+	1    0    0    -1
+$EndComp
+$Comp
+L power:+3V3 #PWR0125
+U 1 1 5DFC2B00
+P 8150 10150
+F 0 "#PWR0125" H 8150 10000 50  0001 C CNN
+F 1 "+3V3" H 8165 10323 50  0000 C CNN
+F 2 "" H 8150 10150 50  0001 C CNN
+F 3 "" H 8150 10150 50  0001 C CNN
+	1    8150 10150
+	1    0    0    -1
+$EndComp
+$Comp
+L power:GND #PWR0126
+U 1 1 5DFDC4C8
+P 8150 10650
+F 0 "#PWR0126" H 8150 10400 50  0001 C CNN
+F 1 "GND" H 8155 10477 50  0000 C CNN
+F 2 "" H 8150 10650 50  0001 C CNN
+F 3 "" H 8150 10650 50  0001 C CNN
+	1    8150 10650
+	1    0    0    -1
+$EndComp
+Wire Wire Line
+	8150 10150 7850 10150
+Wire Wire Line
+	7850 10650 8150 10650
+Text Label 7850 10250 0    50   ~ 0
+SWDIO
+Text Label 7850 10350 0    50   ~ 0
+SWCLK
+Text Label 7850 10450 0    50   ~ 0
+SWO
+Text Label 7850 10550 0    50   ~ 0
+reset
+Text Label 2600 5000 0    50   ~ 0
+SWDIO
+Text Label 2600 5100 0    50   ~ 0
+SWCLK
+Text Label 2600 5700 0    50   ~ 0
+SWO
+Text Label 4200 3550 2    50   ~ 0
+reset
+Wire Wire Line
+	4400 3400 4300 3400
+Wire Wire Line
+	4200 3550 4300 3550
+Wire Wire Line
+	4300 3550 4300 3400
+Connection ~ 4300 3400
+Wire Wire Line
+	4300 3400 4250 3400
+Wire Wire Line
+	3900 3300 4400 3300
 $EndSCHEMATC
