File: hardware/motor_controller/electric-FIAT.sch (KiCad schematic (older format))
At the start: 219 parts, among them J1 Conn_01x02_Male, J10 IMU, J11 SKiiP 613 GD123-3DUL V3, J12 Acc_sensor, J13 12V Battery, J14 Expansion, J2 Program/Debug, J3 RTMI, J4 Micro_SD_Card_Det, J5 Batt_conn, J6 Motor_U, J7 Encoder, J8 Motor_V, J9 Motor_W, Q1 AO3400, Q2 AO3400, Q3 AO3400, Q4 AO3400, Q5 AO3400, Q6 AO3400, U1 74LVC1GU04DRL, U10 ACPL-C87A, U11 OPA356xxDBV, U12 ACS759xCB-200B-PFF, U13 ACS759xCB-200B-PFF, U14 ACPL-C87A, U15 OPA356xxDBV, U16 ACS759xCB-200B-PFF, U17 OPA356xxDBV, U18 OPA356xxDBV, U19 ITW1205SA, U2 MCP2562-E-SN, U20 IU1203SA, U21 TEN40-1215E, U22 SR05S1V8, U23 74LVC1G14, U24 74LVC1G14, U25 74LVC1G14, U3 ACPL-C87A, U4 OPA356xxDBV, U5 ACPL-C87A, U6 OPA356xxDBV, U7 STM32F405RGTx, U8 TMC4671-ES, U9 ACS759xCB-200B-PFF, Y1 32.768MHz, Y2 25MHz

Commit message: Initial work on PCB
Parts:
- removed C41, C68: 100p, Capacitor_SMD:C_0805_2012Metric, symbol Device:C
- removed C51, C52: 100n, Capacitor_SMD:C_0805_2012Metric, symbol Device:C
- removed D1, D2, D3, D4: 3V3, symbol Device:D_Zener
- removed J12: Acc_sensor, Connector_Phoenix_MC_HighVoltage:PhoenixContact_MCV_1,5_2-G-5.08_1x02_P5.08mm_Vertical, symbol Connector:Conn_01x02_Male
- removed L2: 6.8u, Inductor_SMD:L_Coilcraft_LPS4018, symbol Device:L
- removed R54, R55: 4.7k, Resistor_SMD:R_0805_2012Metric, symbol Device:R
- removed R66: 100, Resistor_SMD:R_0805_2012Metric, symbol Device:R
- removed R68, R69: 390, Resistor_SMD:R_0805_2012Metric, symbol Device:R
- removed R92: 1k, Resistor_SMD:R_0805_2012Metric, symbol Device:R
- removed R93: 180, Resistor_SMD:R_0805_2012Metric, symbol Device:R
- removed TH2: Thermistor_NTC, Connector_Phoenix_MC_HighVoltage:PhoenixContact_MCV_1,5_2-G-5.08_1x02_P5.08mm_Vertical, symbol Device:Thermistor_NTC
- removed U22: SR05S1V8, fiat:Converter_DCDC_XP_POWER-SRxxSx_THT, symbol fiat:SR05S1V8
- removed U25: 74LVC1G14, fiat:Texas_R-PDSO-G5, symbol 74xGxx:74LVC1G14
- added C48: 100n, Capacitor_SMD:C_0805_2012Metric, symbol Device:C
- added C49: 50p, Capacitor_SMD:C_0805_2012Metric, symbol Device:C
- added C56: 10u, Capacitor_SMD:C_0805_2012Metric, symbol Device:C
- added D1, D2, D3: LED, LED_SMD:LED_0805_2012Metric, symbol Device:LED
- added J13: Accelerator, Connector_Phoenix_MC_HighVoltage:PhoenixContact_MCV_1,5_3-G-5.08_1x03_P5.08mm_Vertical, symbol Connector:Conn_01x03_Male
- added R64, R75: 1.7k, Resistor_SMD:R_0805_2012Metric, symbol Device:R
- added R76: 3.3k, Resistor_SMD:R_0805_2012Metric, symbol Device:R
- added R82, R83, R84: 1k, Resistor_SMD:R_0805_2012Metric, symbol Device:R
- added R94: 2k, Resistor_SMD:R_0805_2012Metric, symbol Device:R
- added SW1: SW_Push, Button_Switch_SMD:SW_SPST_CK_RS282G05A3, symbol Switch:SW_Push
- added U14, U19: OPA356xxDBV, Package_TO_SOT_SMD:SOT-23-5, symbol Amplifier_Operational:OPA356xxDBV
- added U20: 74LVC1G14, fiat:Texas_R-PDSO-G5, symbol 74xGxx:74LVC1G14
- Brake1: renamed from Pedal_Sensor1; footprint Connector_Phoenix_MC_HighVoltage:PhoenixContact_MCV_1,5_2-G-5.08_1x02_P5.08mm_Vertical -> Connector_Phoenix_MC_HighVoltage:PhoenixContact_MCV_1,5_3-G-5.08_1x03_P5.08mm_Vertical
- C42: value 50p -> 100n
- C55: renamed from C54; value 10u -> 100u; footprint Capacitor_SMD:C_0805_2012Metric -> Capacitor_THT:CP_Radial_D10.0mm_P5.00mm
- C62: renamed from C56; footprint (none) -> Capacitor_THT:CP_Radial_D10.0mm_P5.00mm
- C63, C64: value 470u -> 100n; footprint (none) -> Capacitor_SMD:C_0805_2012Metric
- R65: value 100 -> 3.3k
- R90: value 1k -> 4.5k
- R91: value 3.3k -> 3.2k
- R93: renamed from R88; value 1.8k -> 2.2k
- renumbered C66 to C10, C14 to C11, C15 to C12, C16 to C13, C12 to C14, C13 to C15, C17 to C16, C18 to C17, C19 to C18, C10 to C19, C11 to C20, C20 to C21, C21 to C22, C22 to C23, C23 to C24, C24 to C25, C25 to C26, C26 to C27, C27 to C28, C28 to C29, C31 to C30, C32 to C31, C33 to C32, C29 to C33, C30 to C34, C34 to C35, C35 to C36, C36 to C37, C37 to C38, C38 to C39, C39 to C40, C40 to C41, C67 to C43, C45 to C44, C43 to C45, C44 to C46, C46 to C47, C47 to C50, C48 to C51, C49 to C52, C50 to C53, C53 to C54, C55 to C61, C61 to C65, C65 to C66, C62 to C67, J9 to J10, J7 to J12, J13 to J14, J14 to J3, J3 to J4, J4 to J5, J5 to J6, J6 to J7, J10 to J8, J8 to J9, Q3 to Q1, Q4 to Q2, Q1 to Q3, Q2 to Q4, R12 to R10, R13 to R11, R14 to R12, R3 to R13, R4 to R14, R20 to R19, R19 to R20, R22 to R21, R23 to R22, R24 to R23, R25 to R24, R26 to R25, R27 to R26, R28 to R27, R29 to R28, R30 to R29, R5 to R3, R31 to R30, R21 to R31, R39 to R38, R40 to R39, R6 to R4, R41 to R40, R42 to R41, R43 to R42, R44 to R43, R45 to R44, R46 to R45, R47 to R46, R38 to R47, R94 to R49, R7 to R5, R49 to R50, R50 to R51, R51 to R53, R53 to R54, R56 to R55, R57 to R56, R58 to R57, R59 to R58, R60 to R59, R8 to R6, R61 to R60, R62 to R61, R63 to R62, R64 to R63, R74 to R66, R75 to R68, R76 to R69, R9 to R7, R78 to R70, R79 to R71, R80 to R72, R81 to R73, R77 to R74, R70 to R77, R71 to R78, R72 to R79, R10 to R8, R73 to R80, R82 to R81, R83 to R85, R84 to R86, R85 to R87, R86 to R88, R11 to R9, R87 to R92, U9 to U10, U10 to U11, U11 to U12, U12 to U13, U24 to U15, U13 to U16, U14 to U17, U15 to U18, U23 to U2, U16 to U21, U19 to U22, U21 to U23, U20 to U24, U17 to U25, U18 to U26, U2 to U3, U3 to U4, U4 to U5, U5 to U6, U6 to U7, U7 to U8, U8 to U9
Connections:
- net labels added: DC+, IGBT_Temp
- net labels removed: Inverter_temp
- wire segments 561 -> 543
Other:
- note added: "LED & Buttons"
- note added: "STATUS"
- moved on the sheet: Brake1, C11, C12, C13, C16, C17, C18, C23, C24, C25, C26, C27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

Commit message: Schematic v1.0 and PCB in progress
Parts:
- removed JP1: Clock Selection, Connector_PinHeader_2.54mm:PinHeader_1x03_P2.54mm_Vertical, symbol Jumper:Jumper_3_Bridged12
- removed R1: 1M, Resistor_SMD:R_0805_2012Metric, symbol Device:R
- removed R13: 3k, Resistor_SMD:R_0805_2012Metric, symbol Device:R
- removed SW1: SW_Push, Button_Switch_SMD:SW_SPST_CK_RS282G05A3, symbol Switch:SW_Push
- removed U1: 74LVC1GU04DRL, Package_TO_SOT_SMD:SOT-553, symbol 74xGxx:74LVC1GU04DRL
- removed U2: 74LVC1G14, fiat:Texas_R-PDSO-G5, symbol 74xGxx:74LVC1G14
- added C68, C69, C70, C71, C72, C73, C74: 100n, Capacitor_SMD:C_0805_2012Metric, symbol Device:C
- added D4, D5, D6, D7, D8: LED, LED_SMD:LED_0805_2012Metric, symbol Device:LED
- added R95, R96, R97, R98, R99: 1k, Resistor_SMD:R_0805_2012Metric, symbol Device:R
- C10: value 50p -> 100n
- J1: value Conn_01x02_Male -> CAN
Connections:
- net labels removed: +1V8, Crystal_25MHZ, MCU_MCO
- wire segments 543 -> 517
Other:
- note added: "LEDs"
- note removed: "LED & Buttons"
- moved on the sheet: C1, C14, C15, C19, C2, C20, C21, C22, C3, C4, C5, D1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

Commit message: Add Bus voltage measurement to TMC4671
Parts:
- D1: renamed from D3; value LED -> GREEN
- renumbered C21 to C1, C8 to C10, C9 to C11, C10 to C12, C72 to C13, C11 to C14, C12 to C15, C13 to C16, C68 to C17, C19 to C18, C20 to C19, C22 to C2, C14 to C20, C15 to C21, C16 to C22, C17 to C23, C18 to C24, C23 to C25, C24 to C26, C73 to C27, C74 to C28, C25 to C29, C1 to C3, C26 to C30, C27 to C31, C69 to C32, C28 to C33, C29 to C34, C30 to C35, C31 to C36, C32 to C37, C70 to C38, C33 to C39, C2 to C4, C34 to C40, C35 to C41, C36 to C42, C37 to C43, C38 to C44, C39 to C45, C40 to C46, C41 to C47, C71 to C48, C42 to C49, C3 to C5, C43 to C50, C44 to C51, C45 to C52, C46 to C53, C47 to C54, C48 to C55, C49 to C56, C50 to C57, C51 to C58, C52 to C59, C4 to C6, C53 to C60, C54 to C61, C55 to C62, C56 to C63, C57 to C64, C58 to C65, C59 to C66, C60 to C67, C61 to C68, C62 to C69, C5 to C7, C63 to C70, C64 to C71, C65 to C72, C66 to C73, C67 to C74, C6 to C8, C7 to C9, D1 to D2, D2 to D3, J3 to J2, J2 to J3, R2 to R1, R11 to R10, R12 to R11, R14 to R12, R15 to R13, R16 to R14, R17 to R15, R18 to R16, R19 to R17, R20 to R18, R21 to R19, R3 to R2, R22 to R20, R23 to R21, R24 to R22, R25 to R23, R26 to R24, R27 to R25, R28 to R26, R29 to R27, R30 to R28, R31 to R29, R4 to R3, R32 to R30, R33 to R31, R34 to R32, R35 to R33, R36 to R34, R37 to R35, R38 to R36, R39 to R37, R40 to R38, R41 to R39, R5 to R4, R42 to R40, R43 to R41, R44 to R42, R45 to R43, R46 to R44, R47 to R45, R48 to R46, R49 to R47, R50 to R48, R51 to R49, R6 to R5, R52 to R50, R53 to R51, R54 to R52, R55 to R53, R56 to R54, R57 to R55, R58 to R56, R59 to R57, R60 to R58, R61 to R59, R7 to R6, R62 to R60, R63 to R61, R64 to R62, R65 to R63, R66 to R64, R67 to R65, R68 to R66, R69 to R67, R70 to R68, R71 to R69, R8 to R7, R72 to R70, R73 to R71, R74 to R72, R75 to R73, R76 to R74, R77 to R75, R78 to R76, R79 to R77, R80 to R78, R81 to R79, R9 to R8, R84 to R80, R82 to R81, R83 to R82, R95 to R83, R96 to R84, R97 to R85, R98 to R86, R99 to R87, R85 to R88, R86 to R89, R10 to R9, R87 to R90, R88 to R91, R89 to R92, R90 to R93, R91 to R94, R92 to R95, R93 to R96, R94 to R97, U3 to U1, U12 to U10, U13 to U11, U14 to U12, U15 to U13, U16 to U14, U17 to U15, U18 to U16, U19 to U17, U20 to U18, U21 to U19, U4 to U2, U22 to U20, U23 to U21, U24 to U22, U25 to U23, U26 to U24, U5 to U3, U6 to U4, U7 to U5, U8 to U6, U9 to U7, U10 to U8, U11 to U9
Connections:
- net TMC_VM: now reaches R3.1, R4.1
- net TMC_VM: now also U7.20 (ADC_VM)
- no-connect marks 47 -> 46
Other:
- moved on the sheet: D2, D3, D4, D5, D6, D7, D8, R81, R82, R83, R84, R85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

Commit message: PCB final size
Parts:
- removed C63, C68: 10u, Capacitor_SMD:C_0805_2012Metric, symbol Device:C
- J1: footprint Connector_Phoenix_MC_HighVoltage:PhoenixContact_MCV_1,5_2-G-5.08_1x02_P5.08mm_Vertical -> Connector_Phoenix_MC:PhoenixContact_MCV_1,5_2-G-3.81_1x02_P3.81mm_Vertical
- J12: footprint Connector_PinHeader_2.54mm:PinHeader_1x04_P2.54mm_Vertical -> Connector_Phoenix_MC:PhoenixContact_MCV_1,5_4-G-3.81_1x04_P3.81mm_Vertical
- J13: footprint Connector_Phoenix_MC_HighVoltage:PhoenixContact_MCV_1,5_3-G-5.08_1x03_P5.08mm_Vertical -> Connector_Phoenix_MC:PhoenixContact_MCV_1,5_3-G-3.81_1x03_P3.81mm_Vertical
- J15: renamed from Brake1; footprint Connector_Phoenix_MC_HighVoltage:PhoenixContact_MCV_1,5_3-G-5.08_1x03_P5.08mm_Vertical -> Connector_Phoenix_MC:PhoenixContact_MCV_1,5_3-G-3.81_1x03_P3.81mm_Vertical
- J2, J4: footprint Connector_IDC:IDC-Header_2x05_P2.54mm_Vertical -> Connector_Phoenix_MC:PhoenixContact_MCV_1,5_10-G-3.81_1x10_P3.81mm_Vertical
- J3: footprint Connector_Phoenix_MSTB:PhoenixContact_MSTBVA_2,5_6-G_1x06_P5.00mm_Vertical -> Connector_Phoenix_MC:PhoenixContact_MCV_1,5_6-G-3.81_1x06_P3.81mm_Vertical
- renumbered C69 to C63, C70 to C68, C71 to C69, C72 to C70, C74 to C71, C73 to C72, U22 to U21, U21 to U22
Connections:
- net -BATT: now also J14.2 (Pin_2)
- net GND: no longer J14.2 (Pin_2)
Other:
- moved on the sheet: C63, C71, J14, U21

Commit message: Change debug connectors, Motor W Voltage and round PCB corners
Parts:
- removed J3: Program/Debug, Connector_Phoenix_MC:PhoenixContact_MCV_1,5_6-G-3.81_1x06_P3.81mm_Vertical, symbol Connector:Conn_01x06_Male
- added J3: Debug, Connector_IDC:IDC-Header_2x10_P2.54mm_Vertical, symbol Connector_Generic:Conn_02x10_Odd_Even
- D1: value GREEN -> Green
- D2: value LED -> Blue
- D3: value LED -> White
- D4, D5, D6, D8: value LED -> Red
- D7: value LED -> Yellow
- J2, J4: footprint Connector_Phoenix_MC:PhoenixContact_MCV_1,5_10-G-3.81_1x10_P3.81mm_Vertical -> Connector_IDC:IDC-Header_2x05_P2.54mm_Vertical
Connections:
- net +3V3: now also J2.1 (Pin_1), J3.1 (Pin_1); no longer J2.3 (Pin_3)
- net +5V: now also J2.3 (Pin_3); no longer J2.1 (Pin_1)
- net ENABLE_INPUTS: no longer D3.2 (A)
- net GND: now also J3.10 (Pin_10), J3.12 (Pin_12), J3.4 (Pin_4), J3.6 (Pin_6), J3.8 (Pin_8)
- net SD_DET: now also D3.2 (A)
- net SWCLK: now also J3.9 (Pin_9)
- net SWDIO: now also J3.7 (Pin_7)
- net SWO: now also J3.13 (Pin_13)
- net reset: now also J3.15 (Pin_15)
- no-connect marks 46 -> 56
Changed lines of the file:
@@
 Sheet 1 1
 Title "Motor Controller"
-Date "2019-12-18"
-Rev "1.0.1"
+Date "2019-12-20"
+Rev "1.0.2"
 Comp ""
 Comment1 ""
@@
 	8050 1000 8050 1050
 $Comp
-L power:+3V3 #PWR017
+L power:+3V3 #PWR018
 U 1 1 5DDBD09A
 P 7150 1550
-F 0 "#PWR017" H 7150 1400 50  0001 C CNN
+F 0 "#PWR018" H 7150 1400 50  0001 C CNN
 F 1 "+3V3" H 7165 1723 50  0000 C CNN
 F 2 "" H 7150 1550 50  0001 C CNN
@@
 F 0 "J4" H 1350 3017 50  0000 C CNN
 F 1 "RTMI" H 1350 2926 50  0000 C CNN
-F 2 "Connector_Phoenix_MC:PhoenixContact_MCV_1,5_10-G-3.81_1x10_P3.81mm_Vertical" H 1300 2600 50  0001 C CNN
+F 2 "Connector_IDC:IDC-Header_2x05_P2.54mm_Vertical" H 1300 2600 50  0001 C CNN
 F 3 "~" H 1300 2600 50  0001 C CNN
 	1    1300 2600
@@
 Text Notes 4050 600  0    50   ~ 0
 Decoupling
-Text Label 6450 2000 0    50   ~ 0
+Text Label 6200 2250 2    50   ~ 0
 reset
-Text Label 6450 1900 0    50   ~ 0
+Text Label 6200 2150 2    50   ~ 0
 SWO
-Text Label 6450 1800 0    50   ~ 0
+Text Label 6200 1950 2    50   ~ 0
 SWCLK
-Text Label 6450 1700 0    50   ~ 0
+Text Label 6200 1850 2    50   ~ 0
 SWDIO
 Wire Wire Line
-	6750 1600 6450 1600
-$Comp
-L power:GND #PWR037
-U 1 1 5DFDC4C8
-P 6450 2100
-F 0 "#PWR037" H 6450 1850 50  0001 C CNN
-F 1 "GND" H 6455 1927 50  0000 C CNN
-F 2 "" H 6450 2100 50  0001 C CNN
-F 3 "" H 6450 2100 50  0001 C CNN
-	1    6450 2100
-	1    0    0    -1
-$EndComp
+	7450 1950 7150 1950
 $Comp
-L power:+3V3 #PWR019
+L power:+3V3 #PWR017
 U 1 1 5DFC2B00
-P 6750 1600
-F 0 "#PWR019" H 6750 1450 50  0001 C CNN
-F 1 "+3V3" H 6765 1773 50  0000 C CNN
-F 2 "" H 6750 1600 50  0001 C CNN
-F 3 "" H 6750 1600 50  0001 C CNN
-	1    6750 1600
-	1    0    0    -1
-$EndComp
-$Comp
-L Connector:Conn_01x06_Male J3
-U 1 1 5DFBD3CB
-P 6250 1800
-F 0 "J3" H 6358 2181 50  0000 C CNN
-F 1 "Program/Debug" H 6358 2090 50  0000 C CNN
-F 2 "Connector_Phoenix_MC:PhoenixContact_MCV_1,5_6-G-3.81_1x06_P3.81mm_Vertical" H 6250 1800 50  0001 C CNN
-F 3 "~" H 6250 1800 50  0001 C CNN
-	1    6250 1800
+P 6200 1550
+F 0 "#PWR017" H 6200 1400 50  0001 C CNN
+F 1 "+3V3" H 6215 1723 50  0000 C CNN
+F 2 "" H 6200 1550 50  0001 C CNN
+F 3 "" H 6200 1550 50  0001 C CNN
+	1    6200 1550
 	1    0    0    -1
 $EndComp
@@
 $EndComp
 $Comp
-L power:+3V3 #PWR025
+L power:+3V3 #PWR019
 U 1 1 5E673382
-P 2650 1700
-F 0 "#PWR025" H 2650 1550 50  0001 C CNN
-F 1 "+3V3" H 2665 1873 50  0000 C CNN
-F 2 "" H 2650 1700 50  0001 C CNN
-F 3 "" H 2650 1700 50  0001 C CNN
-	1    2650 1700
+P 2800 1600
+F 0 "#PWR019" H 2800 1450 50  0001 C CNN
+F 1 "+3V3" H 2815 1773 50  0000 C CNN
+F 2 "" H 2800 1600 50  0001 C CNN
+F 3 "" H 2800 1600 50  0001 C CNN
+	1    2800 1600
 	1    0    0    -1
 $EndComp
@@
 IO4
 $Comp
-L power:+5V #PWR018
+L power:+5V #PWR025
 U 1 1 5E7E9E07
-P 2800 1600
-F 0 "#PWR018" H 2800 1450 50  0001 C CNN
-F 1 "+5V" H 2815 1773 50  0000 C CNN
-F 2 "" H 2800 1600 50  0001 C CNN
-F 3 "" H 2800 1600 50  0001 C CNN
-	1    2800 1600
+P 2650 1700
+F 0 "#PWR025" H 2650 1550 50  0001 C CNN
+F 1 "+5V" H 2665 1873 50  0000 C CNN
+F 2 "" H 2650 1700 50  0001 C CNN
+F 3 "" H 2650 1700 50  0001 C CNN
+	1    2650 1700
 	1    0    0    -1
 $EndComp
 Wire Wire Line
-	2800 1600 2850 1600
-Wire Wire Line
 	2650 1700 2850 1700
 Wire Wire Line
+	2800 1600 2850 1600
+Wire Wire Line
 	2500 1800 2850 1800
 $Comp
@@
 F 0 "J2" H 3100 2217 50  0000 C CNN
 F 1 "Expansion" H 3100 2126 50  0000 C CNN
-F 2 "Connector_Phoenix_MC:PhoenixContact_MCV_1,5_10-G-3.81_1x10_P3.81mm_Vertical" H 3050 1800 50  0001 C CNN
+F 2 "Connector_IDC:IDC-Header_2x05_P2.54mm_Vertical" H 3050 1800 50  0001 C CNN
 F 3 "~" H 3050 1800 50  0001 C CNN
 	1    3050 1800
@@
 P 10700 8650
 F 0 "D1" V 10739 8533 50  0000 R CNN
-F 1 "GREEN" V 10648 8533 50  0000 R CNN
+F 1 "Green" V 10648 8533 50  0000 R CNN
 F 2 "LED_SMD:LED_0805_2012Metric" H 10700 8650 50  0001 C CNN
 F 3 "~" H 10700 8650 50  0001 C CNN
@@
 P 11300 8650
 F 0 "D2" V 11339 8533 50  0000 R CNN
-F 1 "LED" V 11248 8533 50  0000 R CNN
+F 1 "Blue" V 11248 8533 50  0000 R CNN
 F 2 "LED_SMD:LED_0805_2012Metric" H 11300 8650 50  0001 C CNN
 F 3 "~" H 11300 8650 50  0001 C CNN
@@
 	1    0    0    -1
 $EndComp
-Text Label 12100 8500 2    50   ~ 0
-ENABLE_INPUTS
-$Comp
-L Device:LED D3
-U 1 1 5F469FBF
-P 11850 8650
-F 0 "D3" V 11889 8533 50  0000 R CNN
-F 1 "LED" V 11798 8533 50  0000 R CNN
-F 2 "LED_SMD:LED_0805_2012Metric" H 11850 8650 50  0001 C CNN
-F 3 "~" H 11850 8650 50  0001 C CNN
-	1    11850 8650
-	0    -1   -1   0
-$EndComp
-$Comp
-L Device:R R82
-U 1 1 5F469FC5
-P 11850 8950
-F 0 "R82" H 11920 8996 50  0000 L CNN
-F 1 "1k" H 11920 8905 50  0000 L CNN
-F 2 "Resistor_SMD:R_0805_2012Metric" V 11780 8950 50  0001 C CNN
-F 3 "~" H 11850 8950 50  0001 C CNN
-	1    11850 8950
-	1    0    0    -1
-$EndComp
-$Comp
-L power:GND #PWR0157
-U 1 1 5F469FCB
-P 11850 9100
-F 0 "#PWR0157" H 11850 8850 50  0001 C CNN
-F 1 "GND" H 11855 8927 50  0000 C CNN
-F 2 "" H 11850 9100 50  0001 C CNN
-F 3 "" H 11850 9100 50  0001 C CNN
-	1    11850 9100
-	1    0    0    -1
-$EndComp
 Wire Wire Line
 	7650 4800 7650 5100
@@
 Text Label 12650 8500 2    50   ~ 0
 ERROR_HB1
-Wire Wire Line
-	12100 8500 11850 8500
 $Comp
 L Device:LED D4
@@
 P 12400 8650
 F 0 "D4" V 12439 8533 50  0000 R CNN
-F 1 "LED" V 12348 8533 50  0000 R CNN
+F 1 "Red" V 12348 8533 50  0000 R CNN
 F 2 "LED_SMD:LED_0805_2012Metric" H 12400 8650 50  0001 C CNN
 F 3 "~" H 12400 8650 50  0001 C CNN
@@
 P 12950 8650
 F 0 "D5" V 12989 8533 50  0000 R CNN
-F 1 "LED" V 12898 8533 50  0000 R CNN
+F 1 "Red" V 12898 8533 50  0000 R CNN
 F 2 "LED_SMD:LED_0805_2012Metric" H 12950 8650 50  0001 C CNN
 F 3 "~" H 12950 8650 50  0001 C CNN
@@
 P 13500 8650
 F 0 "D6" V 13539 8533 50  0000 R CNN
-F 1 "LED" V 13448 8533 50  0000 R CNN
+F 1 "Red" V 13448 8533 50  0000 R CNN
 F 2 "LED_SMD:LED_0805_2012Metric" H 13500 8650 50  0001 C CNN
 F 3 "~" H 13500 8650 50  0001 C CNN
@@
 IGBT_OVER_TEMP
 $Comp
-L Device:LED D7
-U 1 1 5E9865FE
-P 14050 8650
-F 0 "D7" V 14089 8533 50  0000 R CNN
-F 1 "LED" V 13998 8533 50  0000 R CNN
-F 2 "LED_SMD:LED_0805_2012Metric" H 14050 8650 50  0001 C CNN
-F 3 "~" H 14050 8650 50  0001 C CNN
-	1    14050 8650
-	0    -1   -1   0
-$EndComp
-$Comp
 L Device:R R86
 U 1 1 5E986604
@@
 $EndComp
 $Comp
-L Device:LED D8
-U 1 1 5E986612
-P 14600 8650
-F 0 "D8" V 14639 8533 50  0000 R CNN
-F 1 "LED" V 14548 8533 50  0000 R CNN
-F 2 "LED_SMD:LED_0805_2012Metric" H 14600 8650 50  0001 C CNN
-F 3 "~" H 14600 8650 50  0001 C CNN
-	1    14600 8650
-	0    -1   -1   0
-$EndComp
-$Comp
 L Device:R R87
 U 1 1 5E986618
@@
 Wire Wire Line
 	7250 10750 7050 10750
+$Comp
+L power:GND #PWR037
+U 1 1 5DFDC4C8
+P 6800 2050
+F 0 "#PWR037" H 6800 1800 50  0001 C CNN
+F 1 "GND" H 6805 1877 50  0000 C CNN
+F 2 "" H 6800 2050 50  0001 C CNN
+F 3 "" H 6800 2050 50  0001 C CNN
+	1    6800 2050
+	1    0    0    -1
+$EndComp
+NoConn ~ 6700 2150
+NoConn ~ 6700 2250
+NoConn ~ 6700 2350
+NoConn ~ 6700 2450
+NoConn ~ 6200 2450
+NoConn ~ 6200 2350
+NoConn ~ 6200 2050
+NoConn ~ 6200 1750
+NoConn ~ 6200 1650
+NoConn ~ 6700 1550
+Wire Wire Line
+	6800 2050 6700 2050
+$Comp
+L Connector_Generic:Conn_02x10_Odd_Even J3
+U 1 1 5E4EA8D5
+P 6400 1950
+F 0 "J3" H 6450 2567 50  0000 C CNN
+F 1 "Debug" H 6450 2476 50  0000 C CNN
+F 2 "Connector_IDC:IDC-Header_2x10_P2.54mm_Vertical" H 6400 1950 50  0001 C CNN
+F 3 "~" H 6400 1950 50  0001 C CNN
+	1    6400 1950
+	1    0    0    -1
+$EndComp
+Wire Wire Line
+	6700 1650 6700 1750
+Connection ~ 6700 1750
+Wire Wire Line
+	6700 1750 6700 1850
+Connection ~ 6700 1850
+Wire Wire Line
+	6700 1850 6700 1950
+Wire Wire Line
+	6700 1950 6700 2050
+Connection ~ 6700 1950
+Connection ~ 6700 2050
+Wire Wire Line
+	11950 8500 11850 8500
+$Comp
+L power:GND #PWR0157
+U 1 1 5F469FCB
+P 11850 9100
+F 0 "#PWR0157" H 11850 8850 50  0001 C CNN
+F 1 "GND" H 11855 8927 50  0000 C CNN
+F 2 "" H 11850 9100 50  0001 C CNN
+F 3 "" H 11850 9100 50  0001 C CNN
+	1    11850 9100
+	1    0    0    -1
+$EndComp
+$Comp
+L Device:R R82
+U 1 1 5F469FC5
+P 11850 8950
+F 0 "R82" H 11920 8996 50  0000 L CNN
+F 1 "1k" H 11920 8905 50  0000 L CNN
+F 2 "Resistor_SMD:R_0805_2012Metric" V 11780 8950 50  0001 C CNN
+F 3 "~" H 11850 8950 50  0001 C CNN
+	1    11850 8950
+	1    0    0    -1
+$EndComp
+$Comp
+L Device:LED D3
+U 1 1 5F469FBF
+P 11850 8650
+F 0 "D3" V 11889 8533 50  0000 R CNN
+F 1 "White" V 11798 8533 50  0000 R CNN
+F 2 "LED_SMD:LED_0805_2012Metric" H 11850 8650 50  0001 C CNN
+F 3 "~" H 11850 8650 50  0001 C CNN
+	1    11850 8650
+	0    -1   -1   0
+$EndComp
+Text Label 11950 8500 2    50   ~ 0
+SD_DET
+$Comp
+L Device:LED D7
+U 1 1 5E9865FE
+P 14050 8650
+F 0 "D7" V 14089 8533 50  0000 R CNN
+F 1 "Yellow" V 13998 8533 50  0000 R CNN
+F 2 "LED_SMD:LED_0805_2012Metric" H 14050 8650 50  0001 C CNN
+F 3 "~" H 14050 8650 50  0001 C CNN
+	1    14050 8650
+	0    -1   -1   0
+$EndComp
+$Comp
+L Device:LED D8
+U 1 1 5E986612
+P 14600 8650
+F 0 "D8" V 14639 8533 50  0000 R CNN
+F 1 "Red" V 14548 8533 50  0000 R CNN
+F 2 "LED_SMD:LED_0805_2012Metric" H 14600 8650 50  0001 C CNN
+F 3 "~" H 14600 8650 50  0001 C CNN
+	1    14600 8650
+	0    -1   -1   0
+$EndComp
 $EndSCHEMATC

Commit message: Fix SPI
Parts:
- removed R29: 10k, Resistor_SMD:R_0805_2012Metric, symbol Device:R
- added H1, H2, H3, H4: MountingHole, MountingHole:MountingHole_5.3mm_M5, symbol Mechanical:MountingHole
- renumbered R30 to R29, R31 to R30, R32 to R31, R33 to R32, R34 to R33, R35 to R34, R36 to R35, R37 to R36, R38 to R37, R39 to R38, R40 to R39, R41 to R40, R42 to R41, R43 to R42, R44 to R43, R45 to R44, R46 to R45, R47 to R46, R48 to R47, R49 to R48, R50 to R49, R51 to R50, R52 to R51, R53 to R52, R54 to R53, R55 to R54, R56 to R55, R57 to R56, R58 to R57, R59 to R58, R60 to R59, R61 to R60, R62 to R61, R63 to R62, R64 to R63, R65 to R64, R66 to R65, R67 to R66, R68 to R67, R69 to R68, R70 to R69, R71 to R70, R72 to R71, R73 to R72, R74 to R73, R75 to R74, R76 to R75, R77 to R76, R78 to R77, R79 to R78, R80 to R79, R81 to R80, R82 to R81, R83 to R82, R84 to R83, R85 to R84, R86 to R85, R87 to R86, R88 to R87, R89 to R88, R90 to R89, R91 to R90, R92 to R91, R93 to R92, R94 to R93, R95 to R94, R96 to R95, R97 to R96
Connections:
- net TMC_VM: no longer names the net of R3.1, R4.1
- net TMC_VM: no longer U7.20 (ADC_VM)
- no-connect marks 56 -> 57
Other:
- moved on the sheet: J12

Commit message: Add FOC_reset and fix compilation errors
Parts:
- added R29: R, Resistor_SMD:R_0805_2012Metric, symbol Device:R
- renumbered R29 to R30, R30 to R31, R31 to R32, R32 to R33, R33 to R34, R34 to R35, R35 to R36, R36 to R37, R37 to R38, R38 to R39, R39 to R40, R40 to R41, R41 to R42, R42 to R43, R43 to R44, R44 to R45, R45 to R46, R46 to R47, R47 to R48, R48 to R49, R49 to R50, R50 to R51, R51 to R52, R52 to R53, R53 to R54, R54 to R55, R55 to R56, R56 to R57, R57 to R58, R58 to R59, R59 to R60, R60 to R61, R61 to R62, R62 to R63, R63 to R64, R64 to R65, R65 to R66, R66 to R67, R67 to R68, R68 to R69, R69 to R70, R70 to R71, R71 to R72, R72 to R73, R73 to R74, R74 to R75, R75 to R76, R76 to R77, R77 to R78, R78 to R79, R79 to R80, R80 to R81, R81 to R82, R82 to R83, R83 to R84, R84 to R85, R85 to R86, R86 to R87, R87 to R88, R88 to R89, R89 to R90, R90 to R91, R91 to R92, R92 to R93, R93 to R94, R94 to R95, R95 to R96, R96 to R97
Connections:
- net +3V3: now also R29.1
- net SPI2_NSS: no longer U6.21 (PA5)
- net reset: no longer U7.50 (nRST)
- new net FOC_reset: R29.2, U6.21 (PA5), U7.50 (nRST)

Commit message: PCB placing done, missing some connections
Parts:
- removed D2: Blue, LED_SMD:LED_0805_2012Metric, symbol Device:LED
- removed D3: White, LED_SMD:LED_0805_2012Metric, symbol Device:LED
- removed D4, D5, D6, D8: Red, LED_SMD:LED_0805_2012Metric, symbol Device:LED
- removed D7: Yellow, LED_SMD:LED_0805_2012Metric, symbol Device:LED
- removed J2: Expansion, Connector_IDC:IDC-Header_2x05_P2.54mm_Vertical, symbol Connector_Generic:Conn_02x05_Odd_Even
- removed J6: Batt_conn, fiat:Battery, symbol Connector:Conn_01x03_Male
- removed R81, R82, R83, R84, R85, R86: 1k, Resistor_SMD:R_0805_2012Metric, symbol Device:R
- added C14: 4.7u, Capacitor_SMD:C_0603_1608Metric, symbol Device:C
- added C15: 470n, Capacitor_SMD:C_0603_1608Metric, symbol Device:C
- added C2, C3, C32, C4, C5: 100n, Capacitor_SMD:C_0603_1608Metric, symbol Device:C
- added C70, C71: 100n, Capacitor_SMD:C_0805_2012Metric, symbol Device:C
- added J3: DC_Bus, Connector_Phoenix_MC:PhoenixContact_MCV_1,5_2-G-3.81_1x02_P3.81mm_Vertical, symbol Connector:Conn_01x02_Male
- added J6: Batt_conn, fiat:Motor_IGBT, symbol Connector:Conn_01x02_Male
- added R88: 1.8k, Resistor_SMD:R_0805_2012Metric, symbol Device:R
- added R93: 1k, Resistor_SMD:R_0805_2012Metric, symbol Device:R
- added R94: 4.3k, Resistor_SMD:R_0805_2012Metric, symbol Device:R
- added U20: 74LVC1G14, fiat:Texas_R-PDSO-G5, symbol 74xGxx:74LVC1G14
- added U22, U27: OPA356xxDBV, Package_TO_SOT_SMD:SOT-23-5, symbol Amplifier_Operational:OPA356xxDBV
- C1: renamed from C8; footprint Capacitor_SMD:C_0805_2012Metric -> Capacitor_SMD:C_0603_1608Metric
- C11: renamed from C7; footprint Capacitor_SMD:C_0805_2012Metric -> Capacitor_SMD:C_0603_1608Metric
- C22, C23, C24, C6: footprint Capacitor_SMD:C_0805_2012Metric -> Capacitor_SMD:C_0603_1608Metric
- C25: renamed from C18; footprint Capacitor_SMD:C_0805_2012Metric -> Capacitor_SMD:C_0603_1608Metric
- C26: renamed from C19; footprint Capacitor_SMD:C_0805_2012Metric -> Capacitor_SMD:C_0603_1608Metric
- C27: renamed from C20; footprint Capacitor_SMD:C_0805_2012Metric -> Capacitor_SMD:C_0603_1608Metric
- C28: renamed from C21; footprint Capacitor_SMD:C_0805_2012Metric -> Capacitor_SMD:C_0603_1608Metric
- C31: renamed from C9; value 100n -> 4.7u; footprint Capacitor_SMD:C_0805_2012Metric -> Capacitor_SMD:C_0603_1608Metric
- C7: renamed from C3; footprint Capacitor_SMD:C_0805_2012Metric -> Capacitor_SMD:C_0603_1608Metric
- C8: renamed from C4; footprint Capacitor_SMD:C_0805_2012Metric -> Capacitor_SMD:C_0603_1608Metric
- C80: renamed from C70; value 2.2n -> 1n; footprint Capacitor_SMD:C_0805_2012Metric -> Capacitor_SMD:C_1206_3216Metric; Note 3kV -> 1kV
- C81: renamed from C71; value 2.2n -> 1n; footprint Capacitor_SMD:C_0805_2012Metric -> Capacitor_SMD:C_1206_3216Metric; Note 3kV -> 1kV
- C82: renamed from C72; value 470p -> 1n; footprint Capacitor_SMD:C_0805_2012Metric -> Capacitor_SMD:C_1206_3216Metric; Note (none) -> 1kV
- C9: renamed from C5; footprint Capacitor_SMD:C_0805_2012Metric -> Capacitor_SMD:C_0603_1608Metric
- R30: renamed from R29; value R -> 10k
- R48: renamed from R47; footprint Resistor_SMD:R_0805_2012Metric -> Resistor_SMD:R_0603_1608Metric
- renumbered C10 to C12, C11 to C13, C12 to C16, C13 to C17, C14 to C18, C15 to C19, C16 to C20, C17 to C21, C1 to C29, C2 to C30, C25 to C33, C26 to C34, C27 to C35, C28 to C36, C29 to C37, C30 to C38, C31 to C39, C32 to C40, C33 to C41, C34 to C42, C35 to C43, C36 to C44, C37 to C45, C38 to C46, C39 to C47, C40 to C48, C41 to C49, C42 to C50, C43 to C51, C44 to C52, C45 to C53, C46 to C54, C47 to C55, C48 to C56, C49 to C57, C50 to C58, C51 to C59, C52 to C60, C53 to C61, C54 to C62, C55 to C63, C56 to C64, C57 to C65, C58 to C66, C69 to C67, C59 to C68, C60 to C69, C61 to C72, C62 to C73, C63 to C74, C64 to C75, C65 to C76, C66 to C77, C67 to C78, C68 to C79, J3 to J2, R80 to R19, R19 to R20, R20 to R21, R21 to R22, R22 to R23, R23 to R24, R24 to R25, R25 to R26, R26 to R27, R27 to R28, R28 to R29, R30 to R31, R31 to R32, R32 to R33, R33 to R34, R34 to R35, R35 to R36, R36 to R37, R37 to R38, R38 to R39, R39 to R40, R40 to R41, R41 to R42, R42 to R43, R43 to R44, R44 to R45, R45 to R46, R46 to R47, R48 to R49, R49 to R50, R50 to R51, R51 to R52, R52 to R53, R53 to R54, R54 to R55, R55 to R56, R56 to R57, R57 to R58, R58 to R59, R59 to R60, R60 to R61, R61 to R62, R62 to R63, R63 to R64, R64 to R65, R65 to R66, R66 to R67, R67 to R68, R68 to R69, R69 to R70, R70 to R71, R71 to R72, R72 to R73, R73 to R74, R74 to R75, R75 to R76, R76 to R77, R77 to R78, R78 to R79, R79 to R80, R93 to R81, R88 to R82, R89 to R83, R90 to R84, R91 to R85, R96 to R86, R92 to R89, R94 to R90, R95 to R91, R97 to R92, U24 to U21, U20 to U23, U21 to U24, U22 to U25, U23 to U26
Connections:
- net +3V3: now also C14.1, C15.1, C2.1, C3.1, C4.1, C5.1, C70.1, C71.1, U20.5 (VCC), U22.5 (V+), U27.5 (V+)
- net +5V: now also C32.1
- net +VDC: now also J6.1 (Pin_1)
- net DC+: now also J6.2 (Pin_2)
- net ENABLE_INPUTS: no longer U6.56 (PB4)
- net FOC_reset: no longer U6.21 (PA5)
- net GND: now also J11.21 (Pin_21), J11.23 (Pin_23), J11.25 (Pin_25), C14.2, C15.2, C2.2, C3.2, C32.2, C4.2, C5.2, C70.2, C71.2, R93.2, U20.3 (GND), U22.2 (V-), U27.2 (V-); no longer C33.2, C41.2, C49.2, C59.2, R15.2, R33.2, R49.2, R67.2, U15.3 (IN-), U15.4 (GND1), U2.3 (IN-), U2.4 (GND1), U4.3 (IN-), U4.4 (GND1), U9.3 (IN-), U9.4 (GND1)
- net IGBT_Temp: now also R88.1, U22.1; no longer U21.1, U21.4 (-)
- net Motor_temp: now also R94.1, U27.1; no longer U26.1, U26.4 (-)
- net TMC_CLK: now also U20.4; no longer U6.41 (PA8)
- net CAN_N: now reaches J1.1 (Pin_1), R12.2, U1.6 (CANL)
- net CAN_P: now reaches J1.2 (Pin_2), R12.1, U1.7 (CANH)
- net at R87.1: now also R88.2, U22.4 (-)
- net ERROR_HB1: no longer names the net of U6.59 (PB7)
- net ERROR_HB1: no longer J11.3 (Pin_3)
- net ERROR_HB2: no longer names the net of U6.61 (PB8)
- net ERROR_HB2: no longer J11.6 (Pin_6)
- net ERROR_HB3: no longer names the net of U6.62 (PB9)
- net ERROR_HB3: no longer J11.9 (Pin_9)
- net FOC_Status: no longer names the net of U6.58 (PB6)
- net FOC_Status: no longer U7.12 (STATUS)
- net IO0: no longer names the net of U6.42 (PA9)
- net IO1: no longer names the net of U6.43 (PA10)
- net IO2: no longer names the net of U6.50 (PA15)
- net IO3: no longer names the net of U6.37 (PC6)
- net IO4: no longer names the net of U6.30 (PB11)
- net SPI1_CS_Accel renamed SPI_CS_Accel
- net SPI1_CS_Gyro renamed SPI_CS_Gyro
- net SPI1_CS_Magnet renamed SPI_CS_Magnet
- net SPI2_MISO renamed SPI_MISO
- net SPI2_MOSI renamed SPI_MOSI
- net SPI2_NSS renamed SPI_CS_FOC
- net SPI2_SCK renamed SPI_SCK
- removed net VCC_CORE: C22.1, C23.1, C24.1, U7.15 (VCCCORE1), U7.45 (VCCCORE2), U7.63 (VCCCORE3)
- new net: U26.1, U26.4 (-), U27.3 (+)
- new net: U21.1, U21.4 (-), U22.3 (+)
- new net: R93.1, R94.2, U27.4 (-)
- new net 1V8_1: C22.1, U7.63 (VCCCORE3)
- new net 1V8_2: C23.1, U7.15 (VCCCORE1)
- new net 1V8_3: C24.1, U7.45 (VCCCORE2)
- new net GNDPWR: C33.2, C41.2, C49.2, C59.2, J3.1 (Pin_1), J3.2 (Pin_2), R15.2, R33.2, R49.2, R67.2, U15.3 (IN-), U15.4 (GND1), U2.3 (IN-), U2.4 (GND1), U4.3 (IN-), U4.4 (GND1), U9.3 (IN-), U9.4 (GND1)
- new net MCO_TMC_CLK: U20.2, U6.41 (PA8)
- no-connect marks 57 -> 69
Other:
- note removed: "Decoupling"
- note removed: "Decoupling\n"
- note removed: "LEDs"
- note removed: "RTC"
- note removed: "STATUS"
- moved on the sheet: C1, C11, C12, C13, C22, C23, C24, C25, C26, C29, C30, C31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
