File: hardware/motor_controller/logic_converter.sch (KiCad schematic (older format))
At the start: 3 parts, among them Q1 AO3401A

Commit message: IC connections added
Connections:
- net +24V renamed +15V
Changed lines of the file:
@@
 $Descr A4 11693 8268
 encoding utf-8
-Sheet 8 13
+Sheet 12 13
 Title ""
 Date ""
@@
 	1    0    0    -1
 $EndComp
-$Comp
-L power:+24V #PWR091
-U 1 1 5DE58E01
-P 6100 3900
-AR Path="/5DEDB0CD/5DE58E01" Ref="#PWR091"  Part="1"
-AR Path="/5DEE527A/5DE58E01" Ref="#PWR093"  Part="1"
-AR Path="/5DEF4ACC/5DE58E01" Ref="#PWR095"  Part="1"
-AR Path="/5DF13C30/5DE58E01" Ref="#PWR097"  Part="1"
-AR Path="/5DF13C34/5DE58E01" Ref="#PWR099"  Part="1"
-AR Path="/5DF13C38/5DE58E01" Ref="#PWR0101"  Part="1"
-F 0 "#PWR0101" H 6100 3750 50  0001 C CNN
-F 1 "+24V" H 6115 4073 50  0000 C CNN
-F 2 "" H 6100 3900 50  0001 C CNN
-F 3 "" H 6100 3900 50  0001 C CNN
-	1    6100 3900
-	1    0    0    -1
-$EndComp
 Text HLabel 5250 4350 0    50   Input ~ 0
 in
@@
 Wire Wire Line
 	6100 3900 6100 4000
+$Comp
+L power:+15V #PWR0113
+U 1 1 5DEB8F65
+P 6100 3900
+AR Path="/5DF13C38/5DEB8F65" Ref="#PWR0113"  Part="1"
+AR Path="/5DF13C34/5DEB8F65" Ref="#PWR0112"  Part="1"
+AR Path="/5DEDB0CD/5DEB8F65" Ref="#PWR0108"  Part="1"
+AR Path="/5DEE527A/5DEB8F65" Ref="#PWR0109"  Part="1"
+AR Path="/5DEF4ACC/5DEB8F65" Ref="#PWR0110"  Part="1"
+AR Path="/5DF13C30/5DEB8F65" Ref="#PWR0111"  Part="1"
+F 0 "#PWR0113" H 6100 3750 50  0001 C CNN
+F 1 "+15V" H 6115 4073 50  0000 C CNN
+F 2 "" H 6100 3900 50  0001 C CNN
+F 3 "" H 6100 3900 50  0001 C CNN
+	1    6100 3900
+	1    0    0    -1
+$EndComp
 $EndSCHEMATC

Commit message: SD Card and other pins
Parts:
- renumbered R36 to R40, R37 to R41
Changed lines of the file:
@@
 EESchema Schematic File Version 4
-LIBS:electric-FIAT-cache
 EELAYER 30 0
 EELAYER END
@@
 $EndComp
 $Comp
-L Device:R R36
+L Device:R R40
 U 1 1 5DE572D3
 P 5400 4150
-AR Path="/5DEDB0CD/5DE572D3" Ref="R36"  Part="1"
-AR Path="/5DEE527A/5DE572D3" Ref="R38"  Part="1"
-AR Path="/5DEF4ACC/5DE572D3" Ref="R40"  Part="1"
-AR Path="/5DF13C30/5DE572D3" Ref="R42"  Part="1"
-AR Path="/5DF13C34/5DE572D3" Ref="R44"  Part="1"
-AR Path="/5DF13C38/5DE572D3" Ref="R46"  Part="1"
-F 0 "R46" H 5470 4196 50  0000 L CNN
+AR Path="/5DEDB0CD/5DE572D3" Ref="R40"  Part="1"
+AR Path="/5DEE527A/5DE572D3" Ref="R42"  Part="1"
+AR Path="/5DEF4ACC/5DE572D3" Ref="R44"  Part="1"
+AR Path="/5DF13C30/5DE572D3" Ref="R46"  Part="1"
+AR Path="/5DF13C34/5DE572D3" Ref="R48"  Part="1"
+AR Path="/5DF13C38/5DE572D3" Ref="R50"  Part="1"
+F 0 "R50" H 5470 4196 50  0000 L CNN
 F 1 "1k" H 5470 4105 50  0000 L CNN
 F 2 "" V 5330 4150 50  0001 C CNN
@@
 $EndComp
 $Comp
-L Device:R R37
+L Device:R R41
 U 1 1 5DE58624
 P 6100 4150
-AR Path="/5DEDB0CD/5DE58624" Ref="R37"  Part="1"
-AR Path="/5DEE527A/5DE58624" Ref="R39"  Part="1"
-AR Path="/5DEF4ACC/5DE58624" Ref="R41"  Part="1"
-AR Path="/5DF13C30/5DE58624" Ref="R43"  Part="1"
-AR Path="/5DF13C34/5DE58624" Ref="R45"  Part="1"
-AR Path="/5DF13C38/5DE58624" Ref="R47"  Part="1"
-F 0 "R47" H 6170 4196 50  0000 L CNN
+AR Path="/5DEDB0CD/5DE58624" Ref="R41"  Part="1"
+AR Path="/5DEE527A/5DE58624" Ref="R43"  Part="1"
+AR Path="/5DEF4ACC/5DE58624" Ref="R45"  Part="1"
+AR Path="/5DF13C30/5DE58624" Ref="R47"  Part="1"
+AR Path="/5DF13C34/5DE58624" Ref="R49"  Part="1"
+AR Path="/5DF13C38/5DE58624" Ref="R51"  Part="1"
+F 0 "R51" H 6170 4196 50  0000 L CNN
 F 1 "1k" H 6170 4105 50  0000 L CNN
 F 2 "" V 6030 4150 50  0001 C CNN
@@
 $EndComp
 $Comp
-L power:+3.3V #PWR090
+L power:+3.3V #PWR0108
 U 1 1 5DE587FC
 P 5400 3900
-AR Path="/5DEDB0CD/5DE587FC" Ref="#PWR090"  Part="1"
-AR Path="/5DEE527A/5DE587FC" Ref="#PWR092"  Part="1"
-AR Path="/5DEF4ACC/5DE587FC" Ref="#PWR094"  Part="1"
-AR Path="/5DF13C30/5DE587FC" Ref="#PWR096"  Part="1"
-AR Path="/5DF13C34/5DE587FC" Ref="#PWR098"  Part="1"
-AR Path="/5DF13C38/5DE587FC" Ref="#PWR0100"  Part="1"
-F 0 "#PWR0100" H 5400 3750 50  0001 C CNN
+AR Path="/5DEDB0CD/5DE587FC" Ref="#PWR0108"  Part="1"
+AR Path="/5DEE527A/5DE587FC" Ref="#PWR0110"  Part="1"
+AR Path="/5DEF4ACC/5DE587FC" Ref="#PWR0112"  Part="1"
+AR Path="/5DF13C30/5DE587FC" Ref="#PWR0114"  Part="1"
+AR Path="/5DF13C34/5DE587FC" Ref="#PWR0116"  Part="1"
+AR Path="/5DF13C38/5DE587FC" Ref="#PWR0118"  Part="1"
+F 0 "#PWR0118" H 5400 3750 50  0001 C CNN
 F 1 "+3.3V" H 5415 4073 50  0000 C CNN
 F 2 "" H 5400 3900 50  0001 C CNN
@@
 	6100 3900 6100 4000
 $Comp
-L power:+15V #PWR0113
+L power:+15V #PWR0119
 U 1 1 5DEB8F65
 P 6100 3900
-AR Path="/5DF13C38/5DEB8F65" Ref="#PWR0113"  Part="1"
-AR Path="/5DF13C34/5DEB8F65" Ref="#PWR0112"  Part="1"
-AR Path="/5DEDB0CD/5DEB8F65" Ref="#PWR0108"  Part="1"
-AR Path="/5DEE527A/5DEB8F65" Ref="#PWR0109"  Part="1"
-AR Path="/5DEF4ACC/5DEB8F65" Ref="#PWR0110"  Part="1"
-AR Path="/5DF13C30/5DEB8F65" Ref="#PWR0111"  Part="1"
-F 0 "#PWR0113" H 6100 3750 50  0001 C CNN
+AR Path="/5DF13C38/5DEB8F65" Ref="#PWR0119"  Part="1"
+AR Path="/5DF13C34/5DEB8F65" Ref="#PWR0117"  Part="1"
+AR Path="/5DEDB0CD/5DEB8F65" Ref="#PWR0109"  Part="1"
+AR Path="/5DEE527A/5DEB8F65" Ref="#PWR0111"  Part="1"
+AR Path="/5DEF4ACC/5DEB8F65" Ref="#PWR0113"  Part="1"
+AR Path="/5DF13C30/5DEB8F65" Ref="#PWR0115"  Part="1"
+F 0 "#PWR0119" H 6100 3750 50  0001 C CNN
 F 1 "+15V" H 6115 4073 50  0000 C CNN
 F 2 "" H 6100 3900 50  0001 C CNN
