File: hardware/motor_controller/electric-FIAT.kicad_pcb (KiCad board)
At the start: 2 copper layers, 182 parts, among them J1 Conn_01x02_Male, J10 SKiiP 613 GD123-3DUL V3, J11 Acc_sensor, J2 Program/Debug, J3 Micro_SD_Card_Det, J4 RTMI, J5 Batt_conn, J7 IMU, Q1 AO3400, Q2 AO3400, Q3 AO3400, Q4 AO3400, Q5 AO3400, Q6 AO3400, U10 ACPL-C87A, U11 OPA356xxDBV, U12 ACS759xCB-200B-PFF, U13 ACS759xCB-200B-PFF, U14 ACPL-C87A, U15 OPA356xxDBV, U16 ACS759xCB-200B-PFF, U17 OPA356xxDBV, U18 OPA356xxDBV, U19 TEN40-1215E, U2 MCP2562-E-SN, U3 ACPL-C87A, U4 OPA356xxDBV, U5 ACPL-C87A, U6 OPA356xxDBV, U7 STM32F405RGTx, U8 ACS759xCB-200B-PFF, U9 TMC4671-ES, Y1 32.768MHz, Y2 25MHz

Commit message: Encoder and 1.8V Supply - Schematic v0.9.1
Parts:
- moved J5 2.43 mm to (114.4, 144.7)
- moved U8 0.18 mm to (125.9, 108.0)
Routing:
- net Net-(J5-Pad2): track 13.0 -> 0.00 mm
- net +BATT: track 13.0 -> 0.00 mm
Changed lines of the file:
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@@
   (general
     (thickness 1.6)
-    (drawings 2)
-    (tracks 4)
+    (drawings 0)
+    (tracks 0)
     (zones 0)
     (modules 182)
@@
   )
   (module fiat:Battery (layer F.Cu)
-    (at 114.3 142.24)
+    (at 114.38 144.67)
     (fp_text reference J5 (at 0 0.5) (layer F.SilkS)
       (effects (font (size 1 1) (thickness 0.15)))
@@
       (effects (font (size 1 1) (thickness 0.15)))
     )
-    (pad 3 smd rect (at 34.29 -1.27) (size 15 15) (layers F.Cu F.Paste F.Mask)
+    (pad 3 thru_hole rect (at 41.91 -1.27) (size 20 20) (drill 5.3) (layers *.Cu *.Mask)
       (net 1 GND) (clearance 0.5))
-    (pad 2 smd rect (at 17.78 -1.27) (size 15 15) (layers F.Cu F.Paste F.Mask)
+    (pad 2 thru_hole rect (at 20.32 -1.27) (size 20 20) (drill 5.3) (layers *.Cu *.Mask)
       (net 211 "Net-(J5-Pad2)") (clearance 0.5))
-    (pad 1 smd rect (at 1.27 -1.27) (size 15 15) (layers F.Cu F.Paste F.Mask)
+    (pad 1 thru_hole rect (at -1.27 -1.27) (size 20 20) (drill 5.3) (layers *.Cu *.Mask)
       (net 100 +BATT) (clearance 0.5) (zone_connect 0))
   )
@@
   )
   (module Sensor_Current:Allegro_CB_PFF (layer F.Cu)
-    (at 125.73 107.95 180)
+    (at 125.9 108 180)
     (descr "Allegro MicroSystems, CB-PFF Package (http://www.allegromicro.com/en/Products/Current-Sensor-ICs/Fifty-To-Two-Hundred-Amp-Integrated-Conductor-Sensor-ICs/ACS758.aspx) !PADS 4-5 DO NOT MATCH DATASHEET!")
     (tags "Allegro CB-PFF")
@@
     )
   )
-  (gr_poly (pts (xy 139.6 138.5) (xy 124.6 138.5) (xy 124.6 126) (xy 139.6 126)) (layer F.Cu) (width 0.1))
-  (gr_poly (pts (xy 123 138) (xy 108 138) (xy 108 126) (xy 123 126)) (layer F.Cu) (width 0.1))
-  (segment (start 118.82 137.72) (end 115.57 140.97) (width 0.25) (layer F.Cu) (net 100))
-  (segment (start 118.82 129.35) (end 118.82 137.72) (width 0.25) (layer F.Cu) (net 100))
-  (segment (start 128.82 137.71) (end 132.08 140.97) (width 0.25) (layer F.Cu) (net 211))
-  (segment (start 128.82 129.35) (end 128.82 137.71) (width 0.25) (layer F.Cu) (net 211))
 )

Commit message: Schematic v0.11.0
Parts:
- removed C56: 2.2n, Capacitor_SMD:C_0805_2012Metric
- removed PS1: ITX1205SA, Converter_DCDC:Converter_DCDC_XP_POWER-ITXxxxxSA_THT
- removed PS2: IU1203SA, Converter_DCDC:Converter_DCDC_XP_POWER-ITXxxxxSA_THT
- added C55: 10u, Capacitor_SMD:C_0805_2012Metric, F.Cu at (151.9, 134.2)
- added C58: 270u, Capacitor_THT:CP_Radial_D10.0mm_P5.00mm, F.Cu at (155.7, 118.1)
- added C59: 680p, Capacitor_SMD:C_0805_2012Metric, F.Cu at (202.1, 87.8)
- added C60: 10u, Capacitor_SMD:C_0805_2012Metric, F.Cu at (213.3, 76.3)
- added C61: 2.2n, Capacitor_SMD:C_0805_2012Metric, F.Cu at (186.8, 102.8)
- added C62: 2.2n, Capacitor_SMD:C_0805_2012Metric, F.Cu at (164.1, 125.4)
- added C65: 470p, Capacitor_SMD:C_0805_2012Metric, F.Cu at (170.5, 118.7)
- added C66: 50p, Capacitor_SMD:C_0805_2012Metric, F.Cu at (225.2, 63.9)
- added C67: 50p, Capacitor_SMD:C_0805_2012Metric, F.Cu at (166.1, 121.6)
- added C68: 100p, Capacitor_SMD:C_0805_2012Metric, F.Cu at (193.3, 95.4)
- added J12: Acc_sensor, Connector_Phoenix_MC_HighVoltage:PhoenixContact_MCV_1,5_2-G-5.08_1x02_P5.08mm_Vertical, F.Cu at (214.8, 53.8)
- added J13: 12V Battery, Connector_Phoenix_MC_HighVoltage:PhoenixContact_MCV_1,5_2-G-5.08_1x02_P5.08mm_Vertical, F.Cu at (167.2, 104.4)
- added J6: Motor_U, fiat:Motor_IGBT, F.Cu at (87.9, 94.7)
- added J8: Motor_V, fiat:Motor_IGBT, F.Cu at (77.0, 129.0)
- added J9: Motor_W, fiat:Motor_IGBT, F.Cu at (87.9, 73.7)
- added L1: 4.7u, Inductor_SMD:L_Coilcraft_LPS4018, F.Cu at (183.5, 76.8)
- added L2: 6.8u, Inductor_SMD:L_Coilcraft_LPS4018, F.Cu at (126.3, 64.7)
- added Pedal_Sensor1: 5.1k, Connector_Phoenix_MC_HighVoltage:PhoenixContact_MCV_1,5_2-G-5.08_1x02_P5.08mm_Vertical, F.Cu at (205.5, 68.0)
- added R88: 1.8k, Resistor_SMD:R_0805_2012Metric, F.Cu at (168.5, 130.5)
- added R89: 1k, Resistor_SMD:R_0805_2012Metric, F.Cu at (165.1, 134.2)
- added R90: 1k, Resistor_SMD:R_0805_2012Metric, F.Cu at (222.1, 76.9)
- added R91: 3.3k, Resistor_SMD:R_0805_2012Metric, F.Cu at (217.7, 81.9)
- added R92: 1k, Resistor_SMD:R_0805_2012Metric, F.Cu at (200.1, 99.6)
- added R93: 180, Resistor_SMD:R_0805_2012Metric, F.Cu at (188.2, 111.7)
- added U1: 74LVC1GU04DRL, Package_TO_SOT_SMD:SOT-553, F.Cu at (150.4, 114.0)
- added U20: IU1203SA, fiat:Converter_DCDC_XP_POWER-IUxxxxSA_THT, F.Cu at (171.7, 70.7)
- added U21: TEN40-1215E, fiat:Converter_DCDC_TRACO_TEN40-xxxxE, F.Cu at (147.7, 63.1)
- added U22: SR05S1V8, fiat:Converter_DCDC_XP_POWER-SRxxSx_THT, F.Cu at (144.8, 94.9)
- added U23: 74LVC1G14, fiat:Texas_R-PDSO-G5, F.Cu at (204.4, 100.4)
- added U24: 74LVC1G14, fiat:Texas_R-PDSO-G5, F.Cu at (230.8, 76.2)
- added U25: 74LVC1G14, fiat:Texas_R-PDSO-G5, F.Cu at (181.7, 124.5)
- C10: value 100n -> 2.2n
- C11: value 1u -> 2.2n
- C12, C18, C48: value 1n -> 100n
- C13: value 100n -> 1u
- C14, C36, C43, C47: value 100n -> 1n
- C15, C16: value 30p -> 100n
- C17: value 10n -> 100n
- C19, C26, C30, C40: value 100p -> 100n
- C20, C21: value 100n -> 30p
- C22: value 100p -> 10n
- C23, C29: value 100p -> 1n
- C24, C31, C38: value 1n -> 100p
- C27, C28, C34, C45, C46: value 100n -> 100p
- C42: value 1n -> 50p
- C49, C51: value 10u -> 100n
- C50: value 270u -> 100n; footprint Capacitor_THT:CP_Radial_D10.0mm_P5.00mm -> Capacitor_SMD:C_0805_2012Metric
- C52: value 680p -> 100n
- C53: value 10u -> 1n
- C57: value 470p -> 10u
- C6, C7: value 2.2n -> 100n
- J1: footprint Connector_Phoenix_MSTB:PhoenixContact_MSTBVA_2,5_2-G-5,08_1x02_P5.08mm_Vertical -> Connector_Phoenix_MC_HighVoltage:PhoenixContact_MCV_1,5_2-G-5.08_1x02_P5.08mm_Vertical
- J10: value SKiiP 613 GD123-3DUL V3 -> IMU; footprint Connector_IDC:IDC-Header_2x13_P2.54mm_Vertical_Lock -> Connector_PinSocket_2.54mm:PinSocket_1x10_P2.54mm_Vertical
- J11: value Acc_sensor -> SKiiP 613 GD123-3DUL V3; footprint Connector_Phoenix_MC_HighVoltage:PhoenixContact_MCV_1,5_2-G-5.08_1x02_P5.08mm_Vertical -> Connector_IDC:IDC-Header_2x13_P2.54mm_Vertical_Lock
- J3: value Micro_SD_Card_Det -> RTMI; footprint Connector_Card:microSD_HC_Hirose_DM3D-SF -> Connector_PinHeader_2.54mm:PinHeader_2x05_P2.54mm_Vertical
- J4: value RTMI -> Micro_SD_Card_Det; footprint Connector_PinHeader_2.54mm:PinHeader_2x05_P2.54mm_Vertical -> Connector_Card:microSD_HC_Hirose_DM3D-SF
- J7: value IMU -> Encoder; footprint Connector_PinSocket_2.54mm:PinSocket_1x10_P2.54mm_Vertical -> Connector_PinHeader_2.54mm:PinHeader_1x04_P2.54mm_Vertical
- JP1: value Clock Source -> Clock Selection
- R22: value 200k -> 10k
- R31: value 10k -> 200k
- R54, R55: value 200k -> 4.7k
- R63: value 4.7k -> 200k
- R64: value 1k -> 200k
- R65, R66: value 1k -> 100
- R67: value 1k -> 4.7k
- R68, R69: value 10k -> 390
- R70, R71: value 10k -> 1k
- R74, R75, R77: value 1k -> 10k
- R76: value 4.7k -> 10k
- R81: value 2.7k -> 1k
- R82: value 1.8k -> 4.7k
- R85: value 3.3k -> 1k
- R87: value 180 -> 2.7k
- TH1, TH2: footprint TerminalBlock_RND:TerminalBlock_RND_205-00012_1x02_P5.00mm_Horizontal -> Connector_Phoenix_MC_HighVoltage:PhoenixContact_MCV_1,5_2-G-5.08_1x02_P5.08mm_Vertical
- U19: value TEN40-1215E -> ITW1205SA; footprint fiat:Converter_DCDC_TRACO_TEN40-xxxxE -> fiat:Converter_DCDC_XP_POWER-ITWxxxxSA_THT
- U8: value ACS759xCB-200B-PFF -> TMC4671-ES; footprint Sensor_Current:Allegro_CB_PFF -> fiat:QFN76P
- U9: value TMC4671-ES -> ACS759xCB-200B-PFF; footprint trinamic:TMC4671-ES -> Sensor_Current:Allegro_CB_PFF
- moved C8 188.1 mm to (114.4, 136.8)
- moved U7 182.6 mm to (115.0, 128.1)
- moved TH1 175.9 mm to (140.0, 129.9)
- moved Q2 175.6 mm to (150.8, 126.8)
- moved C52 173.2 mm to (150.8, 130.5)
- moved C51 164.1 mm to (155.3, 128.3)
- moved Q6 158.8 mm to (121.0, 91.7)
- moved C15 158.5 mm to (166.1, 112.8)
- moved R31 156.2 mm to (159.7, 131.3)
- moved J11 154.8 mm to (69.8, 74.4)
- moved R42 152.2 mm to (169.5, 133.4)
- moved R22 146.9 mm to (170.5, 121.6)
- moved R70 139.1 mm to (156.3, 134.2)
- moved C9 135.7 mm to (143.0, 135.3)
- moved C34 135.6 mm to (183.8, 117.6)
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Connections:
- C10 pad 1: +3V3 -> /VCAP_1
- C11 pad 1: +3V3 -> /VCAP_2
- C12 pad 1: Net-(C12-Pad1) -> +3V3
- C12 pad 2: /DC_Bus_Voltage -> GND
- C13 pad 1: +5V -> +3V3
- C14 pad 1: +3V3 -> Net-(C14-Pad1)
- C14 pad 2: GND -> /DC_Bus_Voltage
- C15 pad 1: /HSE_IN -> +5V
- C16 pad 1: /HSE_OUT -> +3V3
- C17 pad 1: Net-(C17-Pad1) -> /VCC_CORE
- C18 pad 1: Net-(C12-Pad1) -> /VCC_CORE
- C19 pad 1: Net-(C19-Pad1) -> /VCC_CORE
- C19 pad 2: /Motor_Voltage_U -> GND
- C20 pad 1: +5V -> /HSE_IN
- C21 pad 1: +3V3 -> /HSE_OUT
- C23 pad 1: Net-(C19-Pad1) -> Net-(C14-Pad1)
- C24 pad 1: /DC_Current -> Net-(C24-Pad1)
- C24 pad 2: GND -> /Motor_Voltage_U
- C25 pad 1: +3V3 -> +5V
- C26 pad 1: Net-(C26-Pad1) -> +3V3
- C26 pad 2: /Motor_Voltage_V -> GND
- C27 pad 1: +5V -> Net-(C27-Pad1)
- C28 pad 1: +3V3 -> Net-(C24-Pad1)
- C29 pad 1: Net-(C29-Pad1) -> /DC_Current
- C30 pad 1: Net-(C26-Pad1) -> +3V3
- C31 pad 1: /Motor_Current_U -> Net-(C31-Pad1)
- C31 pad 2: GND -> /Motor_Voltage_V
- C32 pad 1: +3V3 -> +5V
- C34 pad 1: +5V -> Net-(C34-Pad1)
- C35 pad 1: Net-(C35-Pad1) -> Net-(C31-Pad1)
- C35 pad 2: /Motor_Voltage_W -> GND
- C36 pad 1: +5V -> /Motor_Current_U
- C38 pad 1: /Motor_Current_V -> Net-(C38-Pad1)
- C38 pad 2: GND -> /Motor_Voltage_W
- C39 pad 1: +3V3 -> +5V
- C40 pad 1: Net-(C40-Pad1) -> +3V3
- C41 pad 1: Net-(C35-Pad1) -> /ENC_A
- C42 pad 1: /Motor_Current_W -> /ENC_A_T
- C43 pad 1: +3V3 -> /Motor_Current_V
- C45 pad 1: +3V3 -> Net-(C45-Pad1)
- C46 pad 1: +1V8 -> Net-(C38-Pad1)
- C47 pad 1: +1V8 -> /Motor_Current_W
- C48 pad 1: +12V -> +3V3
- C48 pad 2: Net-(C48-Pad2) -> GND
- C49 pad 1: +5V -> +3V3
- C49 pad 2: Net-(C49-Pad2) -> GND
- C50 pad 1: +12V -> +3V3
- C51 pad 1: +12V -> +1V8
- C52 pad 1: +12V -> +1V8
- C52 pad 2: Net-(C52-Pad2) -> GND
- C53 pad 1: +12V -> +BATT
- C53 pad 2: GND -> +24V
- C54 pad 1: +3V3 -> +5V
- C57 pad 1: GND -> +BATT
- C57 pad 2: Net-(C52-Pad2) -> -BATT
- C6 pad 1: /VCAP_1 -> +3V3
- C7 pad 1: /VCAP_2 -> +5V
- J10 pad 1: GND -> +3V3
- J10 pad 10: /PWM_WY1_H_15V -> /SPI1_CS_Magnet
- J10 pad 2: /PWM_UX1_L_15V -> GND
- J10 pad 3: /ERROR_HB1 -> /SPI2_SCK
- J10 pad 4: /PWM_UX1_H_15V -> /SPI2_MOSI
- J10 pad 5: /PWM_VX2_L_15V -> GND
- J10 pad 6: /ERROR_HB2 -> /SPI2_MISO
- J10 pad 7: /PWM_VX2_H_15V -> /SPI2_MISO
- J10 pad 8: /PWM_WY1_L_15V -> /SPI1_CS_Accel
- J10 pad 9: /ERROR_HB3 -> /SPI1_CS_Gyro
- J11 pad 1: /accelerator_pedal -> GND
- J11 pad 2: GND -> /HB_UB
- J3 pad 1: /SD_DAT2 -> +3V3
- J3 pad 10: +3V3 -> GND
- J3 pad 2: /SD_DAT3 -> (no net)
- J3 pad 3: /SD_CMD -> /DBGSPI_nSCS
- J3 pad 4: +3V3 -> /DBGSPI_TRG
- J3 pad 5: /SD_CLK -> /DBGSPI_SCK
- J3 pad 7: /SD_DAT0 -> /DBGSPI_MOSI
- J3 pad 8: /SD_DAT1 -> GND
- J3 pad 9: /SD_DET -> /DBGSPI_MISO
- J4 pad 1: +3V3 -> /SD_DAT2
- J4 pad 10: GND -> +3V3
- J4 pad 2: /GPIO0 -> /SD_DAT3
- J4 pad 3: /DBGSPI_nSCS -> /SD_CMD
- J4 pad 4: /GPIO1 -> +3V3
- J4 pad 5: /DBGSPI_SCK -> /SD_CLK
- J4 pad 7: /DBGSPI_MOSI -> /SD_DAT0
- J4 pad 8: GND -> /SD_DAT1
- J4 pad 9: /DBGSPI_MISO -> /SD_DET
- J5 pad 1: +BATT -> +VDC
- J7 pad 1: +3V3 -> +5V
- J7 pad 2: GND -> /ENC_A_R
- J7 pad 3: /SPI2_SCK -> /ENC_B_R
- J7 pad 4: /SPI2_MOSI -> GND
- JP1 pad 1: /MCU_25MHZ -> /Crystal_25MHZ
- JP1 pad 3: /Crystal_25MHZ -> /MCU_MCO
- Q1 pad 2: /PWM_VX2_L_3V3 -> /PWM_VT
- Q1 pad 3: /PWM_VX2_L_15V -> /HB_VT
- Q2 pad 2: /PWM_UX1_H_3V3 -> /PWM_VB
- Q2 pad 3: /PWM_UX1_H_15V -> /HB_VB
- Q3 pad 2: /PWM_WY1_H_3V3 -> /PWM_UT
- Q3 pad 3: /PWM_WY1_H_15V -> /HB_UT
- Q4 pad 2: /PWM_UX1_L_3V3 -> /PWM_UB
- Q4 pad 3: /PWM_UX1_L_15V -> /HB_UB
- Q5 pad 2: /PWM_WY1_L_3V3 -> /PWM_WT
- Q5 pad 3: /PWM_WY1_L_15V -> /HB_WT
- Q6 pad 2: /PWM_VX2_H_3V3 -> /PWM_WB
- Q6 pad 3: /PWM_VX2_H_15V -> /HB_WB
- R1 pad 1: /Crystal_25MHZ -> Net-(R1-Pad1)
- R15 pad 1: Net-(C17-Pad1) -> Net-(C22-Pad1)
- R18 pad 2: Net-(C12-Pad1) -> Net-(C14-Pad1)
- R2 pad 1: Net-(C12-Pad1) -> Net-(C14-Pad1)
- R20 pad 1: Net-(C12-Pad1) -> Net-(C14-Pad1)
- R21 pad 1: Net-(C19-Pad1) -> +3V3
- R21 pad 2: /Motor_Voltage_U -> /reset
- R22 pad 1: Net-(R22-Pad1) -> Net-(C24-Pad1)
- R22 pad 2: Net-(C22-Pad1) -> /Motor_Voltage_U
- R23 pad 1: Net-(R22-Pad1) -> Net-(R23-Pad1)
- R23 pad 2: Net-(R23-Pad2) -> Net-(C27-Pad1)
- R24 pad 1: Net-(R24-Pad1) -> Net-(R23-Pad1)
- R24 pad 2: Net-(R23-Pad2) -> Net-(R24-Pad2)
- R25 pad 1: Net-(R24-Pad1) -> Net-(R25-Pad1)
- R25 pad 2: Net-(R25-Pad2) -> Net-(R24-Pad2)
- R26 pad 1: Net-(R26-Pad1) -> Net-(R25-Pad1)
- R26 pad 2: Net-(R25-Pad2) -> Net-(R26-Pad2)
- R27 pad 1: Net-(R26-Pad1) -> Net-(R27-Pad1)
- R27 pad 2: Net-(R27-Pad2) -> Net-(R26-Pad2)
- R28 pad 1: Net-(R28-Pad1) -> Net-(R27-Pad1)
- R28 pad 2: Net-(R27-Pad2) -> Net-(R28-Pad2)
- R29 pad 1: Net-(R28-Pad1) -> Net-(R29-Pad1)
- R29 pad 2: Net-(R29-Pad2) -> Net-(R28-Pad2)
- R3 pad 1: /Crystal_25MHZ -> Net-(R1-Pad1)
- R30 pad 1: /Motor_U -> Net-(R29-Pad1)
- R30 pad 2: Net-(R29-Pad2) -> Net-(R30-Pad2)
- R31 pad 1: /SD_DET -> /Motor_U
- R31 pad 2: GND -> Net-(R30-Pad2)
- R32 pad 1: /reset -> /SD_DET
- R34 pad 1: Net-(C22-Pad1) -> Net-(C27-Pad1)
- R35 pad 2: Net-(C19-Pad1) -> Net-(C24-Pad1)
- R36 pad 1: Net-(C19-Pad1) -> Net-(C24-Pad1)
- R37 pad 1: Net-(C26-Pad1) -> Net-(C31-Pad1)
- R39 pad 2: Net-(R39-Pad2) -> Net-(C34-Pad1)
- R49 pad 1: Net-(C29-Pad1) -> Net-(C34-Pad1)
- R50 pad 2: Net-(C26-Pad1) -> Net-(C31-Pad1)
- R52 pad 1: Net-(C26-Pad1) -> Net-(C31-Pad1)
- R53 pad 1: Net-(C35-Pad1) -> Net-(C38-Pad1)
- R54 pad 1: Net-(R54-Pad1) -> +5V
- R54 pad 2: Net-(R54-Pad2) -> /ENC_A_R
- R55 pad 1: Net-(R54-Pad1) -> +5V
- R55 pad 2: Net-(R55-Pad2) -> /ENC_B_R
- R56 pad 2: Net-(R55-Pad2) -> Net-(C45-Pad1)
- R62 pad 1: /Motor_W -> Net-(R62-Pad1)
- R63 pad 1: /Motor_Current_V -> Net-(R62-Pad1)
- R64 pad 1: +3V3 -> /Motor_W
- R64 pad 2: /PWM_VX2_L_3V3 -> Net-(R63-Pad2)
- R65 pad 1: +15V -> /ENC_A
- R65 pad 2: /PWM_VX2_L_15V -> /ENC_A_R
- R66 pad 1: +3V3 -> /ENC_B
- R66 pad 2: /PWM_UX1_H_3V3 -> /ENC_B_R
- R67 pad 1: +15V -> /Motor_Current_V
- R67 pad 2: /PWM_UX1_H_15V -> Net-(R67-Pad2)
- R68 pad 1: Net-(R68-Pad1) -> /ENC_A
- R68 pad 2: Net-(R68-Pad2) -> GND
- R69 pad 1: Net-(C40-Pad1) -> /ENC_B
- R70 pad 1: Net-(R70-Pad1) -> +3V3
- R70 pad 2: Net-(C35-Pad1) -> /PWM_VT
- R71 pad 1: Net-(C35-Pad1) -> +15V
- R71 pad 2: GND -> /HB_VT
- R72 pad 2: /PWM_WY1_H_3V3 -> /PWM_VB
- R73 pad 2: /PWM_WY1_H_15V -> /HB_VB
- R74 pad 1: +3V3 -> Net-(R74-Pad1)
- R74 pad 2: /PWM_UX1_L_3V3 -> Net-(R74-Pad2)
- R75 pad 1: +15V -> Net-(C45-Pad1)
- R75 pad 2: /PWM_UX1_L_15V -> GND
- R76 pad 1: /Motor_Current_W -> Net-(R76-Pad1)
- R76 pad 2: Net-(R76-Pad2) -> Net-(C38-Pad1)
- R77 pad 1: +3V3 -> Net-(C38-Pad1)
- R77 pad 2: /PWM_WY1_L_3V3 -> GND
- R78 pad 1: +15V -> +3V3
- R78 pad 2: /PWM_WY1_L_15V -> /PWM_UT
- R79 pad 1: +3V3 -> +15V
- R79 pad 2: /PWM_VX2_H_3V3 -> /HB_UT
- R80 pad 1: +15V -> +3V3
- R80 pad 2: /PWM_VX2_H_15V -> /PWM_UB
- R81 pad 1: Net-(R81-Pad1) -> +15V
- R81 pad 2: GND -> /HB_UB
- R82 pad 1: Net-(R82-Pad1) -> /Motor_Current_W
- R82 pad 2: GND -> Net-(R82-Pad2)
- R83 pad 2: Net-(Pedal_Sensor1-Pad1) -> /PWM_WT
- R84 pad 1: Net-(R84-Pad1) -> +15V
- R84 pad 2: +1V8 -> /HB_WT
- R85 pad 1: /Motor_temp -> +3V3
- R85 pad 2: Net-(R84-Pad1) -> /PWM_WB
- R86 pad 1: Net-(R86-Pad1) -> +15V
- R86 pad 2: +1V8 -> /HB_WB
- R87 pad 1: /Inverter_temp -> Net-(R87-Pad1)
- R87 pad 2: Net-(R86-Pad1) -> GND
- TH1 pad 2: Net-(R81-Pad1) -> Net-(R87-Pad1)
- TH2 pad 2: Net-(R82-Pad1) -> Net-(R88-Pad1)
- U10 pad 2: Net-(C29-Pad1) -> Net-(C34-Pad1)
- U11 pad 4: Net-(C26-Pad1) -> Net-(C31-Pad1)
- U12 pad 4: /IGBT_W -> /IGBT_U
- U12 pad 5: /Motor_W -> /Motor_U
- U13 pad 3: Net-(R63-Pad2) -> Net-(R67-Pad2)
- U14 pad 2: Net-(C40-Pad1) -> Net-(C45-Pad1)
- U14 pad 6: Net-(R70-Pad1) -> Net-(R76-Pad1)
- U14 pad 7: Net-(R68-Pad2) -> Net-(R74-Pad2)
- U15 pad 3: Net-(R68-Pad1) -> Net-(R74-Pad1)
- U15 pad 4: Net-(C35-Pad1) -> Net-(C38-Pad1)
- U16 pad 3: Net-(R76-Pad2) -> Net-(R82-Pad2)
- U17 pad 3: Net-(R81-Pad1) -> Net-(R87-Pad1)
- U17 pad 4: Net-(R84-Pad1) -> Net-(R90-Pad1)
- U18 pad 3: Net-(R82-Pad1) -> Net-(R88-Pad1)
- U18 pad 4: Net-(R86-Pad1) -> Net-(R92-Pad1)
- U19 pad 1: +12V -> -BATT
- U19 pad 2: GND -> Net-(L1-Pad2)
- U19 pad 4: Net-(C48-Pad2) -> +5V
- U19 pad 5: Net-(C52-Pad2) -> (no net)
- U19 pad 6: Net-(U19-Pad6) -> GND
- U3 pad 2: Net-(C17-Pad1) -> Net-(C22-Pad1)
- U4 pad 4: Net-(C12-Pad1) -> Net-(C14-Pad1)
- U5 pad 2: Net-(C22-Pad1) -> Net-(C27-Pad1)
- U6 pad 4: Net-(C19-Pad1) -> Net-(C24-Pad1)
- U7 pad 1: Net-(U7-Pad1) -> (no net)
- U7 pad 14: /Motor_Current_U -> /ENC_A_T
- U7 pad 15: /Motor_Current_V -> /ENC_B_T
- U7 pad 2: /IGBT_TEMP_ERROR -> /IGBT_OVER_TEMP
- U7 pad 30: Net-(U7-Pad30) -> (no net)
- U7 pad 37: Net-(U7-Pad37) -> (no net)
- U7 pad 41: /MCU_25MHZ -> /MCU_MCO
- U7 pad 42: Net-(U7-Pad42) -> (no net)
- U7 pad 43: Net-(U7-Pad43) -> (no net)
- U7 pad 50: Net-(U7-Pad50) -> (no net)
- U7 pad 8: /ENCODER_VA -> /Motor_Current_U
- U7 pad 9: /ENCODER_VB -> /Motor_Current_V
- U8 pad 1: +3V3 -> /DBGSPI_MOSI
- U8 pad 2: GND -> +3V3
- U8 pad 3: Net-(R38-Pad2) -> GND
- U8 pad 4: +BATT -> /DBGSPI_MISO
- U8 pad 5: Net-(J5-Pad2) -> /DBGSPI_TRG
- U9 pad 1: /DBGSPI_MOSI -> +3V3
- U9 pad 2: +3V3 -> GND
- U9 pad 3: GND -> Net-(R38-Pad2)
- U9 pad 4: /DBGSPI_MISO -> +VDC
- U9 pad 5: /DBGSPI_TRG -> Net-(J5-Pad2)
- Y2 pad 2: Net-(Y2-Pad2) -> (no net)
- Y2 pad 4: Net-(Y2-Pad4) -> (no net)

Commit message: Expansion port and connectors
Parts:
- added J14: Expansion, Connector_IDC:IDC-Header_2x05_P2.54mm_Vertical, F.Cu at (111.9, 122.2)
- added R94: 10k, Resistor_SMD:R_0805_2012Metric, F.Cu at (228.3, 74.1)
- J3: footprint Connector_PinHeader_2.54mm:PinHeader_2x05_P2.54mm_Vertical -> Connector_IDC:IDC-Header_2x05_P2.54mm_Vertical
- moved C5 138.3 mm to (231.3, 56.4)
- moved JP1 133.2 mm to (110.9, 107.3)
- moved R13 113.1 mm to (235.7, 51.8)
- moved Y1 110.8 mm to (115.8, 111.1)
- moved C47 109.9 mm to (226.9, 59.4)
- moved Q3 101.4 mm to (164.5, 118.6)
- moved Q5 100.2 mm to (210.0, 65.8)
- moved C50 99.4 mm to (226.9, 56.4)
- moved Q1 98.5 mm to (147.7, 133.9)
- moved R47 96.3 mm to (230.9, 68.2)
- moved C4 94.2 mm to (152.1, 136.0)
- moved C24 93.6 mm to (156.5, 136.0)
- moved R33 92.8 mm to (235.7, 60.6)
- moved C55 91.6 mm to (218.8, 71.7)
- moved R30 90.5 mm to (167.3, 129.6)
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Connections:
- net /CLK_25MHZ renamed /TMC_CLK
- U7 pad 30: (no net) -> /IO4
- U7 pad 37: (no net) -> /IO3
- U7 pad 42: (no net) -> /IO0
- U7 pad 43: (no net) -> /IO1
- U7 pad 50: (no net) -> /IO2
- U8 pad 59: Net-(U8-Pad59) -> GND
- U8 pad 60: Net-(U8-Pad59) -> GND
