File: hardware/motor_controller/electric-FIAT.kicad_pcb (KiCad board)
At the start: 2 copper layers, 212 parts, among them J1 Conn_01x02_Male, J10 IMU, J11 SKiiP 613 GD123-3DUL V3, J12 Acc_sensor, J13 12V Battery, J14 Expansion, J2 Program/Debug, J3 RTMI, J4 Micro_SD_Card_Det, J5 Batt_conn, J6 Motor_U, J7 Encoder, J8 Motor_V, J9 Motor_W, Q1 AO3400, Q2 AO3400, Q3 AO3400, Q4 AO3400, Q5 AO3400, Q6 AO3400, U1 74LVC1GU04DRL, U10 ACPL-C87A, U11 OPA356xxDBV, U12 ACS759xCB-200B-PFF, U13 ACS759xCB-200B-PFF, U14 ACPL-C87A, U15 OPA356xxDBV, U16 ACS759xCB-200B-PFF, U17 OPA356xxDBV, U18 OPA356xxDBV, U19 ITW1205SA, U2 MCP2562-E-SN, U20 IU1203SA, U21 TEN40-1215E, U22 SR05S1V8, U23 74LVC1G14, U24 74LVC1G14, U25 74LVC1G14, U3 ACPL-C87A, U4 OPA356xxDBV, U5 ACPL-C87A, U6 OPA356xxDBV, U7 STM32F405RGTx, U8 TMC4671-ES, U9 ACS759xCB-200B-PFF, Y1 32.768MHz, Y2 25MHz

Commit message: Initial work on PCB
Parts:
- removed C68: 100p, Capacitor_SMD:C_0805_2012Metric
- removed L2: 6.8u, Inductor_SMD:L_Coilcraft_LPS4018
- removed Pedal_Sensor1: 5.1k, Connector_Phoenix_MC_HighVoltage:PhoenixContact_MCV_1,5_2-G-5.08_1x02_P5.08mm_Vertical
- removed TH2: Thermistor_NTC, Connector_Phoenix_MC_HighVoltage:PhoenixContact_MCV_1,5_2-G-5.08_1x02_P5.08mm_Vertical
- added Brake1: 5.1k, Connector_Phoenix_MC_HighVoltage:PhoenixContact_MCV_1,5_3-G-5.08_1x03_P5.08mm_Vertical, F.Cu at (253.9, 198.1)
- added C56: 10u, Capacitor_SMD:C_0805_2012Metric, F.Cu at (261.9, 229.5)
- added C63: 100n, Capacitor_SMD:C_0805_2012Metric, F.Cu at (261.9, 232.4)
- added C64: 100n, Capacitor_SMD:C_0805_2012Metric, F.Cu at (293.2, 199.3)
- added D1: LED, LED_SMD:LED_0805_2012Metric, F.Cu at (216.0, 243.0)
- added D2: LED, LED_SMD:LED_0805_2012Metric, F.Cu at (184.4, 263.9)
- added D3: LED, LED_SMD:LED_0805_2012Metric, F.Cu at (190.0, 238.4)
- added SW1: SW_Push, Button_Switch_SMD:SW_SPST_CK_RS282G05A3, F.Cu at (306.5, 168.6)
- added U26: OPA356xxDBV, Package_TO_SOT_SMD:SOT-23-5, F.Cu at (270.0, 204.3)
- C10: value 2.2n -> 50p
- C11: value 2.2n -> 1n
- C13: value 1u -> 100n
- C14, C53: value 1n -> 100n
- C15: value 100n -> 1u
- C19: value 100n -> 2.2n
- C20: value 30p -> 2.2n
- C22: value 10n -> 30p
- C23: value 1n -> 10n
- C24, C45: value 100p -> 1n
- C25, C30, C39, C44: value 100n -> 100p
- C27, C31, C34, C38, C41, C46: value 100p -> 100n
- C29, C36, C47: value 1n -> 100p
- C33, C37, C50: value 100n -> 1n
- C42: value 50p -> 100n
- C43: value 1n -> 50p
- C49: value 100n -> 50p
- C54: value 10u -> 1n
- C55: value 10u -> 100u; footprint Capacitor_SMD:C_0805_2012Metric -> Capacitor_THT:CP_Radial_D10.0mm_P5.00mm
- C61: value 2.2n -> 10u
- C62: value 2.2n -> 100u; footprint Capacitor_SMD:C_0805_2012Metric -> Capacitor_THT:CP_Radial_D10.0mm_P5.00mm
- C65: value 470p -> 2.2n
- C66: value 50p -> 470p
- C67: value 50p -> 2.2n
- J10: value IMU -> Motor_W; footprint Connector_PinSocket_2.54mm:PinSocket_1x10_P2.54mm_Vertical -> fiat:Motor_IGBT
- J12: value Acc_sensor -> Encoder; footprint Connector_Phoenix_MC_HighVoltage:PhoenixContact_MCV_1,5_2-G-5.08_1x02_P5.08mm_Vertical -> Connector_PinHeader_2.54mm:PinHeader_1x04_P2.54mm_Vertical
- J13: value 12V Battery -> Accelerator; footprint Connector_Phoenix_MC_HighVoltage:PhoenixContact_MCV_1,5_2-G-5.08_1x02_P5.08mm_Vertical -> Connector_Phoenix_MC_HighVoltage:PhoenixContact_MCV_1,5_3-G-5.08_1x03_P5.08mm_Vertical
- J14: value Expansion -> 12V Battery; footprint Connector_IDC:IDC-Header_2x05_P2.54mm_Vertical -> Connector_Phoenix_MC_HighVoltage:PhoenixContact_MCV_1,5_2-G-5.08_1x02_P5.08mm_Vertical
- J3: value RTMI -> Expansion
- J4: value Micro_SD_Card_Det -> RTMI; footprint Connector_Card:microSD_HC_Hirose_DM3D-SF -> Connector_IDC:IDC-Header_2x05_P2.54mm_Vertical
- J5: value Batt_conn -> Micro_SD_Card_Det; footprint fiat:Battery -> Connector_Card:microSD_HC_Hirose_DM3D-SF
- J6: value Motor_U -> Batt_conn; footprint fiat:Motor_IGBT -> fiat:Battery
- J7: value Encoder -> Motor_U; footprint Connector_PinHeader_2.54mm:PinHeader_1x04_P2.54mm_Vertical -> fiat:Motor_IGBT
- J8: value Motor_V -> IMU; footprint fiat:Motor_IGBT -> Connector_PinSocket_2.54mm:PinSocket_1x10_P2.54mm_Vertical
- J9: value Motor_W -> Motor_V
- R10, R11: moved to B.Cu
- R13: value 30k -> 3k
- R14: value 30k -> 120
- R19: value 10k -> 20k
- R20: value 20k -> 10k
- R22: value 10k -> 200k
- R3: value 3k -> 30k
- R31: value 200k -> 10k
- R38, R55: value 4.7k -> 200k
- R4: value 120 -> 30k
- R47: value 200k -> 4.7k
- R51, R54: value 4.7k -> 10k
- R53: value 10k -> 4.7k
- R64: value 200k -> 1.7k
- R65: value 100 -> 3.3k
- R66: value 100 -> 10k
- R68, R69: value 390 -> 10k
- R75: value 10k -> 1.7k
- R76: value 10k -> 3.3k
- R77: value 10k -> 1k
- R81: value 1k -> 4.7k
- R82: value 4.7k -> 1k
- R87: value 2.7k -> 1k
- R88: value 1.8k -> 1k
- R90: value 1k -> 4.5k
- R91: value 3.3k -> 3.2k
- R92: value 1k -> 2.7k
- R93: value 180 -> 2.2k
- R94: value 10k -> 2k
- U10: value ACPL-C87A -> ACS759xCB-200B-PFF; footprint Package_SO:SSO-8_6.8x5.9mm_P1.27mm_Clearance8mm -> Sensor_Current:Allegro_CB_PFF
- U11, U17, U4, U6: value OPA356xxDBV -> ACPL-C87A; footprint Package_TO_SOT_SMD:SOT-23-5 -> Package_SO:SSO-8_6.8x5.9mm_P1.27mm_Clearance8mm
- U12: value ACS759xCB-200B-PFF -> OPA356xxDBV; footprint Sensor_Current:Allegro_CB_PFF -> Package_TO_SOT_SMD:SOT-23-5
- U14, U5: value ACPL-C87A -> OPA356xxDBV; footprint Package_SO:SSO-8_6.8x5.9mm_P1.27mm_Clearance8mm -> Package_TO_SOT_SMD:SOT-23-5
- U15: value OPA356xxDBV -> 74LVC1G14; footprint Package_TO_SOT_SMD:SOT-23-5 -> fiat:Texas_R-PDSO-G5
- U19: value ITW1205SA -> OPA356xxDBV; footprint fiat:Converter_DCDC_XP_POWER-ITWxxxxSA_THT -> Package_TO_SOT_SMD:SOT-23-5
- U2: value MCP2562-E-SN -> 74LVC1G14; footprint Package_SO:SOIC-8_3.9x4.9mm_P1.27mm -> fiat:Texas_R-PDSO-G5
- U20: value IU1203SA -> 74LVC1G14; footprint fiat:Converter_DCDC_XP_POWER-IUxxxxSA_THT -> fiat:Texas_R-PDSO-G5
- U21: value TEN40-1215E -> ACS759xCB-200B-PFF; footprint fiat:Converter_DCDC_TRACO_TEN40-xxxxE -> Sensor_Current:Allegro_CB_PFF
- U22: value SR05S1V8 -> ITW1205SA; footprint fiat:Converter_DCDC_XP_POWER-SRxxSx_THT -> fiat:Converter_DCDC_XP_POWER-ITWxxxxSA_THT
- U23: value 74LVC1G14 -> TEN40-1215E; footprint fiat:Texas_R-PDSO-G5 -> fiat:Converter_DCDC_TRACO_TEN40-xxxxE
- U24: value 74LVC1G14 -> IU1203SA; footprint fiat:Texas_R-PDSO-G5 -> fiat:Converter_DCDC_XP_POWER-IUxxxxSA_THT
- U25: value 74LVC1G14 -> OPA356xxDBV; footprint fiat:Texas_R-PDSO-G5 -> Package_TO_SOT_SMD:SOT-23-5
- U3: value ACPL-C87A -> MCP2562-E-SN; footprint Package_SO:SSO-8_6.8x5.9mm_P1.27mm_Clearance8mm -> Package_SO:SOIC-8_3.9x4.9mm_P1.27mm
- U7: value STM32F405RGTx -> OPA356xxDBV; footprint Package_QFP:LQFP-64_10x10mm_P0.5mm -> Package_TO_SOT_SMD:SOT-23-5
- U8: value TMC4671-ES -> STM32F405RGTx; footprint fiat:QFN76P -> Package_QFP:LQFP-64_10x10mm_P0.5mm
- U9: value ACS759xCB-200B-PFF -> TMC4671-ES; footprint Sensor_Current:Allegro_CB_PFF -> fiat:QFN76P
- moved J5 235.6 mm to (200.3, 253.4)
- moved C40 198.3 mm to (235.9, 251.7)
- moved U5 197.6 mm to (231.6, 242.9)
- moved J7 195.1 mm to (43.0, 173.9)
- moved R19 190.8 mm to (232.0, 262.3)
- moved R69 189.6 mm to (235.9, 257.6)
- moved U20 188.5 mm to (302.2, 207.6)
- moved J14 187.5 mm to (290.6, 178.8)
- moved C47 186.7 mm to (236.2, 245.8)
- moved R80 186.6 mm to (245.2, 263.3)
- moved R50 186.3 mm to (236.4, 260.6)
- moved C22 182.5 mm to (231.0, 259.4)
- moved R39 180.8 mm to (245.2, 260.3)
- moved C55 180.5 mm to (225.4, 252.1)
- moved C19 179.5 mm to (245.0, 245.6)
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Connections:
- C10 pad 1: /VCAP_1 -> /Crystal_25MHZ
- C11 pad 1: /VCAP_2 -> Net-(C11-Pad1)
- C11 pad 2: GND -> /DC_Bus_Voltage
- C12 pad 1: +3V3 -> +5V
- C14 pad 1: Net-(C14-Pad1) -> +3V3
- C14 pad 2: /DC_Bus_Voltage -> GND
- C15 pad 1: +5V -> +3V3
- C16 pad 1: +3V3 -> /VCC_CORE
- C19 pad 1: /VCC_CORE -> /VCAP_1
- C20 pad 1: /HSE_IN -> /VCAP_2
- C21 pad 1: /HSE_OUT -> /HSE_IN
- C22 pad 1: Net-(C22-Pad1) -> /HSE_OUT
- C23 pad 1: Net-(C14-Pad1) -> Net-(C23-Pad1)
- C24 pad 1: Net-(C24-Pad1) -> Net-(C11-Pad1)
- C24 pad 2: /Motor_Voltage_U -> GND
- C25 pad 1: +5V -> Net-(C25-Pad1)
- C25 pad 2: GND -> /Motor_Voltage_U
- C26 pad 1: +3V3 -> +5V
- C27 pad 1: Net-(C27-Pad1) -> +3V3
- C28 pad 1: Net-(C24-Pad1) -> Net-(C28-Pad1)
- C29 pad 1: /DC_Current -> Net-(C25-Pad1)
- C30 pad 1: +3V3 -> Net-(C30-Pad1)
- C30 pad 2: GND -> /Motor_Voltage_V
- C31 pad 1: Net-(C31-Pad1) -> +5V
- C31 pad 2: /Motor_Voltage_V -> GND
- C32 pad 1: +5V -> +3V3
- C33 pad 1: +3V3 -> /DC_Current
- C34 pad 1: Net-(C34-Pad1) -> +3V3
- C35 pad 1: Net-(C31-Pad1) -> Net-(C35-Pad1)
- C36 pad 1: /Motor_Current_U -> Net-(C30-Pad1)
- C37 pad 1: +3V3 -> /Motor_Current_U
- C38 pad 1: Net-(C38-Pad1) -> +3V3
- C38 pad 2: /Motor_Voltage_W -> GND
- C39 pad 1: +5V -> Net-(C39-Pad1)
- C39 pad 2: GND -> /Motor_Voltage_W
- C40 pad 1: +3V3 -> +5V
- C41 pad 1: /ENC_A -> +3V3
- C42 pad 1: /ENC_A_T -> Net-(C42-Pad1)
- C43 pad 1: /Motor_Current_V -> /ENC_B_T
- C44 pad 1: +3V3 -> Net-(C44-Pad1)
- C45 pad 1: Net-(C45-Pad1) -> /Motor_Current_V
- C46 pad 1: Net-(C38-Pad1) -> +3V3
- C47 pad 1: /Motor_Current_W -> Net-(C39-Pad1)
- C48 pad 1: +3V3 -> Net-(C48-Pad1)
- C49 pad 1: +3V3 -> /ENC_B_T
- C50 pad 1: +3V3 -> /Motor_Current_W
- C51 pad 1: +1V8 -> +3V3
- C52 pad 1: +1V8 -> +3V3
- C53 pad 1: +BATT -> +3V3
- C53 pad 2: +24V -> GND
- C54 pad 1: +5V -> +BATT
- C54 pad 2: GND -> +24V
- C55 pad 1: +3V3 -> +5V
- C61 pad 1: -BATT -> +3V3
- C62 pad 1: -BATT -> +3V3
- C66 pad 1: /Crystal_25MHZ -> -BATT
- C67 pad 1: /ENC_B_T -> -BATT
- J10 pad 1: +3V3 -> /IGBT_W
- J10 pad 2: GND -> /Motor_W
- J11 pad 20: (no net) -> /TEMP_OUT
- J12 pad 1: /accelerator_pedal -> +5V
- J12 pad 2: GND -> (no net)
- J13 pad 1: +BATT -> +5V
- J13 pad 2: GND -> Net-(J13-Pad2)
- J14 pad 1: +1V8 -> +BATT
- J14 pad 2: /IO4 -> GND
- J3 pad 1: +3V3 -> (no net)
- J3 pad 10: GND -> /IO0
- J3 pad 2: (no net) -> /IO4
- J3 pad 3: /DBGSPI_nSCS -> +3V3
- J3 pad 4: /DBGSPI_TRG -> /IO3
- J3 pad 5: /DBGSPI_SCK -> +5V
- J3 pad 6: GND -> /IO2
- J3 pad 7: /DBGSPI_MOSI -> +24V
- J3 pad 8: GND -> /IO1
- J3 pad 9: /DBGSPI_MISO -> GND
- J4 pad 1: /SD_DAT2 -> +3V3
- J4 pad 10: +3V3 -> GND
- J4 pad 2: /SD_DAT3 -> (no net)
- J4 pad 3: /SD_CMD -> /DBGSPI_nSCS
- J4 pad 4: +3V3 -> /DBGSPI_TRG
- J4 pad 5: /SD_CLK -> /DBGSPI_SCK
- J4 pad 7: /SD_DAT0 -> /DBGSPI_MOSI
- J4 pad 8: /SD_DAT1 -> GND
- J4 pad 9: /SD_DET -> /DBGSPI_MISO
- J5 pad 1: +VDC -> /SD_DAT2
- J5 pad 2: Net-(J5-Pad2) -> /SD_DAT3
- J5 pad 3: GND -> /SD_CMD
- J6 pad 1: /IGBT_U -> /DC+
- J6 pad 2: /Motor_U -> +VDC
- J7 pad 1: +5V -> /IGBT_U
- J7 pad 2: /ENC_A_R -> /Motor_U
- J8 pad 1: /IGBT_V -> +3V3
- J8 pad 2: /Motor_V -> GND
- J9 pad 1: /IGBT_W -> /IGBT_V
- J9 pad 2: /Motor_W -> /Motor_V
- Q1 pad 2: /PWM_VT -> /PWM_UT
- Q1 pad 3: /HB_VT -> /HB_UT
- Q2 pad 2: /PWM_VB -> /PWM_UB
- Q2 pad 3: /HB_VB -> /HB_UB
- Q3 pad 2: /PWM_UT -> /PWM_VT
- Q3 pad 3: /HB_UT -> /HB_VT
- Q4 pad 2: /PWM_UB -> /PWM_VB
- Q4 pad 3: /HB_UB -> /HB_VB
- R12 pad 1: Net-(R12-Pad1) -> +VDC
- R13 pad 1: Net-(R12-Pad1) -> Net-(R1-Pad1)
- R13 pad 2: Net-(R13-Pad2) -> /HSE_OUT
- R14 pad 1: +BATT -> Net-(J1-Pad2)
- R14 pad 2: Net-(R13-Pad2) -> Net-(J1-Pad1)
- R15 pad 1: Net-(C22-Pad1) -> Net-(C23-Pad1)
- R18 pad 2: Net-(C14-Pad1) -> Net-(C11-Pad1)
- R19 pad 1: +3V3 -> Net-(C11-Pad1)
- R19 pad 2: /reset -> GND
- R2 pad 1: Net-(C14-Pad1) -> Net-(C11-Pad1)
- R20 pad 1: Net-(C14-Pad1) -> +3V3
- R20 pad 2: GND -> /reset
- R21 pad 1: +3V3 -> Net-(C25-Pad1)
- R21 pad 2: /reset -> /Motor_Voltage_U
- R22 pad 1: Net-(C24-Pad1) -> Net-(R22-Pad1)
- R22 pad 2: /Motor_Voltage_U -> Net-(C28-Pad1)
- R23 pad 1: Net-(R23-Pad1) -> Net-(R22-Pad1)
- R23 pad 2: Net-(C27-Pad1) -> Net-(R23-Pad2)
- R24 pad 1: Net-(R23-Pad1) -> Net-(R24-Pad1)
- R24 pad 2: Net-(R24-Pad2) -> Net-(R23-Pad2)
- R25 pad 1: Net-(R25-Pad1) -> Net-(R24-Pad1)
- R25 pad 2: Net-(R24-Pad2) -> Net-(R25-Pad2)
- R26 pad 1: Net-(R25-Pad1) -> Net-(R26-Pad1)
- R26 pad 2: Net-(R26-Pad2) -> Net-(R25-Pad2)
- R27 pad 1: Net-(R27-Pad1) -> Net-(R26-Pad1)
- R27 pad 2: Net-(R26-Pad2) -> Net-(R27-Pad2)
- R28 pad 1: Net-(R27-Pad1) -> Net-(R28-Pad1)
- R28 pad 2: Net-(R28-Pad2) -> Net-(R27-Pad2)
- R29 pad 1: Net-(R29-Pad1) -> Net-(R28-Pad1)
- R29 pad 2: Net-(R28-Pad2) -> Net-(R29-Pad2)
- R3 pad 1: Net-(R1-Pad1) -> Net-(R15-Pad2)
- R3 pad 2: /HSE_OUT -> Net-(R3-Pad2)
- R30 pad 1: Net-(R29-Pad1) -> /Motor_U
- R30 pad 2: Net-(R30-Pad2) -> Net-(R29-Pad2)
- R31 pad 1: /Motor_U -> +3V3
- R31 pad 2: Net-(R30-Pad2) -> /reset
- R34 pad 1: Net-(C27-Pad1) -> Net-(C28-Pad1)
- R35 pad 2: Net-(C24-Pad1) -> Net-(C25-Pad1)
- R36 pad 1: Net-(C24-Pad1) -> Net-(C25-Pad1)
- R37 pad 1: Net-(C31-Pad1) -> Net-(C30-Pad1)
- R38 pad 1: /DC_Current -> Net-(R38-Pad1)
- R38 pad 2: Net-(R38-Pad2) -> Net-(C35-Pad1)
- R39 pad 1: Net-(R39-Pad1) -> Net-(R38-Pad1)
- R39 pad 2: Net-(C34-Pad1) -> Net-(R39-Pad2)
- R4 pad 1: Net-(J1-Pad2) -> Net-(R4-Pad1)
- R4 pad 2: Net-(J1-Pad1) -> Net-(R3-Pad2)
- R40 pad 1: Net-(R39-Pad1) -> Net-(R40-Pad1)
- R40 pad 2: Net-(R40-Pad2) -> Net-(R39-Pad2)
- R41 pad 1: Net-(R41-Pad1) -> Net-(R40-Pad1)
- R41 pad 2: Net-(R40-Pad2) -> Net-(R41-Pad2)
- R42 pad 1: Net-(R41-Pad1) -> Net-(R42-Pad1)
- R42 pad 2: Net-(R42-Pad2) -> Net-(R41-Pad2)
- R43 pad 1: Net-(R43-Pad1) -> Net-(R42-Pad1)
- R43 pad 2: Net-(R42-Pad2) -> Net-(R43-Pad2)
- R44 pad 1: Net-(R43-Pad1) -> Net-(R44-Pad1)
- R44 pad 2: Net-(R44-Pad2) -> Net-(R43-Pad2)
- R45 pad 1: Net-(R45-Pad1) -> Net-(R44-Pad1)
- R45 pad 2: Net-(R44-Pad2) -> Net-(R45-Pad2)
- R46 pad 1: Net-(R45-Pad1) -> /Motor_V
- R46 pad 2: Net-(R46-Pad2) -> Net-(R45-Pad2)
- R47 pad 1: /Motor_V -> /DC_Current
- R47 pad 2: Net-(R46-Pad2) -> Net-(R47-Pad2)
- R49 pad 1: Net-(C34-Pad1) -> +3V3
- R49 pad 2: GND -> /ENABLE_INPUTS
- R5 pad 1: Net-(R15-Pad2) -> Net-(R4-Pad1)
- R50 pad 1: Net-(R50-Pad1) -> Net-(C35-Pad1)
- R50 pad 2: Net-(C31-Pad1) -> GND
- R51 pad 1: /Motor_Current_U -> Net-(R51-Pad1)
- R51 pad 2: Net-(R51-Pad2) -> Net-(C30-Pad1)
- R52 pad 1: Net-(C31-Pad1) -> Net-(C30-Pad1)
- R53 pad 1: Net-(C38-Pad1) -> /Motor_Current_U
- R53 pad 2: /Motor_Voltage_W -> Net-(R53-Pad2)
- R54 pad 1: +5V -> Net-(C39-Pad1)
- R54 pad 2: /ENC_A_R -> /Motor_Voltage_W
- R55 pad 1: +5V -> Net-(R55-Pad1)
- R55 pad 2: /ENC_B_R -> Net-(C44-Pad1)
- R56 pad 1: Net-(R56-Pad1) -> Net-(R55-Pad1)
- R56 pad 2: Net-(C45-Pad1) -> Net-(R56-Pad2)
- R57 pad 1: Net-(R56-Pad1) -> Net-(R57-Pad1)
- R57 pad 2: Net-(R57-Pad2) -> Net-(R56-Pad2)
- R58 pad 1: Net-(R58-Pad1) -> Net-(R57-Pad1)
- R58 pad 2: Net-(R57-Pad2) -> Net-(R58-Pad2)
- R59 pad 1: Net-(R58-Pad1) -> Net-(R59-Pad1)
- R59 pad 2: Net-(R59-Pad2) -> Net-(R58-Pad2)
- R60 pad 1: Net-(R60-Pad1) -> Net-(R59-Pad1)
- R60 pad 2: Net-(R59-Pad2) -> Net-(R60-Pad2)
- R61 pad 1: Net-(R60-Pad1) -> Net-(R61-Pad1)
- R61 pad 2: Net-(R61-Pad2) -> Net-(R60-Pad2)
- R62 pad 1: Net-(R62-Pad1) -> Net-(R61-Pad1)
- R62 pad 2: Net-(R61-Pad2) -> Net-(R62-Pad2)
- R63 pad 1: Net-(R62-Pad1) -> /Motor_W
- R63 pad 2: Net-(R63-Pad2) -> Net-(R62-Pad2)
- R64 pad 1: /Motor_W -> /ENC_B_R
- R64 pad 2: Net-(R63-Pad2) -> Net-(C42-Pad1)
- R65 pad 1: /ENC_A -> Net-(C42-Pad1)
- R65 pad 2: /ENC_A_R -> GND
- R66 pad 1: /ENC_B -> Net-(R66-Pad1)
- R66 pad 2: /ENC_B_R -> Net-(R66-Pad2)
- R68 pad 1: /ENC_A -> Net-(C44-Pad1)
- R69 pad 1: /ENC_B -> Net-(R69-Pad1)
- R69 pad 2: GND -> Net-(C39-Pad1)
- R70 pad 2: /PWM_VT -> /PWM_UT
- R71 pad 2: /HB_VT -> /HB_UT
- R72 pad 2: /PWM_VB -> /PWM_UB
- R73 pad 2: /HB_VB -> /HB_UB
- R74 pad 1: Net-(R74-Pad1) -> Net-(C39-Pad1)
- R74 pad 2: Net-(R74-Pad2) -> GND
- R75 pad 1: Net-(C45-Pad1) -> /ENC_B_R
- R75 pad 2: GND -> Net-(C48-Pad1)
- R76 pad 1: Net-(R76-Pad1) -> Net-(C48-Pad1)
- R76 pad 2: Net-(C38-Pad1) -> GND
- R77 pad 1: Net-(C38-Pad1) -> +3V3
- R77 pad 2: GND -> /PWM_VT
- R78 pad 1: +3V3 -> +15V
- R78 pad 2: /PWM_UT -> /HB_VT
- R79 pad 1: +15V -> +3V3
- R79 pad 2: /HB_UT -> /PWM_VB
- R80 pad 1: +3V3 -> +15V
- R80 pad 2: /PWM_UB -> /HB_VB
- R81 pad 1: +15V -> /Motor_Current_W
- R81 pad 2: /HB_UB -> Net-(R81-Pad2)
- R82 pad 1: /Motor_Current_W -> Net-(D1-Pad1)
- R82 pad 2: Net-(R82-Pad2) -> GND
- R83 pad 1: +3V3 -> Net-(D2-Pad1)
- R83 pad 2: /PWM_WT -> GND
- R84 pad 1: +15V -> Net-(D3-Pad1)
- R84 pad 2: /HB_WT -> GND
- R85 pad 2: /PWM_WB -> /PWM_WT
- R86 pad 2: /HB_WB -> /HB_WT
- R87 pad 1: Net-(R87-Pad1) -> +3V3
- R87 pad 2: GND -> /PWM_WB
- R88 pad 1: Net-(R88-Pad1) -> +15V
- R88 pad 2: GND -> /HB_WB
- R90 pad 1: Net-(R90-Pad1) -> /TEMP_OUT
- R90 pad 2: +1V8 -> Net-(C64-Pad1)
- R91 pad 1: /Motor_temp -> /accelerator_pedal
- R91 pad 2: Net-(R90-Pad1) -> Net-(J13-Pad2)
- R92 pad 1: Net-(R92-Pad1) -> Net-(C63-Pad1)
- R92 pad 2: +1V8 -> GND
- R93 pad 1: /Inverter_temp -> Net-(C64-Pad1)
- R93 pad 2: Net-(R92-Pad1) -> GND
- R94 pad 1: +3V3 -> Net-(J13-Pad2)
- R94 pad 2: /ENABLE_INPUTS -> GND
- TH1 pad 2: Net-(R87-Pad1) -> Net-(C63-Pad1)
- U10 pad 1: +5V -> +3V3
- U10 pad 2: Net-(C34-Pad1) -> GND
- U10 pad 3: GND -> Net-(R47-Pad2)
- U10 pad 4: GND -> +VDC
- U10 pad 5: GND -> /DC+
- U11 pad 1: /Motor_Voltage_V -> +5V
- U11 pad 2: GND -> Net-(C35-Pad1)
- U11 pad 3: Net-(R48-Pad1) -> GND
- U11 pad 4: Net-(C31-Pad1) -> GND
- U11 pad 5: +3V3 -> GND
- U12 pad 1: +3V3 -> /Motor_Voltage_V
- U12 pad 3: Net-(R51-Pad2) -> Net-(R48-Pad1)
- U12 pad 4: /IGBT_U -> Net-(C30-Pad1)
- U12 pad 5: /Motor_U -> +3V3
- U13 pad 3: Net-(R67-Pad2) -> Net-(R53-Pad2)
- U13 pad 4: /IGBT_V -> /IGBT_U
- U13 pad 5: /Motor_V -> /Motor_U
- U14 pad 1: +5V -> /ENC_B
- U14 pad 2: Net-(C45-Pad1) -> GND
- U14 pad 3: GND -> Net-(C42-Pad1)
- U14 pad 4: GND -> /ENC_B
- U14 pad 5: GND -> +3V3
- U15 pad 1: /Motor_Voltage_W -> (no net)
- U15 pad 2: GND -> /ENC_B
- U15 pad 3: Net-(R74-Pad1) -> GND
- U15 pad 4: Net-(C38-Pad1) -> /ENC_B_T
- U16 pad 3: Net-(R82-Pad2) -> Net-(R67-Pad2)
- U16 pad 4: /IGBT_W -> /IGBT_V
- U16 pad 5: /Motor_W -> /Motor_V
- U17 pad 1: /Motor_temp -> +5V
- U17 pad 2: GND -> Net-(C44-Pad1)
- U17 pad 3: Net-(R87-Pad1) -> GND
- U17 pad 4: Net-(R90-Pad1) -> GND
- U17 pad 5: +3V3 -> GND
- U18 pad 1: /Inverter_temp -> /Motor_Voltage_W
- U18 pad 3: Net-(R88-Pad1) -> Net-(R66-Pad1)
- U18 pad 4: Net-(R92-Pad1) -> Net-(C39-Pad1)
- U19 pad 1: -BATT -> /ENC_B
- U19 pad 2: Net-(L1-Pad2) -> GND
- U19 pad 4: +5V -> /ENC_B
- U19 pad 5: (no net) -> +3V3
- U2 pad 1: /CAN_RX -> (no net)
- U2 pad 2: GND -> Net-(R1-Pad1)
- U2 pad 3: +5V -> GND
- U2 pad 4: /CAN_TX -> /Crystal_25MHZ
- U20 pad 1: -BATT -> (no net)
- U20 pad 2: +BATT -> /ENC_B
- U20 pad 3: (no net) -> GND
- U20 pad 5: (no net) -> +3V3
- U21 pad 1: +BATT -> +3V3
- U21 pad 2: -BATT -> GND
- U21 pad 3: (no net) -> Net-(R81-Pad2)
- U21 pad 4: +24V -> /IGBT_W
- U21 pad 5: GND -> /Motor_W
- U22 pad 1: Net-(C64-Pad1) -> -BATT
- U22 pad 2: GND -> Net-(L1-Pad2)
- U23 pad 1: (no net) -> +BATT
- U23 pad 2: Net-(R1-Pad1) -> -BATT
- U23 pad 3: GND -> (no net)
- U23 pad 4: /Crystal_25MHZ -> +24V
- U23 pad 5: +3V3 -> GND
- U24 pad 1: (no net) -> -BATT
- U24 pad 2: /ENC_B -> +BATT
- U24 pad 3: GND -> (no net)
- U24 pad 5: +3V3 -> (no net)
- U25 pad 1: (no net) -> /Motor_temp
- U25 pad 2: /ENC_A -> GND
- U25 pad 3: GND -> Net-(C63-Pad1)
- U25 pad 4: /ENC_A_T -> /Motor_temp
- U3 pad 1: +5V -> /CAN_RX
- U3 pad 2: Net-(C22-Pad1) -> GND
- U3 pad 3: GND -> +5V
- U3 pad 4: GND -> /CAN_TX
- U3 pad 5: GND -> +3V3
- U3 pad 6: Net-(R18-Pad1) -> Net-(J1-Pad1)
- U3 pad 7: Net-(R16-Pad2) -> Net-(J1-Pad2)
- U3 pad 8: +3V3 -> /CAN_STBY
- U4 pad 1: /DC_Bus_Voltage -> +5V
- U4 pad 2: GND -> Net-(C23-Pad1)
- U4 pad 3: Net-(R16-Pad1) -> GND
- U4 pad 4: Net-(C14-Pad1) -> GND
- U4 pad 5: +3V3 -> GND
- U5 pad 1: +5V -> /DC_Bus_Voltage
- U5 pad 2: Net-(C27-Pad1) -> GND
- U5 pad 3: GND -> Net-(R16-Pad1)
- U5 pad 4: GND -> Net-(C11-Pad1)
- U5 pad 5: GND -> +3V3
- U6 pad 1: /Motor_Voltage_U -> +5V
- U6 pad 2: GND -> Net-(C28-Pad1)
- U6 pad 3: Net-(R33-Pad1) -> GND
- U6 pad 4: Net-(C24-Pad1) -> GND
- U6 pad 5: +3V3 -> GND
- U7 pad 1: (no net) -> /Motor_Voltage_U
- U7 pad 2: /IGBT_OVER_TEMP -> GND
- U7 pad 3: /LSE_IN -> Net-(R33-Pad1)
- U7 pad 4: /LSE_OUT -> Net-(C25-Pad1)
- U7 pad 5: /HSE_IN -> +3V3
- U8 pad 1: /DBGSPI_MOSI -> (no net)
- U8 pad 10: (no net) -> /braking_pedal
- U8 pad 11: (no net) -> /accelerator_pedal
- U8 pad 12: /FOC_Status -> GND
- U8 pad 14: GND -> (no net)
- U8 pad 15: /VCC_CORE -> /ENC_B_T
- U8 pad 16: /Motor_Current_U -> /Motor_Current_W
- U8 pad 17: (no net) -> /DC_Bus_Voltage
- U8 pad 18: /Motor_Current_V -> GND
- U8 pad 19: (no net) -> +3V3
- U8 pad 2: +3V3 -> /IGBT_OVER_TEMP
- U8 pad 20: (no net) -> /SPI1_CS_Accel
- U8 pad 21: (no net) -> /SPI2_NSS
- U8 pad 22: (no net) -> /DC_Current
- U8 pad 23: +5V -> /Motor_Voltage_U
- U8 pad 24: GND -> /Motor_Voltage_V
- U8 pad 25: /ENC_A -> /Motor_Voltage_W
- U8 pad 26: (no net) -> /Motor_temp
- U8 pad 27: (no net) -> /IGBT_Temp
- U8 pad 28: (no net) -> /SPI1_CS_Gyro
- U8 pad 29: /ENC_B -> /SPI1_CS_Magnet
- U8 pad 3: GND -> /LSE_IN
- U8 pad 30: (no net) -> /IO4
- U8 pad 31: (no net) -> /VCAP_1
- U8 pad 32: (no net) -> +3V3
- U8 pad 33: (no net) -> /SPI2_NSS
- U8 pad 34: (no net) -> /SPI2_SCK
- U8 pad 35: (no net) -> /SPI2_MISO
- U8 pad 36: (no net) -> /SPI2_MOSI
- U8 pad 37: (no net) -> /IO3
- U8 pad 38: (no net) -> /SD_DET
- U8 pad 39: /PWM_UT -> /SD_DAT0
- U8 pad 4: /DBGSPI_MISO -> /LSE_OUT
- U8 pad 40: /PWM_UB -> /SD_DAT1
- U8 pad 41: /PWM_VT -> /MCU_MCO
- U8 pad 42: /PWM_VB -> /IO0
- U8 pad 43: +3V3 -> /IO1
- U8 pad 44: GND -> /CAN_RX
- U8 pad 45: /VCC_CORE -> /CAN_TX
- U8 pad 46: /PWM_WT -> /SWDIO
- U8 pad 47: /PWM_WB -> /VCAP_2
- U8 pad 48: (no net) -> +3V3
- U8 pad 49: (no net) -> /SWCLK
- U8 pad 5: /DBGSPI_TRG -> /HSE_IN
- U8 pad 50: /reset -> /IO2
- U8 pad 51: /TMC_CLK -> /SD_DAT2
- U8 pad 52: +3V3 -> /SD_DAT3
- U8 pad 53: GND -> /SD_CLK
- U8 pad 54: GND -> /SD_CMD
- U8 pad 55: /ENABLE_INPUTS -> /SWO
- U8 pad 56: (no net) -> /ENABLE_INPUTS
- U8 pad 57: (no net) -> /CAN_STBY
- U8 pad 58: (no net) -> /FOC_Status
- U8 pad 59: GND -> /ERROR_HB1
- U8 pad 6: /SPI2_NSS -> /HSE_OUT
- U8 pad 61: +3V3 -> /ERROR_HB2
- U8 pad 62: GND -> /ERROR_HB3
- U8 pad 63: /VCC_CORE -> GND
- U8 pad 64: (no net) -> +3V3
- U8 pad 7: /SPI2_SCK -> /reset
- U8 pad 8: /SPI2_MOSI -> /Motor_Current_U
- U8 pad 9: /SPI2_MISO -> /Motor_Current_V
- U9 pad 1: +3V3 -> /DBGSPI_MOSI
- U9 pad 2: GND -> +3V3
- U9 pad 3: Net-(R38-Pad2) -> GND
- U9 pad 4: +VDC -> /DBGSPI_MISO
- U9 pad 5: Net-(J5-Pad2) -> /DBGSPI_TRG
Routing:
- net +VDC: track 0.00 -> 27.0 mm
- net /DC+: track 0.00 -> 14.1 mm
- net Net-(R47-Pad2): track 0.00 -> 3.28 mm
- net +3V3: track 0.00 -> 2.16 mm
- net /DC_Current: track 0.00 -> 2.00 mm
- net Net-(R11-Pad2): vias 0 -> 1
- added copper zone on F.Cu, net GND
Other:
- net class PWR added: clearance 1, trace_width 20, via_dia 0.8, via_drill 0.4

Commit message: Schematic v1.0 and PCB in progress
Parts:
- removed JP1: Clock Selection, Connector_PinHeader_2.54mm:PinHeader_1x03_P2.54mm_Vertical
- removed R1: 1M, Resistor_SMD:R_0805_2012Metric
- removed R13: 3k, Resistor_SMD:R_0805_2012Metric
- removed SW1: SW_Push, Button_Switch_SMD:SW_SPST_CK_RS282G05A3
- removed U1: 74LVC1GU04DRL, Package_TO_SOT_SMD:SOT-553
- removed U2: 74LVC1G14, fiat:Texas_R-PDSO-G5
- added C68: 100n, Capacitor_SMD:C_0805_2012Metric, F.Cu at (93.7, 58.2)
- added C69: 100n, Capacitor_SMD:C_0805_2012Metric, F.Cu at (-89.9, 25.2)
- added C70: 100n, Capacitor_SMD:C_0805_2012Metric, F.Cu at (-89.9, 28.1)
- added C71: 100n, Capacitor_SMD:C_0805_2012Metric, F.Cu at (-85.5, 25.2)
- added C72: 100n, Capacitor_SMD:C_0805_2012Metric, F.Cu at (-84.6, 99.3)
- added C73: 100n, Capacitor_SMD:C_0805_2012Metric, F.Cu at (-80.2, 96.4)
- added C74: 100n, Capacitor_SMD:C_0805_2012Metric, F.Cu at (-80.2, 99.3)
- added D4: LED, LED_SMD:LED_0805_2012Metric, F.Cu at (-130.9, 16.4)
- added D5: LED, LED_SMD:LED_0805_2012Metric, F.Cu at (-130.9, 19.4)
- added D6: LED, LED_SMD:LED_0805_2012Metric, F.Cu at (-126.5, 16.4)
- added D7: LED, LED_SMD:LED_0805_2012Metric, F.Cu at (-130.9, 22.5)
- added D8: LED, LED_SMD:LED_0805_2012Metric, F.Cu at (-126.5, 19.4)
- added R95: 1k, Resistor_SMD:R_0805_2012Metric, F.Cu at (-122.0, 16.4)
- added R96: 1k, Resistor_SMD:R_0805_2012Metric, F.Cu at (-126.5, 22.4)
- added R97: 1k, Resistor_SMD:R_0805_2012Metric, F.Cu at (-122.0, 19.3)
- added R98: 1k, Resistor_SMD:R_0805_2012Metric, F.Cu at (-117.6, 16.4)
- added R99: 1k, Resistor_SMD:R_0805_2012Metric, F.Cu at (-122.1, 22.4)
- C10: value 50p -> 100n
- C11, C12, C24, C33, C34, C37, C38, C45, C46, C50, C51, J11, R15, R16, R17, R18, R19, R2, R3, R47, R53, R6, R67, R7, R81: moved to B.Cu
- J1: value Conn_01x02_Male -> CAN
- moved J5 433.4 mm to (-117.8, -40.9), turned to 180 degrees
- moved C52 428.4 mm to (-108.7, 27.5)
- moved C53 425.5 mm to (-104.3, 27.5)
- moved C32 385.1 mm to (-112.7, 110.8)
- moved D2 385.1 mm to (-169.1, 111.2)
- moved R54 385.1 mm to (-117.1, 110.8)
- moved R80 385.1 mm to (-108.3, 110.6)
- moved Brake1 385.1 mm to (-99.6, 45.4)
- moved C1 385.1 mm to (-126.9, 106.7)
- moved C14 385.1 mm to (-131.3, 106.7)
- moved C15 385.1 mm to (-139.1, 111.5)
- moved C16 385.1 mm to (-96.0, 76.8)
- moved C17 385.1 mm to (-134.7, 111.5)
- moved C18 385.1 mm to (-40.3, 25.8)
- moved C19 385.1 mm to (-108.5, 92.9)
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Connections:
- C10 pad 1: /Crystal_25MHZ -> +5V
- C43 pad 1: /ENC_B_T -> /ENC_A_T
- J12 pad 2: (no net) -> /ENC_A_R
- J3 pad 1: (no net) -> +5V
- J3 pad 5: +5V -> +15V
- R64 pad 1: /ENC_B_R -> /ENC_A_R
- U14 pad 1: /ENC_B -> /ENC_A
- U14 pad 4: /ENC_B -> /ENC_A
- U15 pad 2: /ENC_B -> /ENC_A
- U15 pad 4: /ENC_B_T -> /ENC_A_T
- U8 pad 14: (no net) -> /ENC_A_T
- U8 pad 41: /MCU_MCO -> /TMC_CLK
- U9 pad 25: (no net) -> /ENC_A
Routing:
- net /Motor_W: track 0.00 -> 15.0 mm
- net /IGBT_W: track 0.00 -> 14.3 mm
- net GND: track 0.00 -> 14.3 mm, vias 0 -> 4
- net /Motor_U: track 0.00 -> 14.2 mm
- net /IGBT_V: track 0.00 -> 14.2 mm
- net /IGBT_U: track 0.00 -> 14.1 mm
- net /Motor_V: track 0.00 -> 13.9 mm
- net Net-(C11-Pad1): track 0.00 -> 11.8 mm, vias 0 -> 2
- net +VDC: track 27.0 -> 16.4 mm
- net +3V3: track 2.16 -> 11.7 mm
- net Net-(C23-Pad1): track 0.00 -> 6.23 mm, vias 0 -> 1
- net Net-(R16-Pad2): track 0.00 -> 5.25 mm, vias 0 -> 1
- net Net-(R16-Pad1): track 0.00 -> 4.68 mm, vias 0 -> 1
- net Net-(R15-Pad2): track 0.00 -> 4.01 mm
- net /DC_Bus_Voltage: track 0.00 -> 3.14 mm, vias 0 -> 1
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- removed copper zone on F.Cu, net GND
Other:
- board outline added: 185 x 192 mm
- net class Default: trace_width 0.25 -> 0.2

Commit message: PCB final size
Parts:
- removed the C11 at (93.8, 55.2)
- removed the C12 at (89.4, 48.8)
- removed the C13 at (88.2, 61.7)
- removed the C23 at (83.7, 49.7)
- removed the C24 at (90.8, 53.1)
- removed the C33 at (88.4, 64.1)
- removed the C34 at (90.9, 69.0)
- removed the C37 at (127.1, -1.00)
- removed the C38 at (124.5, -5.90)
- removed the C45 at (127.2, 60.9)
- removed the C46 at (124.6, 56.0)
- removed the C50 at (127.2, 122.9)
- removed the C51 at (124.6, 118.0)
- removed the C56 at (-91.6, 76.8)
- removed the C61 at (-82.1, 58.4)
- removed the C68 at (93.7, 58.2)
- removed the R12 at (83.7, 59.7)
- removed the R18 at (88.1, 57.1)
- removed the R19 at (88.1, 53.1)
- removed the R47 at (90.2, 66.1)
- removed the R53 at (125.2, -3.00)
- removed the R67 at (125.3, 58.9)
- removed the R81 at (125.3, 120.9)
- removed the U10 at (92.6, 69.9)
- removed the U13 at (122.8, -6.80)
- removed the U16 at (122.9, 55.1)
- removed the U21 at (122.9, 117.1)
- removed the U4 at (88.7, 54.1)
- removed the U5 at (93.8, 55.2)
- removed the U9 at (104.8, 46.4)
- added C14: 1n, Capacitor_SMD:C_0805_2012Metric, B.Cu at (108.2, 107.7)
- added C15: 100n, Capacitor_SMD:C_0805_2012Metric, B.Cu at (103.8, 101.3)
- added C16: 100n, Capacitor_SMD:C_0805_2012Metric, F.Cu at (102.6, 114.2)
- added C17: 100n, Capacitor_SMD:C_0805_2012Metric, F.Cu at (108.1, 110.7)
- added C25: 10n, Capacitor_SMD:C_0805_2012Metric, F.Cu at (98.1, 102.2)
- added C26: 1n, Capacitor_SMD:C_0805_2012Metric, B.Cu at (105.2, 105.6)
- added C39: 1n, Capacitor_SMD:C_0805_2012Metric, B.Cu at (102.8, 116.6)
- added C40: 100n, Capacitor_SMD:C_0805_2012Metric, B.Cu at (105.3, 121.5)
- added C43: 1n, Capacitor_SMD:C_0805_2012Metric, B.Cu at (124.8, 47.4)
- added C44: 100n, Capacitor_SMD:C_0805_2012Metric, B.Cu at (122.2, 42.5)
- added C52: 1n, Capacitor_SMD:C_0805_2012Metric, B.Cu at (124.9, 109.3)
- added C53: 100n, Capacitor_SMD:C_0805_2012Metric, B.Cu at (122.3, 104.4)
- added C57: 1n, Capacitor_SMD:C_0805_2012Metric, B.Cu at (124.9, 171.3)
- added C58: 100n, Capacitor_SMD:C_0805_2012Metric, B.Cu at (122.3, 166.4)
- added R1: 20k, Resistor_SMD:R_0805_2012Metric, B.Cu at (108.2, 109.7)
- added R13: 39, Resistor_SMD:R_0805_2012Metric, B.Cu at (98.1, 102.2)
- added R14: 20k, Resistor_SMD:R_0805_2012Metric, B.Cu at (102.5, 107.6)
- added R45: 4.7k, Resistor_SMD:R_0805_2012Metric, B.Cu at (104.6, 118.6)
- added R51: 4.7k, Resistor_SMD:R_0805_2012Metric, B.Cu at (122.9, 45.4)
- added R65: 4.7k, Resistor_SMD:R_0805_2012Metric, B.Cu at (123.0, 107.3)
- added R79: 4.7k, Resistor_SMD:R_0805_2012Metric, B.Cu at (123.0, 169.3)
- added U11: ACS759xCB-200B-PFF, Sensor_Current:Allegro_CB_PFF, F.Cu at (120.5, 41.6)
- added U14: ACS759xCB-200B-PFF, Sensor_Current:Allegro_CB_PFF, F.Cu at (120.6, 103.5)
- added U19: ACS759xCB-200B-PFF, Sensor_Current:Allegro_CB_PFF, F.Cu at (120.6, 165.5)
- added U2: ACPL-C87A, Package_SO:SSO-8_6.8x5.9mm_P1.27mm_Clearance8mm, F.Cu at (103.1, 106.6)
- added U3: OPA356xxDBV, Package_TO_SOT_SMD:SOT-23-5, F.Cu at (108.2, 107.7)
- added U7: TMC4671-ES, fiat:QFN76P, F.Cu at (100.5, 95.2)
- added U8: ACS759xCB-200B-PFF, Sensor_Current:Allegro_CB_PFF, F.Cu at (107.0, 122.4)
- C64: renamed from C57; moved to B.Cu
- C66: renamed from C59; moved to B.Cu
- C70: renamed from C65; moved to B.Cu
- C72: renamed from C66; moved to B.Cu
- D1: renamed from D3; value LED -> GREEN
- J1: footprint Connector_Phoenix_MC_HighVoltage:PhoenixContact_MCV_1,5_2-G-5.08_1x02_P5.08mm_Vertical -> Connector_Phoenix_MC:PhoenixContact_MCV_1,5_2-G-3.81_1x02_P3.81mm_Vertical
- J12: footprint Connector_PinHeader_2.54mm:PinHeader_1x04_P2.54mm_Vertical -> Connector_Phoenix_MC:PhoenixContact_MCV_1,5_4-G-3.81_1x04_P3.81mm_Vertical
- J13: footprint Connector_Phoenix_MC_HighVoltage:PhoenixContact_MCV_1,5_3-G-5.08_1x03_P5.08mm_Vertical -> Connector_Phoenix_MC:PhoenixContact_MCV_1,5_3-G-3.81_1x03_P3.81mm_Vertical
- J15: renamed from Brake1; footprint Connector_Phoenix_MC_HighVoltage:PhoenixContact_MCV_1,5_3-G-5.08_1x03_P5.08mm_Vertical -> Connector_Phoenix_MC:PhoenixContact_MCV_1,5_3-G-3.81_1x03_P3.81mm_Vertical
- J2: renamed from J3; footprint Connector_IDC:IDC-Header_2x05_P2.54mm_Vertical -> Connector_Phoenix_MC:PhoenixContact_MCV_1,5_10-G-3.81_1x10_P3.81mm_Vertical
- J3: renamed from J2; footprint Connector_Phoenix_MSTB:PhoenixContact_MSTBVA_2,5_6-G_1x06_P5.00mm_Vertical -> Connector_Phoenix_MC:PhoenixContact_MCV_1,5_6-G-3.81_1x06_P3.81mm_Vertical
- J4: footprint Connector_IDC:IDC-Header_2x05_P2.54mm_Vertical -> Connector_Phoenix_MC:PhoenixContact_MCV_1,5_10-G-3.81_1x10_P3.81mm_Vertical
- R11, R3, R7: moved to F.Cu
- R12: renamed from R14; moved to B.Cu
- R15: value 39 -> 2k
- R17: value 2k -> 20k
- R2: value 20k -> 30k
- R5, R9: moved to B.Cu
- moved J3 309.2 mm to (106.8, 43.1), turned to 180 degrees
- moved J4 293.9 mm to (126.8, 93.7), turned to 90 degrees
- moved L1 281.9 mm to (110.0, 139.1)
- moved J8 279.2 mm to (119.0, 71.8), turned to 270 degrees
- moved C62 256.6 mm to (123.2, 151.6), turned to 180 degrees
- moved J2 253.2 mm to (113.8, 28.3), turned to 180 degrees
- moved C63 238.4 mm to (136.8, 131.0), turned to 270 degrees
- moved TH1 235.2 mm to (90.2, 69.8), turned to 90 degrees
- moved J15 218.2 mm to (118.3, 56.7), turned to 180 degrees
- moved J13 215.5 mm to (104.3, 56.7), turned to 180 degrees
- moved J5 213.4 mm to (67.7, 64.6), turned to 270 degrees
- moved C61 211.3 mm to (108.7, 146.2), turned to 270 degrees
- moved C67 205.6 mm to (110.8, 135.7)
- moved U1 199.3 mm to (76.5, 51.8), turned to 180 degrees
- moved J14 196.7 mm to (103.4, 131.1)
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- renumbered C21 to C1, C8 to C10, C9 to C11, C10 to C12, C72 to C13, C19 to C18, C20 to C19, C22 to C2, C14 to C20, C15 to C21, C16 to C22, C17 to C23, C18 to C24, C73 to C27, C74 to C28, C25 to C29, C1 to C3, C26 to C30, C27 to C31, C69 to C32, C28 to C33, C29 to C34, C30 to C35, C31 to C36, C32 to C37, C70 to C38, C2 to C4, C35 to C41, C36 to C42, C39 to C45, C40 to C46, C41 to C47, C71 to C48, C42 to C49, C3 to C5, C43 to C50, C44 to C51, C47 to C54, C48 to C55, C49 to C56, C52 to C59, C4 to C6, C53 to C60, C54 to C61, C55 to C62, C62 to C63, C58 to C65, C60 to C67, C63 to C68, C64 to C69, C5 to C7, C67 to C71, C6 to C8, C7 to C9, D1 to D2, D2 to D3, R20 to R18, R21 to R19, R22 to R20, R23 to R21, R24 to R22, R25 to R23, R26 to R24, R27 to R25, R28 to R26, R29 to R27, R30 to R28, R31 to R29, R32 to R30, R33 to R31, R34 to R32, R35 to R33, R36 to R34, R37 to R35, R38 to R36, R39 to R37, R40 to R38, R41 to R39, R42 to R40, R43 to R41, R44 to R42, R45 to R43, R46 to R44, R48 to R46, R49 to R47, R50 to R48, R51 to R49, R52 to R50, R54 to R52, R55 to R53, R56 to R54, R57 to R55, R58 to R56, R59 to R57, R60 to R58, R61 to R59, R62 to R60, R63 to R61, R64 to R62, R65 to R63, R66 to R64, R68 to R66, R69 to R67, R70 to R68, R71 to R69, R72 to R70, R73 to R71, R74 to R72, R75 to R73, R76 to R74, R77 to R75, R78 to R76, R79 to R77, R80 to R78, R84 to R80, R82 to R81, R83 to R82, R95 to R83, R96 to R84, R97 to R85, R98 to R86, R99 to R87, R85 to R88, R86 to R89, R87 to R90, R88 to R91, R89 to R92, R90 to R93, R91 to R94, R92 to R95, R93 to R96, R94 to R97, U3 to U1, U12 to U10, U14 to U12, U15 to U13, U17 to U15, U18 to U16, U19 to U17, U20 to U18, U22 to U20, U24 to U21, U23 to U22, U25 to U23, U26 to U24, U6 to U4, U7 to U5, U8 to U6, U11 to U9
Connections:
- J14 pad 2: GND -> -BATT
- R11 pad 1: Net-(R10-Pad1) -> +VDC
- R11 pad 2: Net-(R11-Pad2) -> Net-(R10-Pad2)
- R15 pad 1: Net-(C23-Pad1) -> Net-(R13-Pad2)
- R15 pad 2: Net-(R15-Pad2) -> GND
- R16 pad 2: Net-(R16-Pad2) -> Net-(C14-Pad1)
- R17 pad 1: Net-(R15-Pad2) -> Net-(C14-Pad1)
- R2 pad 1: Net-(C11-Pad1) -> Net-(R13-Pad2)
- R2 pad 2: /DC_Bus_Voltage -> Net-(R2-Pad2)
- R3 pad 1: Net-(R15-Pad2) -> /TMC_VM
- R3 pad 2: Net-(R3-Pad2) -> Net-(R2-Pad2)
- R4 pad 1: Net-(R4-Pad1) -> /TMC_VM
- R4 pad 2: Net-(R3-Pad2) -> Net-(R4-Pad2)
- R5 pad 1: Net-(R4-Pad1) -> Net-(R5-Pad1)
- R5 pad 2: Net-(R5-Pad2) -> Net-(R4-Pad2)
- R6 pad 1: Net-(R6-Pad1) -> Net-(R5-Pad1)
- R6 pad 2: Net-(R5-Pad2) -> Net-(R6-Pad2)
- R7 pad 1: Net-(R6-Pad1) -> Net-(R7-Pad1)
- R7 pad 2: Net-(R7-Pad2) -> Net-(R6-Pad2)
- R8 pad 1: Net-(R8-Pad1) -> Net-(R7-Pad1)
- R8 pad 2: Net-(R7-Pad2) -> Net-(R8-Pad2)
- R9 pad 1: Net-(R8-Pad1) -> Net-(R10-Pad1)
- R9 pad 2: Net-(R10-Pad2) -> Net-(R8-Pad2)
Routing:
- net -BATT: track 0.00 -> 104.1 mm
- net /Motor_Current_V: track 2.01 -> 40.2 mm, vias 0 -> 1
- net +BATT: track 0.00 -> 35.7 mm
- net /PWM_VT: track 0.00 -> 14.7 mm
- net /PWM_VB: track 0.00 -> 14.7 mm
- net Net-(C11-Pad1): track 11.8 -> 0.00 mm, vias 2 -> 0
- net Net-(C14-Pad1): track 0.00 -> 11.8 mm, vias 0 -> 2
- net /PWM_WB: track 0.00 -> 10.5 mm, vias 0 -> 2
- net /PWM_WT: track 0.00 -> 9.77 mm, vias 0 -> 2
- net /PWM_UB: track 0.00 -> 9.77 mm, vias 0 -> 2
- net +5V: track 0.29 -> 9.44 mm
- net /TMC_VM: track 0.00 -> 8.76 mm
- net Net-(L1-Pad2): track 0.00 -> 8.17 mm
- net /PWM_UT: track 0.00 -> 7.29 mm, vias 0 -> 2
- net Net-(C23-Pad1): track 6.23 -> 0.00 mm, vias 1 -> 0
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- added copper zone on B.Cu, net +3V3
- added copper zone on F.Cu, net GND
Other:
- board size 185 x 192 mm -> 105.3 x 169.1 mm

Commit message: Change debug connectors, Motor W Voltage and round PCB corners
Parts:
- C45, C51, C54, C71, R52, R55, R56, R59, R60, R64, R67, R72: moved to B.Cu
- D1: value GREEN -> Green
- D2: value LED -> Blue
- D3: value LED -> White
- D4, D5, D6, D8: value LED -> Red
- D7: value LED -> Yellow
- J2, J4: footprint Connector_Phoenix_MC:PhoenixContact_MCV_1,5_10-G-3.81_1x10_P3.81mm_Vertical -> Connector_IDC:IDC-Header_2x05_P2.54mm_Vertical
- J3: value Program/Debug -> Debug; footprint Connector_Phoenix_MC:PhoenixContact_MCV_1,5_6-G-3.81_1x06_P3.81mm_Vertical -> Connector_IDC:IDC-Header_2x10_P2.54mm_Vertical
- moved Y2 268.0 mm to (104.8, 76.6), turned to 270 degrees
- moved Y1 263.8 mm to (100.5, 75.1)
- moved U15 257.9 mm to (122.1, 153.6), turned to 270 degrees
- moved C46 249.4 mm to (127.1, 147.3)
- moved C54 245.2 mm to (119.1, 158.3), turned to 270 degrees
- moved R67 244.6 mm to (121.1, 158.3), turned to 90 degrees
- moved C51 244.0 mm to (127.1, 149.3)
- moved C71 242.4 mm to (126.6, 134.3)
- moved R58 242.3 mm to (127.1, 157.2), turned to 180 degrees
- moved R60 239.2 mm to (127.1, 159.1), turned to 180 degrees
- moved C48 238.5 mm to (116.5, 151.9), turned to 180 degrees
- moved R59 235.8 mm to (127.1, 157.2), turned to 180 degrees
- moved R52 235.5 mm to (114.0, 156.1), turned to 90 degrees
- moved R57 232.8 mm to (127.1, 155.2), turned to 180 degrees
- moved R53 225.9 mm to (127.1, 151.2), turned to 180 degrees
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Connections:
- D3 pad 2: /ENABLE_INPUTS -> /SD_DET
- J2 pad 1: +5V -> +3V3
- J2 pad 3: +3V3 -> +5V
- J3 pad 2: /SWDIO -> (no net)
- J3 pad 3: /SWCLK -> (no net)
- J3 pad 4: /SWO -> GND
- J3 pad 5: /reset -> (no net)
Routing:
- net +BATT: track 35.7 -> 103.6 mm
- net /Motor_W: track 15.1 -> 30.4 mm
- net +VDC: track 16.4 -> 29.3 mm
- net Net-(C45-Pad1): track 0.00 -> 10.4 mm, vias 0 -> 1
- net +5V: track 9.44 -> 19.9 mm
- net /HSE_OUT: track 0.00 -> 8.80 mm
- net /HSE_IN: track 0.00 -> 7.46 mm
- net Net-(C51-Pad1): track 0.00 -> 6.89 mm, vias 0 -> 1
- net -BATT: track 104.1 -> 97.9 mm
- net +3V3: track 11.7 -> 16.2 mm, vias 0 -> 2
- net /Motor_Voltage_W: track 0.00 -> 3.58 mm, vias 0 -> 1
- net /LSE_IN: track 0.00 -> 3.11 mm
- net /LSE_OUT: track 0.00 -> 2.53 mm
- net GND: track 14.3 -> 11.9 mm, vias 5 -> 13
- net Net-(R55-Pad1): track 0.00 -> 1.98 mm
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Other:
- outline, holes or cut-outs redrawn
- net class supply added: clearance 0.4, trace_width 0.6, via_dia 0.8, via_drill 0.4

Commit message: Fix SPI
Parts:
- removed the R29 at (-2.67, 115.3)
- removed the R45 at (104.6, 118.6)
- added H1: MountingHole, MountingHole:MountingHole_5.3mm_M5, F.Cu at (33.8, 139.8)
- added H2: MountingHole, MountingHole:MountingHole_5.3mm_M5, F.Cu at (33.8, 151.9)
- added H3: MountingHole, MountingHole:MountingHole_5.3mm_M5, F.Cu at (155.0, 136.3)
- added H4: MountingHole, MountingHole:MountingHole_5.3mm_M5, F.Cu at (186.3, 75.0)
- added R44: 4.7k, Resistor_SMD:R_0805_2012Metric, B.Cu at (104.6, 118.6)
- moved J4 51.3 mm to (102.5, 74.5), turned to 0 degrees
- moved Y2 12.4 mm to (92.5, 75.9), turned to 180 degrees
- moved U6 7.11 mm to (90.8, 84.4)
- moved Y1 4.63 mm to (96.2, 77.0), turned to 90 degrees
- moved J13 2.80 mm to (104.3, 53.9)
- moved J15 2.80 mm to (118.3, 53.9)
- moved J8 2.80 mm to (118.9, 69.4)
- moved J12 1.77 mm to (79.8, 56.1)
- moved TH1 1.77 mm to (90.7, 68.1)
- moved J1 1.77 mm to (66.1, 52.2)
- moved J5 1.77 mm to (68.2, 62.9)
- moved R12 1.77 mm to (68.0, 49.6)
- moved U1 1.77 mm to (77.0, 50.1)
- moved J2 0.88 mm to (111.3, 43.8)
- renumbered R30 to R29, R31 to R30, R32 to R31, R33 to R32, R34 to R33, R35 to R34, R36 to R35, R37 to R36, R38 to R37, R39 to R38, R40 to R39, R41 to R40, R42 to R41, R43 to R42, R44 to R43, R46 to R45, R47 to R46, R48 to R47, R49 to R48, R50 to R49, R51 to R50, R52 to R51, R53 to R52, R54 to R53, R55 to R54, R56 to R55, R57 to R56, R58 to R57, R59 to R58, R60 to R59, R61 to R60, R62 to R61, R63 to R62, R64 to R63, R65 to R64, R66 to R65, R67 to R66, R68 to R67, R69 to R68, R70 to R69, R71 to R70, R72 to R71, R73 to R72, R74 to R73, R75 to R74, R76 to R75, R77 to R76, R78 to R77, R79 to R78, R80 to R79, R81 to R80, R82 to R81, R83 to R82, R84 to R83, R85 to R84, R86 to R85, R87 to R86, R88 to R87, R89 to R88, R90 to R89, R91 to R90, R92 to R91, R93 to R92, R94 to R93, R95 to R94, R96 to R95, R97 to R96
Connections:
- R3 pad 1: /TMC_VM -> Net-(R3-Pad1)
- R4 pad 1: /TMC_VM -> Net-(R3-Pad1)
- U7 pad 20: /TMC_VM -> (no net)
Routing:
- net /TMC_VM: track 8.76 -> 0.00 mm
- net /HSE_OUT: track 8.80 -> 2.23 mm
- net /LSE_IN: track 3.11 -> 7.48 mm
- net /LSE_OUT: track 2.53 -> 5.58 mm
- net /HSE_IN: track 7.46 -> 4.60 mm
- net Net-(R3-Pad1): track 0.00 -> 2.00 mm
- net GND: vias 13 -> 15
