File: hardware/motor_controller/electric-FIAT.kicad_pcb (KiCad board)
At the start: 2 copper layers, 105.3 x 169.1 mm, 232 parts, among them J1 CAN, J10 Motor_W, J11 SKiiP 613 GD123-3DUL V3, J12 Encoder, J13 Accelerator, J14 12V Battery, J15 5.1k, J2 Debug, J3 DC_Bus, J4 RTMI, J5 Micro_SD_Card_Det, J6 Batt_conn, J7 Motor_U, J8 IMU, J9 Motor_V, Q1 AO3400, Q2 AO3400, Q3 AO3400, Q4 AO3400, Q5 AO3400, Q6 AO3400, U1 MCP2562-E-SN, U10 OPA356xxDBV, U11 ACS759xCB-200B-PFF, U12 OPA356xxDBV, U13 74LVC1G14, U14 ACS759xCB-200B-PFF, U15 ACPL-C87A, U16 OPA356xxDBV, U17 OPA356xxDBV, U18 74LVC1G14, U19 ACS759xCB-200B-PFF, U2 ACPL-C87A, U20 74LVC1G14, U21 OPA356xxDBV, U22 OPA356xxDBV, U23 ITW1205SA, U24 IU1203SA, U25 TEN40-1215E, U26 OPA356xxDBV, U27 OPA356xxDBV, U3 OPA356xxDBV, U4 ACPL-C87A, U5 OPA356xxDBV, U6 STM32F405RGTx, U7 TMC4671-ES, U8 ACS759xCB-200B-PFF, U9 ACPL-C87A, Y1 32.768MHz, Y2 25MHz

Commit message: Silkscreen ready
Parts:
- removed the C48 at (79.7, 66.1)
- added C47: 100n, Capacitor_SMD:C_0805_2012Metric, F.Cu at (79.7, 66.1)
- J14: value 12V Battery -> 9-18V Battery
- renumbered C11 to C10, C12 to C11, C13 to C12, C14 to C13, C15 to C14, C16 to C15, C17 to C16, C18 to C17, C19 to C18, C20 to C19, C21 to C20, C22 to C21, C23 to C22, C24 to C23, C25 to C24, C26 to C25, C27 to C26, C28 to C27, C29 to C28, C30 to C29, C31 to C30, C32 to C31, C33 to C32, C34 to C33, C35 to C34, C36 to C35, C37 to C36, C38 to C37, C39 to C38, C40 to C39, C41 to C40, C42 to C41, C43 to C42, C44 to C43, C45 to C44, C46 to C45, C47 to C46, C49 to C48, C50 to C49, C51 to C50, C52 to C51, C53 to C52, C54 to C53, C55 to C54, C56 to C55, C57 to C56, C58 to C57, C59 to C58, C60 to C59, C61 to C60, C62 to C61, C63 to C62, C64 to C63, C65 to C64, C66 to C65, C67 to C66, C68 to C67, C69 to C68, C70 to C69, C71 to C70, C72 to C71, C73 to C72, C74 to C73, C75 to C74, C76 to C75, C77 to C76, C78 to C77, C79 to C78, C80 to C79, C81 to C80, C82 to C81
Connections:
- net /FOC_reset renamed Net-(R30-Pad2)

Commit message: Change voltage sensor resistors to match each other
Parts:
- R10, R11, R7, R8, R9: value 30k -> 27k
- R2, R3, R4, R5, R6: value 30k -> 33k
- R20, R32, R36, R47, R53, R65: value 10k -> 5k1
- R24, R25, R26, R40, R41, R42, R57, R58, R59: value 200k -> 220k
- R27, R28, R43, R44, R60, R61: value 200k -> 270k
- R29, R45, R62: value 200k -> 0
- R34, R35, R50, R51, R68, R73: value 10k -> 12k
- R63, R74: value 1.7k -> 1.5k
- R69, R71, R76, R78, R82, R84: value 1k -> 910
- R70, R72, R77, R79, R83, R85: value 1k -> 1k2
- R81: value 4.5k -> 4.7k
- R88: value 1.8k -> 2k
- R90: value 3.2k -> 3.3k
- R94: value 4.3k -> 4.7k
